File: io.sch (KiCad schematic (older format))
At the start: 1 part

Commit message: cpu power done
Other:
- moved on the sheet: IC?A
Changed lines of the file:
@@
 LIBS:tl5209
 LIBS:tl1963adcqr
+LIBS:ddr3_sdram
 LIBS:mateboard-cache
 EELAYER 25 0
@@
 $Descr A4 11693 8268
 encoding utf-8
-Sheet 4 4
+Sheet 4 6
 Title ""
 Date ""
@@
 L AM335X_ZCZ IC?
 U 1 1 589C81F5
-P 2075 1250
-F 0 "IC?" V 2025 1550 60  0000 C CNN
-F 1 "AM335X_ZCZ" V 2025 950 60  0000 C CNN
-F 2 "" H 2075 1250 60  0001 C CNN
-F 3 "" H 2075 1250 60  0001 C CNN
-	1    2075 1250
+P 675 1050
+F 0 "IC?" V 625 1350 60  0000 C CNN
+F 1 "AM335X_ZCZ" V 625 750 60  0000 C CNN
+F 2 "" H 675 1050 60  0001 C CNN
+F 3 "" H 675 1050 60  0001 C CNN
+	1    675  1050
 	1    0    0    -1
 $EndComp
