File: io.sch (KiCad schematic (older format))
At the start: 23 parts

Commit message: wip gpio
Parts:
- added C?: 10uF/10V, symbol C
- added R?: 10k, symbol R
- added U?: 24LC32AT-I, TO_SOT_Packages_SMD:SOT-23-5, symbol AT24CS32-STUM
Connections:
- net GNDD: now also C?.2, U?.2 (GND)
- net I2C0_SCL: now also U?.1 (SCL)
- net I2C0_SDA: now also U?.3 (SDA)
- net VDD_3V3B: now also C?.1, R?.1, U?.4 (VCC)
- new net: R?.2, U?.5 (WP)
Other:
- moved on the sheet: R?
Changed lines of the file:
@@
 $Descr A4 11693 8268
 encoding utf-8
-Sheet 4 10
+Sheet 10 10
 Title ""
 Date ""
@@
 Text HLabel 7500 800  2    60   BiDi ~ 0
 GPIO0_7
-Text HLabel 5950 4900 2    60   BiDi ~ 0
+Text HLabel 6325 4900 2    60   BiDi ~ 0
 I2C0_SCL
 Wire Wire Line
-	5700 4900 5950 4900
-Text HLabel 5950 4800 2    60   BiDi ~ 0
+	5700 4900 6175 4900
+Wire Wire Line
+	6175 4900 6325 4900
+Text HLabel 6325 4800 2    60   BiDi ~ 0
 I2C0_SDA
 Wire Wire Line
-	5700 4800 5950 4800
+	5700 4800 6175 4800
+Wire Wire Line
+	6175 4800 6325 4800
 $Comp
 L R R?
 U 1 1 58BBAFBC
-P 6650 4750
-F 0 "R?" V 6600 4925 50  0000 C CNN
-F 1 "1.5k" V 6650 4750 50  0000 C CNN
-F 2 "" V 6580 4750 50  0001 C CNN
-F 3 "" H 6650 4750 50  0001 C CNN
-	1    6650 4750
+P 7025 4750
+F 0 "R?" V 6975 4925 50  0000 C CNN
+F 1 "1.5k" V 7025 4750 50  0000 C CNN
+F 2 "" V 6955 4750 50  0001 C CNN
+F 3 "" H 7025 4750 50  0001 C CNN
+	1    7025 4750
 	0    1    1    0
 $EndComp
@@
 L R R?
 U 1 1 58BBB220
-P 6650 4850
-F 0 "R?" V 6600 5025 50  0000 C CNN
-F 1 "1.5k" V 6650 4850 50  0000 C CNN
-F 2 "" V 6580 4850 50  0001 C CNN
-F 3 "" H 6650 4850 50  0001 C CNN
-	1    6650 4850
-	0    1    1    0
-$EndComp
-Wire Wire Line
-	6500 4750 5800 4750
-Wire Wire Line
-	5800 4750 5800 4800
-Connection ~ 5800 4800
-Wire Wire Line
-	5800 4900 5800 4850
-Wire Wire Line
-	5800 4850 6500 4850
-Connection ~ 5800 4900
+P 7025 4850
+F 0 "R?" V 6975 5025 50  0000 C CNN
+F 1 "1.5k" V 7025 4850 50  0000 C CNN
+F 2 "" V 6955 4850 50  0001 C CNN
+F 3 "" H 7025 4850 50  0001 C CNN
+	1    7025 4850
+	0    1    1    0
+$EndComp
+Wire Wire Line
+	6875 4750 6175 4750
+Wire Wire Line
+	6175 4750 6175 4800
+Connection ~ 6175 4800
+Wire Wire Line
+	6175 4900 6175 4850
+Wire Wire Line
+	6175 4850 6875 4850
+Connection ~ 6175 4900
 $Comp
 L VDD_3V3B #PWR?
 U 1 1 58BBB25B
-P 6950 4800
-F 0 "#PWR?" H 6950 4650 50  0001 C CNN
-F 1 "VDD_3V3B" V 6950 5100 50  0000 C CNN
-F 2 "" H 6950 4800 50  0000 C CNN
-F 3 "" H 6950 4800 50  0000 C CNN
-	1    6950 4800
-	0    1    1    0
-$EndComp
-Wire Wire Line
-	6950 4800 6900 4800
-Wire Wire Line
-	6900 4750 6900 4850
-Wire Wire Line
-	6900 4750 6800 4750
-Wire Wire Line
-	6900 4850 6800 4850
-Connection ~ 6900 4800
+P 7325 4800
+F 0 "#PWR?" H 7325 4650 50  0001 C CNN
+F 1 "VDD_3V3B" V 7325 5100 50  0000 C CNN
+F 2 "" H 7325 4800 50  0000 C CNN
+F 3 "" H 7325 4800 50  0000 C CNN
+	1    7325 4800
+	0    1    1    0
+$EndComp
+Wire Wire Line
+	7325 4800 7275 4800
+Wire Wire Line
+	7275 4750 7275 4800
+Wire Wire Line
+	7275 4800 7275 4850
+Wire Wire Line
+	7275 4750 7175 4750
+Wire Wire Line
+	7275 4850 7175 4850
+Connection ~ 7275 4800
 Text HLabel 5950 4400 2    60   BiDi ~ 0
 I2C2_SCL
@@
 $EndComp
 Wire Wire Line
-	5675 3150 5775 3150
+	5675 3150 5725 3150
+Wire Wire Line
+	5725 3150 5775 3150
 Wire Wire Line
 	5775 3250 5725 3250
@@
 	8300 2800 8225 2800
 Wire Wire Line
-	8225 2750 8225 2950
+	8225 2750 8225 2800
+Wire Wire Line
+	8225 2800 8225 2950
 $Comp
 L VDD_3V3B #PWR?
@@
 	7200 3725 7200 3350
 Wire Wire Line
-	7125 3350 7775 3350
+	7125 3350 7200 3350
+Wire Wire Line
+	7200 3350 7775 3350
 $Comp
 L GNDD #PWR?
@@
 Wire Wire Line
 	5750 3850 5700 3850
+$Comp
+L VDD_3V3B #PWR?
+U 1 1 58B9D244
+P 9300 4500
+F 0 "#PWR?" H 9300 4350 50  0001 C CNN
+F 1 "VDD_3V3B" H 9300 4650 50  0000 C CNN
+F 2 "" H 9300 4500 50  0000 C CNN
+F 3 "" H 9300 4500 50  0000 C CNN
+	1    9300 4500
+	1    0    0    -1
+$EndComp
+$Comp
+L C C?
+U 1 1 58B9D24A
+P 8600 4550
+F 0 "C?" V 8650 4625 50  0000 L CNN
+F 1 "10uF/10V" V 8725 4325 50  0000 L CNN
+F 2 "" H 8638 4400 50  0000 C CNN
+F 3 "" H 8600 4550 50  0000 C CNN
+	1    8600 4550
+	0    1    1    0
+$EndComp
+$Comp
+L GNDD #PWR?
+U 1 1 58B9D251
+P 8450 4550
+F 0 "#PWR?" H 8450 4300 50  0001 C CNN
+F 1 "GNDD" V 8450 4350 50  0000 C CNN
+F 2 "" H 8450 4550 50  0000 C CNN
+F 3 "" H 8450 4550 50  0000 C CNN
+	1    8450 4550
+	0    1    1    0
+$EndComp
+Wire Wire Line
+	8750 4550 8800 4550
+Wire Wire Line
+	8800 4550 9300 4550
+Wire Wire Line
+	9300 4500 9300 4550
+Wire Wire Line
+	9300 4550 9300 4600
+Connection ~ 9300 4550
+$Comp
+L R R?
+U 1 1 58B9D25C
+P 8800 4950
+F 0 "R?" V 8880 4950 50  0000 C CNN
+F 1 "10k" V 8800 4950 50  0000 C CNN
+F 2 "" V 8730 4950 50  0001 C CNN
+F 3 "" H 8800 4950 50  0001 C CNN
+	1    8800 4950
+	1    0    0    -1
+$EndComp
+Wire Wire Line
+	8800 5100 8800 5150
+Wire Wire Line
+	8800 5150 8900 5150
+Wire Wire Line
+	8800 4550 8800 4800
+Connection ~ 8800 4550
+$Comp
+L GNDD #PWR?
+U 1 1 58B9D267
+P 9300 5350
+F 0 "#PWR?" H 9300 5100 50  0001 C CNN
+F 1 "GNDD" H 9300 5200 50  0000 C CNN
+F 2 "" H 9300 5350 50  0000 C CNN
+F 3 "" H 9300 5350 50  0000 C CNN
+	1    9300 5350
+	1    0    0    -1
+$EndComp
+Wire Wire Line
+	9700 5000 10300 5000
+Text Label 10300 4850 2    60   ~ 0
+I2C0_SDA
+Text Label 10300 5000 2    60   ~ 0
+I2C0_SCL
+$Comp
+L AT24CS32-STUM U?
+U 1 1 58B9D23D
+P 9300 4950
+F 0 "U?" H 9100 5200 50  0000 C CNN
+F 1 "24LC32AT-I" H 9600 4650 50  0000 C CNN
+F 2 "TO_SOT_Packages_SMD:SOT-23-5" H 9300 4950 50  0001 C CIN
+F 3 "" H 9300 4950 50  0001 C CNN
+	1    9300 4950
+	1    0    0    -1
+$EndComp
+Wire Wire Line
+	10300 4850 9700 4850
+Text Label 6125 4800 2    60   ~ 0
+I2C0_SDA
+Text Label 6125 4900 2    60   ~ 0
+I2C0_SCL
 $EndSCHEMATC
