File: io.sch (KiCad schematic (older format))
At the start: 26 parts

Commit message: gpio assignment done
Changed lines of the file:
@@
 I2C0_SCL
 Wire Wire Line
-	5700 4900 6175 4900
-Wire Wire Line
-	6175 4900 6325 4900
+	5700 4900 6325 4900
 Text HLabel 6325 4800 2    60   BiDi ~ 0
 I2C0_SDA
 Wire Wire Line
-	5700 4800 6175 4800
-Wire Wire Line
-	6175 4800 6325 4800
+	5700 4800 6325 4800
 $Comp
 L R R?
@@
 	7325 4800 7275 4800
 Wire Wire Line
-	7275 4750 7275 4800
-Wire Wire Line
-	7275 4800 7275 4850
+	7275 4750 7275 4850
 Wire Wire Line
 	7275 4750 7175 4750
@@
 $EndComp
 Wire Wire Line
-	5675 3150 5725 3150
-Wire Wire Line
-	5725 3150 5775 3150
+	5675 3150 5775 3150
 Wire Wire Line
 	5775 3250 5725 3250
@@
 	8300 2800 8225 2800
 Wire Wire Line
-	8225 2750 8225 2800
-Wire Wire Line
-	8225 2800 8225 2950
+	8225 2750 8225 2950
 $Comp
 L VDD_3V3B #PWR?
@@
 	7200 3725 7200 3350
 Wire Wire Line
-	7125 3350 7200 3350
-Wire Wire Line
-	7200 3350 7775 3350
+	7125 3350 7775 3350
 $Comp
 L GNDD #PWR?
@@
 $EndComp
 Wire Wire Line
-	8750 4550 8800 4550
-Wire Wire Line
-	8800 4550 9300 4550
-Wire Wire Line
-	9300 4500 9300 4550
-Wire Wire Line
-	9300 4550 9300 4600
+	8750 4550 9300 4550
+Wire Wire Line
+	9300 4500 9300 4600
 Connection ~ 9300 4550
 $Comp

Commit message: annotation, wip erc
Parts:
- gave numbers to parts that had none: 21
Changed lines of the file:
@@
 $EndDescr
 $Comp
-L AM335X_ZCZ IC?
+L AM335X_ZCZ IC2
 U 1 1 589C81F5
 P 675 1050
-F 0 "IC?" H 775 1550 60  0000 C CNN
+F 0 "IC2" H 775 1550 60  0000 C CNN
 F 1 "AM335X_ZCZ" H 1325 1550 60  0000 C CNN
 F 2 "" H 675 1050 60  0001 C CNN
@@
 P 675 1900
 AR Path="/58AE72E9" Ref="IC?"  Part="12"
-AR Path="/589C7F89/58AE72E9" Ref="IC?"  Part="12"
-F 0 "IC?" H 775 2250 60  0000 C CNN
+AR Path="/589C7F89/58AE72E9" Ref="IC2"  Part="12"
+F 0 "IC2" H 775 2250 60  0000 C CNN
 F 1 "AM335X_ZCZ" H 1400 2250 60  0000 C CNN
 F 2 "" H 675 1900 60  0001 C CNN
@@
 P 4975 2800
 AR Path="/58AD08D3" Ref="IC?"  Part="5"
-AR Path="/589C7F89/58AD08D3" Ref="IC?"  Part="5"
-F 0 "IC?" H 5075 3300 60  0000 C CNN
+AR Path="/589C7F89/58AD08D3" Ref="IC2"  Part="5"
+F 0 "IC2" H 5075 3300 60  0000 C CNN
 F 1 "AM335X_ZCZ" H 5150 2300 60  0000 C CNN
 F 2 "" H 4975 2800 60  0001 C CNN
@@
 $EndComp
 $Comp
-L AM335X_ZCZ IC?
+L AM335X_ZCZ IC2
 U 13 1 58AD1F79
 P 700 3700
-F 0 "IC?" H 800 4000 60  0000 C CNN
+F 0 "IC2" H 800 4000 60  0000 C CNN
 F 1 "AM335X_ZCZ" H 1400 4000 60  0000 C CNN
 F 2 "" H 700 3700 60  0001 C CNN
@@
 $EndComp
 $Comp
-L AM335X_ZCZ IC?
+L AM335X_ZCZ IC2
 U 14 1 58AD203C
 P 1900 4350
-F 0 "IC?" H 1975 4650 60  0000 C CNN
+F 0 "IC2" H 1975 4650 60  0000 C CNN
 F 1 "AM335X_ZCZ" H 2500 4650 60  0000 C CNN
 F 2 "" H 1900 4350 60  0001 C CNN
@@
 P 3200 4850
 AR Path="/58AD3B53" Ref="IC?"  Part="7"
-AR Path="/589C7F89/58AD3B53" Ref="IC?"  Part="7"
-F 0 "IC?" H 3050 4900 60  0000 C CNN
+AR Path="/589C7F89/58AD3B53" Ref="IC2"  Part="7"
+F 0 "IC2" H 3050 4900 60  0000 C CNN
 F 1 "AM335X_ZCZ" H 2900 4800 60  0000 C CNN
 F 2 "" H 3200 4850 60  0001 C CNN
@@
 GPIO3_18
 $Comp
-L R R?
+L R R122
 U 1 1 58B968BF
 P 7275 800
-F 0 "R?" V 7355 800 50  0000 C CNN
+F 0 "R122" V 7355 800 50  0000 C CNN
 F 1 "0R" V 7275 800 50  0000 C CNN
 F 2 "" V 7205 800 50  0001 C CNN
@@
 	5700 4800 6325 4800
 $Comp
-L R R?
+L R R119
 U 1 1 58BBAFBC
 P 7025 4750
-F 0 "R?" V 6975 4925 50  0000 C CNN
+F 0 "R119" V 6975 4925 50  0000 C CNN
 F 1 "1.5k" V 7025 4750 50  0000 C CNN
 F 2 "" V 6955 4750 50  0001 C CNN
@@
 $EndComp
 $Comp
-L R R?
+L R R120
 U 1 1 58BBB220
 P 7025 4850
-F 0 "R?" V 6975 5025 50  0000 C CNN
+F 0 "R120" V 6975 5025 50  0000 C CNN
 F 1 "1.5k" V 7025 4850 50  0000 C CNN
 F 2 "" V 6955 4850 50  0001 C CNN
@@
 Connection ~ 6175 4900
 $Comp
-L VDD_3V3B #PWR?
+L VDD_3V3B #PWR304
 U 1 1 58BBB25B
 P 7325 4800
-F 0 "#PWR?" H 7325 4650 50  0001 C CNN
+F 0 "#PWR304" H 7325 4650 50  0001 C CNN
 F 1 "VDD_3V3B" V 7325 5100 50  0000 C CNN
 F 2 "" H 7325 4800 50  0000 C CNN
@@
 	5675 2100 5900 2100
 $Comp
-L R R?
+L R R117
 U 1 1 58BBFAD4
 P 5925 3150
-F 0 "R?" V 5875 3325 50  0000 C CNN
+F 0 "R117" V 5875 3325 50  0000 C CNN
 F 1 "4.7k" V 5925 3150 50  0000 C CNN
 F 2 "" V 5855 3150 50  0001 C CNN
@@
 $EndComp
 $Comp
-L R R?
+L R R118
 U 1 1 58BBFADA
 P 5925 3250
-F 0 "R?" V 5875 3425 50  0000 C CNN
+F 0 "R118" V 5875 3425 50  0000 C CNN
 F 1 "4.7k" V 5925 3250 50  0000 C CNN
 F 2 "" V 5855 3250 50  0001 C CNN
@@
 Connection ~ 5725 3150
 $Comp
-L VDD_3V3B #PWR?
+L VDD_3V3B #PWR301
 U 1 1 58BC017C
 P 6125 3150
-F 0 "#PWR?" H 6125 3000 50  0001 C CNN
+F 0 "#PWR301" H 6125 3000 50  0001 C CNN
 F 1 "VDD_3V3B" V 6125 3450 50  0000 C CNN
 F 2 "" H 6125 3150 50  0000 C CNN
@@
 	6125 3150 6075 3150
 $Comp
-L GNDD #PWR?
+L GNDD #PWR302
 U 1 1 58BC0258
 P 6125 3250
-F 0 "#PWR?" H 6125 3000 50  0001 C CNN
+F 0 "#PWR302" H 6125 3000 50  0001 C CNN
 F 1 "GNDD" V 6125 3025 50  0000 C CNN
 F 2 "" H 6125 3250 50  0001 C CNN
@@
 AIN0
 $Comp
-L R R?
+L R R110
 U 1 1 58BC0457
 P 5925 2450
-F 0 "R?" V 5875 2625 50  0000 C CNN
+F 0 "R110" V 5875 2625 50  0000 C CNN
 F 1 "10k" V 5925 2450 50  0000 C CNN
 F 2 "" V 5855 2450 50  0001 C CNN
@@
 AIN1
 $Comp
-L R R?
+L R R111
 U 1 1 58BC05AC
 P 5925 2550
-F 0 "R?" V 5875 2725 50  0000 C CNN
+F 0 "R111" V 5875 2725 50  0000 C CNN
 F 1 "10k" V 5925 2550 50  0000 C CNN
 F 2 "" V 5855 2550 50  0001 C CNN
@@
 AIN2
 $Comp
-L R R?
+L R R112
 U 1 1 58BC05FD
 P 5925 2650
-F 0 "R?" V 5875 2825 50  0000 C CNN
+F 0 "R112" V 5875 2825 50  0000 C CNN
 F 1 "10k" V 5925 2650 50  0000 C CNN
 F 2 "" V 5855 2650 50  0001 C CNN
@@
 AIN3
 $Comp
-L R R?
+L R R113
 U 1 1 58BC0606
 P 5925 2750
-F 0 "R?" V 5875 2925 50  0000 C CNN
+F 0 "R113" V 5875 2925 50  0000 C CNN
 F 1 "10k" V 5925 2750 50  0000 C CNN
 F 2 "" V 5855 2750 50  0001 C CNN
@@
 AIN4
 $Comp
-L R R?
+L R R114
 U 1 1 58BC06AB
 P 5925 2850
-F 0 "R?" V 5875 3025 50  0000 C CNN
+F 0 "R114" V 5875 3025 50  0000 C CNN
 F 1 "10k" V 5925 2850 50  0000 C CNN
 F 2 "" V 5855 2850 50  0001 C CNN
@@
 AIN5
 $Comp
-L R R?
+L R R115
 U 1 1 58BC06B4
 P 5925 2950
-F 0 "R?" V 5875 3125 50  0000 C CNN
+F 0 "R115" V 5875 3125 50  0000 C CNN
 F 1 "10k" V 5925 2950 50  0000 C CNN
 F 2 "" V 5855 2950 50  0001 C CNN
@@
 AIN6
 $Comp
-L R R?
+L R R116
 U 1 1 58BC06BD
 P 5925 3050
-F 0 "R?" V 5875 3225 50  0000 C CNN
+F 0 "R116" V 5875 3225 50  0000 C CNN
 F 1 "10k" V 5925 3050 50  0000 C CNN
 F 2 "" V 5855 3050 50  0001 C CNN
@@
 	5950 4200 5700 4200
 $Comp
-L LOGIC-2G125_Dual_3ST_NonInv_Buffer IC?
+L LOGIC-2G125_Dual_3ST_NonInv_Buffer IC6
 U 1 1 58BC9C06
 P 8225 3400
-F 0 "IC?" H 8450 3000 50  0000 C CNN
+F 0 "IC6" H 8450 3000 50  0000 C CNN
 F 1 "SN74LVC2G241DCUR" H 8600 3775 25  0000 C CNN
 F 2 "" H 8225 3400 60  0001 C CNN
@@
 	8750 3250 8675 3250
 $Comp
-L GNDD #PWR?
+L GNDD #PWR308
 U 1 1 58BCA9AB
 P 8225 3925
-F 0 "#PWR?" H 8225 3675 50  0001 C CNN
+F 0 "#PWR308" H 8225 3675 50  0001 C CNN
 F 1 "GNDD" H 8225 3775 50  0000 C CNN
 F 2 "" H 8225 3925 50  0001 C CNN
@@
 	8225 3925 8225 3850
 $Comp
-L GNDD #PWR?
+L GNDD #PWR305
 U 1 1 58BCBFDB
 P 7775 3250
-F 0 "#PWR?" H 7775 3000 50  0001 C CNN
+F 0 "#PWR305" H 7775 3000 50  0001 C CNN
 F 1 "GNDD" V 7775 3025 50  0000 C CNN
 F 2 "" H 7775 3250 50  0001 C CNN
@@
 $EndComp
 $Comp
-L VDD_3V3B #PWR?
+L VDD_3V3B #PWR306
 U 1 1 58BCC036
 P 7775 3450
-F 0 "#PWR?" H 7775 3300 50  0001 C CNN
+F 0 "#PWR306" H 7775 3300 50  0001 C CNN
 F 1 "VDD_3V3B" V 7775 3750 50  0000 C CNN
 F 2 "" H 7775 3450 50  0000 C CNN
@@
 $EndComp
 $Comp
-L C C?
+L C C140
 U 1 1 58BCC9AB
 P 8450 2800
-F 0 "C?" V 8500 2875 50  0000 L CNN
+F 0 "C140" V 8500 2875 50  0000 L CNN
 F 1 "100nF/6.3V" V 8575 2400 50  0000 L CNN
 F 2 "" H 8488 2650 50  0000 C CNN
@@
 $EndComp
 $Comp
-L GNDD #PWR?
+L GNDD #PWR310
 U 1 1 58BCC9B2
 P 8600 2800
-F 0 "#PWR?" H 8600 2550 50  0001 C CNN
+F 0 "#PWR310" H 8600 2550 50  0001 C CNN
 F 1 "GNDD" V 8600 2600 50  0000 C CNN
 F 2 "" H 8600 2800 50  0000 C CNN
@@
 	8225 2750 8225 2950
 $Comp
-L VDD_3V3B #PWR?
+L VDD_3V3B #PWR307
 U 1 1 58BCCC2F
 P 8225 2750
-F 0 "#PWR?" H 8225 2600 50  0001 C CNN
+F 0 "#PWR307" H 8225 2600 50  0001 C CNN
 F 1 "VDD_3V3B" H 8225 2900 50  0000 C CNN
 F 2 "" H 8225 2750 50  0000 C CNN
@@
 Connection ~ 8225 2800
 $Comp
-L R R?
+L R R121
 U 1 1 58BCCDFA
 P 7200 3875
-F 0 "R?" V 7150 4050 50  0000 C CNN
+F 0 "R121" V 7150 4050 50  0000 C CNN
 F 1 "100k" V 7200 3875 50  0000 C CNN
 F 2 "" V 7130 3875 50  0001 C CNN
@@
 	7125 3350 7775 3350
 $Comp
-L GNDD #PWR?
+L GNDD #PWR303
 U 1 1 58BCD10A
 P 7200 4025
-F 0 "#PWR?" H 7200 3775 50  0001 C CNN
+F 0 "#PWR303" H 7200 3775 50  0001 C CNN
 F 1 "GNDD" H 7200 3875 50  0000 C CNN
 F 2 "" H 7200 4025 50  0001 C CNN
@@
 	8850 3450 8675 3450
 $Comp
-L TEST_1P J?
+L TEST_1P J14
 U 1 1 58BCE4DB
 P 5750 3850
-F 0 "J?" H 5750 4075 50  0000 C CNN
+F 0 "J14" H 5750 4075 50  0000 C CNN
 F 1 "TEST_1P" H 5750 4050 50  0001 C CNN
 F 2 "" H 5950 3850 50  0001 C CNN
@@
 $EndComp
 $Comp
-L TEST_1P J?
+L TEST_1P J15
 U 1 1 58BCE4E2
 P 5800 3750
-F 0 "J?" H 5800 3975 50  0000 C CNN
+F 0 "J15" H 5800 3975 50  0000 C CNN
 F 1 "TEST_1P" H 5800 3950 50  0001 C CNN
 F 2 "" H 6000 3750 50  0001 C CNN
@@
 	5750 3850 5700 3850
 $Comp
-L VDD_3V3B #PWR?
+L VDD_3V3B #PWR311
 U 1 1 58B9D244
 P 9300 4500
-F 0 "#PWR?" H 9300 4350 50  0001 C CNN
+F 0 "#PWR311" H 9300 4350 50  0001 C CNN
 F 1 "VDD_3V3B" H 9300 4650 50  0000 C CNN
 F 2 "" H 9300 4500 50  0000 C CNN
@@
 $EndComp
 $Comp
-L C C?
+L C C141
 U 1 1 58B9D24A
 P 8600 4550
-F 0 "C?" V 8650 4625 50  0000 L CNN
+F 0 "C141" V 8650 4625 50  0000 L CNN
 F 1 "10uF/10V" V 8725 4325 50  0000 L CNN
 F 2 "" H 8638 4400 50  0000 C CNN
@@
 $EndComp
 $Comp
-L GNDD #PWR?
+L GNDD #PWR309
 U 1 1 58B9D251
 P 8450 4550
-F 0 "#PWR?" H 8450 4300 50  0001 C CNN
+F 0 "#PWR309" H 8450 4300 50  0001 C CNN
 F 1 "GNDD" V 8450 4350 50  0000 C CNN
 F 2 "" H 8450 4550 50  0000 C CNN
@@
 Connection ~ 9300 4550
 $Comp
-L R R?
+L R R123
 U 1 1 58B9D25C
 P 8800 4950
-F 0 "R?" V 8880 4950 50  0000 C CNN
+F 0 "R123" V 8880 4950 50  0000 C CNN
 F 1 "10k" V 8800 4950 50  0000 C CNN
 F 2 "" V 8730 4950 50  0001 C CNN
@@
 Connection ~ 8800 4550
 $Comp
-L GNDD #PWR?
+L GNDD #PWR312
 U 1 1 58B9D267
 P 9300 5350
-F 0 "#PWR?" H 9300 5100 50  0001 C CNN
+F 0 "#PWR312" H 9300 5100 50  0001 C CNN
 F 1 "GNDD" H 9300 5200 50  0000 C CNN
 F 2 "" H 9300 5350 50  0000 C CNN
@@
 I2C0_SCL
 $Comp
-L AT24CS32-STUM U?
+L AT24CS32-STUM U11
 U 1 1 58B9D23D
 P 9300 4950
-F 0 "U?" H 9100 5200 50  0000 C CNN
+F 0 "U11" H 9100 5200 50  0000 C CNN
 F 1 "24LC32AT-I" H 9600 4650 50  0000 C CNN
 F 2 "TO_SOT_Packages_SMD:SOT-23-5" H 9300 4950 50  0001 C CIN
