File: mateboard.sch (KiCad schematic (older format))
At the start: 0 parts

Commit message: power mgmnt done
Parts:
- added P?: POWER, symbol USB_OTG
- added P?: HOST, symbol USB_A
- added P?: DEVICE, symbol USB_OTG
- added R?: 0.1, Resistors_SMD:R_0805, symbol R
Connections:
- new net GNDD: P?.5 (GND), R?.1
- new net GNDSHIELD: P?.5 (shield), P?.6 (shield), P?.6 (shield), R?.2
- new net VDD_5V: P?.1 (VBUS)
- no-connect marks 0 -> 3
Changed lines of the file:
@@
 LIBS:tps65217c
 LIBS:pwr
+LIBS:pushbutton
+LIBS:tl5209
+LIBS:tl1963adcqr
 LIBS:mateboard-cache
 EELAYER 25 0
@@
 $EndDescr
 $Sheet
-S 1025 950  2100 1675
+S 2375 1525 2100 1675
 U 589A190D
 F0 "Power Management" 60
@@
 $EndSheet
 $Sheet
-S 1000 2975 2100 2075
+S 2375 3650 2100 2075
 U 589C7F66
 F0 "DDR Memory" 60
@@
 F1 "io.sch" 60
 $EndSheet
+$Comp
+L USB_OTG P?
+U 1 1 589C9196
+P 1400 1100
+F 0 "P?" V 1725 975 50  0000 C CNN
+F 1 "POWER" V 1100 1100 50  0000 C CNN
+F 2 "" V 1350 1000 50  0000 C CNN
+F 3 "" V 1350 1000 50  0000 C CNN
+	1    1400 1100
+	0    -1   1    0
+$EndComp
+$Comp
+L USB_A P?
+U 1 1 589C92E9
+P 1425 3250
+F 0 "P?" V 1625 3050 50  0000 C CNN
+F 1 "HOST" V 1125 3250 50  0000 C CNN
+F 2 "" V 1375 3150 50  0000 C CNN
+F 3 "" V 1375 3150 50  0000 C CNN
+	1    1425 3250
+	0    -1   1    0
+$EndComp
+$Comp
+L USB_OTG P?
+U 1 1 589C94AD
+P 1400 2150
+F 0 "P?" V 1725 2025 50  0000 C CNN
+F 1 "DEVICE" V 1100 2150 50  0000 C CNN
+F 2 "" V 1350 2050 50  0000 C CNN
+F 3 "" V 1350 2050 50  0000 C CNN
+	1    1400 2150
+	0    -1   1    0
+$EndComp
+$Comp
+L GNDD #PWR?
+U 1 1 589C99DB
+P 1700 1300
+F 0 "#PWR?" H 1700 1050 50  0001 C CNN
+F 1 "GNDD" H 1700 1150 50  0000 C CNN
+F 2 "" H 1700 1300 50  0000 C CNN
+F 3 "" H 1700 1300 50  0000 C CNN
+	1    1700 1300
+	1    0    0    -1
+$EndComp
+$Comp
+L VDD_5V #PWR?
+U 1 1 589C99F5
+P 1700 900
+F 0 "#PWR?" H 1700 750 50  0001 C CNN
+F 1 "VDD_5V" V 1700 1175 50  0000 C CNN
+F 2 "" H 1700 900 50  0000 C CNN
+F 3 "" H 1700 900 50  0000 C CNN
+	1    1700 900
+	0    1    1    0
+$EndComp
+NoConn ~ 1700 1000
+NoConn ~ 1700 1100
+NoConn ~ 1700 1200
+$Comp
+L GNDSHIELD #PWR?
+U 1 1 589C9AC7
+P 1300 1500
+F 0 "#PWR?" H 1300 1550 40  0001 C CNN
+F 1 "GNDSHIELD" H 1300 1440 25  0000 C CNN
+F 2 "" H 1300 1500 60  0001 C CNN
+F 3 "" H 1300 1500 60  0001 C CNN
+	1    1300 1500
+	1    0    0    -1
+$EndComp
+$Comp
+L GNDSHIELD #PWR?
+U 1 1 589C9BDB
+P 1325 3550
+F 0 "#PWR?" H 1325 3600 40  0001 C CNN
+F 1 "GNDSHIELD" H 1325 3490 25  0000 C CNN
+F 2 "" H 1325 3550 60  0001 C CNN
+F 3 "" H 1325 3550 60  0001 C CNN
+	1    1325 3550
+	1    0    0    -1
+$EndComp
+$Comp
+L GNDSHIELD #PWR?
+U 1 1 589C9C79
+P 1300 2550
+F 0 "#PWR?" H 1300 2600 40  0001 C CNN
+F 1 "GNDSHIELD" H 1300 2490 25  0000 C CNN
+F 2 "" H 1300 2550 60  0001 C CNN
+F 3 "" H 1300 2550 60  0001 C CNN
+	1    1300 2550
+	1    0    0    -1
+$EndComp
+$Comp
+L GNDSHIELD #PWR?
+U 1 1 589C9CB7
+P 850 4000
+F 0 "#PWR?" H 850 4050 40  0001 C CNN
+F 1 "GNDSHIELD" H 850 3940 25  0000 C CNN
+F 2 "" H 850 4000 60  0001 C CNN
+F 3 "" H 850 4000 60  0001 C CNN
+	1    850  4000
+	1    0    0    -1
+$EndComp
+$Comp
+L GNDD #PWR?
+U 1 1 589C9CCE
+P 1475 3950
+F 0 "#PWR?" H 1475 3700 50  0001 C CNN
+F 1 "GNDD" H 1475 3800 50  0000 C CNN
+F 2 "" H 1475 3950 50  0000 C CNN
+F 3 "" H 1475 3950 50  0000 C CNN
+	1    1475 3950
+	1    0    0    -1
+$EndComp
+$Comp
+L R R?
+U 1 1 589C9CED
+P 1150 3900
+F 0 "R?" V 1230 3900 50  0000 C CNN
+F 1 "0.1" V 1150 3900 50  0000 C CNN
+F 2 "Resistors_SMD:R_0805" V 1080 3900 50  0001 C CNN
+F 3 "" H 1150 3900 50  0000 C CNN
+	1    1150 3900
+	0    1    1    0
+$EndComp
+Wire Wire Line
+	1000 3900 850  3900
+Wire Wire Line
+	850  3900 850  4000
+Wire Wire Line
+	1300 3900 1475 3900
+Wire Wire Line
+	1475 3900 1475 3950
 $EndSCHEMATC

Commit message: cpu power done
Parts:
- added IC? (x10): AM335X_ZCZ, symbol AM335X_ZCZ
Changed lines of the file:
@@
 LIBS:tl5209
 LIBS:tl1963adcqr
+LIBS:ddr3_sdram
 LIBS:mateboard-cache
 EELAYER 25 0
@@
 $Descr A4 11693 8268
 encoding utf-8
-Sheet 1 4
+Sheet 1 6
 Title ""
 Date ""
@@
 $EndDescr
 $Sheet
-S 2375 1525 2100 1675
+S 2600 850  1250 1650
 U 589A190D
 F0 "Power Management" 60
@@
 $EndSheet
 $Sheet
-S 2375 3650 2100 2075
+S 5275 850  1475 1650
 U 589C7F66
 F0 "DDR Memory" 60
@@
 $EndSheet
 $Sheet
-S 5675 2150 2100 2025
+S 5075 3875 2100 2025
 U 589C7F89
 F0 "GPIO - I2C - SPI - UART" 60
@@
 Wire Wire Line
 	1475 3900 1475 3950
+$Sheet
+S 3975 850  1175 1650
+U 589E2993
+F0 "CPU Power" 60
+F1 "cpu_power.sch" 60
+$EndSheet
+$Sheet
+S 6900 850  1725 1650
+U 58AC1B74
+F0 "System" 60
+F1 "system.sch" 60
+$EndSheet
+$Comp
+L AM335X_ZCZ IC?
+U 5 1 58AC1D76
+P 9825 2025
+F 0 "IC?" V 9775 2325 60  0000 C CNN
+F 1 "AM335X_ZCZ" V 9775 1725 60  0000 C CNN
+F 2 "" H 9825 2025 60  0001 C CNN
+F 3 "" H 9825 2025 60  0001 C CNN
+	5    9825 2025
+	1    0    0    -1
+$EndComp
+$Comp
+L AM335X_ZCZ IC?
+U 6 1 58AC1DC3
+P 11600 3000
+F 0 "IC?" V 11550 3300 60  0000 C CNN
+F 1 "AM335X_ZCZ" V 11550 2700 60  0000 C CNN
+F 2 "" H 11600 3000 60  0001 C CNN
+F 3 "" H 11600 3000 60  0001 C CNN
+	6    11600 3000
+	1    0    0    -1
+$EndComp
+$Comp
+L AM335X_ZCZ IC?
+U 7 1 58AC1E72
+P 11275 16175
+F 0 "IC?" V 11225 16475 60  0000 C CNN
+F 1 "AM335X_ZCZ" V 11225 15875 60  0000 C CNN
+F 2 "" H 11275 16175 60  0001 C CNN
+F 3 "" H 11275 16175 60  0001 C CNN
+	7    11275 16175
+	1    0    0    -1
+$EndComp
+$Comp
+L AM335X_ZCZ IC?
+U 8 1 58AC1F48
+P 11550 6225
+F 0 "IC?" V 11500 6525 60  0000 C CNN
+F 1 "AM335X_ZCZ" V 11500 5925 60  0000 C CNN
+F 2 "" H 11550 6225 60  0001 C CNN
+F 3 "" H 11550 6225 60  0001 C CNN
+	8    11550 6225
+	1    0    0    -1
+$EndComp
+$Comp
+L AM335X_ZCZ IC?
+U 9 1 58AC20AF
+P 11525 8400
+F 0 "IC?" V 11475 8700 60  0000 C CNN
+F 1 "AM335X_ZCZ" V 11475 8100 60  0000 C CNN
+F 2 "" H 11525 8400 60  0001 C CNN
+F 3 "" H 11525 8400 60  0001 C CNN
+	9    11525 8400
+	1    0    0    -1
+$EndComp
+$Comp
+L AM335X_ZCZ IC?
+U 10 1 58AC21F3
+P 11600 10000
+F 0 "IC?" V 11550 10300 60  0000 C CNN
+F 1 "AM335X_ZCZ" V 11550 9700 60  0000 C CNN
+F 2 "" H 11600 10000 60  0001 C CNN
+F 3 "" H 11600 10000 60  0001 C CNN
+	10   11600 10000
+	1    0    0    -1
+$EndComp
+$Comp
+L AM335X_ZCZ IC?
+U 11 1 58AC22BA
+P 11425 11600
+F 0 "IC?" V 11375 11900 60  0000 C CNN
+F 1 "AM335X_ZCZ" V 11375 11300 60  0000 C CNN
+F 2 "" H 11425 11600 60  0001 C CNN
+F 3 "" H 11425 11600 60  0001 C CNN
+	11   11425 11600
+	1    0    0    -1
+$EndComp
+$Comp
+L AM335X_ZCZ IC?
+U 12 1 58AC233F
+P 11300 13000
+F 0 "IC?" V 11250 13300 60  0000 C CNN
+F 1 "AM335X_ZCZ" V 11250 12700 60  0000 C CNN
+F 2 "" H 11300 13000 60  0001 C CNN
+F 3 "" H 11300 13000 60  0001 C CNN
+	12   11300 13000
+	1    0    0    -1
+$EndComp
+$Comp
+L AM335X_ZCZ IC?
+U 13 1 58AC2482
+P 11250 14125
+F 0 "IC?" V 11200 14425 60  0000 C CNN
+F 1 "AM335X_ZCZ" V 11200 13825 60  0000 C CNN
+F 2 "" H 11250 14125 60  0001 C CNN
+F 3 "" H 11250 14125 60  0001 C CNN
+	13   11250 14125
+	1    0    0    -1
+$EndComp
+$Comp
+L AM335X_ZCZ IC?
+U 14 1 58AC2515
+P 11225 15275
+F 0 "IC?" V 11175 15575 60  0000 C CNN
+F 1 "AM335X_ZCZ" V 11175 14975 60  0000 C CNN
+F 2 "" H 11225 15275 60  0001 C CNN
+F 3 "" H 11225 15275 60  0001 C CNN
+	14   11225 15275
+	1    0    0    -1
+$EndComp
 $EndSCHEMATC

Commit message: emmc nand and micro sd
Parts:
- removed IC? (x4): AM335X_ZCZ, symbol AM335X_ZCZ
- added P?: microSD, symbol microSD
- added R? (x7): 10k, symbol R
Connections:
- net GNDD: now also P?.4 (GND), P?.5 (GND), P?.10 (DetectSW), P?.6 (VSS)
- net GNDSHIELD: now also P?.11 (SHIELD)
- net USB1_VBUS: now reaches P?.1 (VBUS)
- net USB1_DM: now reaches P?.2 (D-)
- net USB1_DP: now reaches P?.3 (D+)
- net USB_DC: now reaches P?.1 (VBUS)
- net USB0_DM: now reaches P?.2 (D-)
- net USB0_DP: now reaches P?.3 (D+)
- net USB0_ID: now reaches P?.4 (ID)
- new net GPIO-I2C-SPI-UART/MMC0_CD: P?.9 (DetectSW), R?.2
- new net MMC Interface/MMC0_CLK: P?.5 (CLK), R?.2
- new net MMC Interface/MMC0_CMD: P?.3 (CMD), R?.2
- new net MMC Interface/MMC0_DAT0: P?.7 (DAT0), R?.2
- new net MMC Interface/MMC0_DAT1: P?.8 (DAT1), R?.2
- new net MMC Interface/MMC0_DAT2: P?.1 (DAT2), R?.2
- new net MMC Interface/MMC0_DAT3: P?.2 (DAT3/CD), R?.2
- new net VDD_3V3B: P?.4 (VDD), R?.1, R?.1, R?.1, R?.1, R?.1, R?.1, R?.1
Other:
- moved on the sheet: IC?E

Commit message: usb
Other:
- moved on the sheet: P?, R?
Changed lines of the file:
@@
 LIBS:nand_4gb
 LIBS:microsd
+LIBS:tpd4s012
+LIBS:tps2065cdgn
 LIBS:mateboard-cache
 EELAYER 25 0
@@
 $EndSheet
 $Sheet
-S 2550 5100 1475 1650
+S 3825 4200 1475 1650
 U 589C7F66
 F0 "DDR Memory" 60
@@
 L USB_OTG P?
 U 1 1 589C9196
-P 1400 1100
-F 0 "P?" V 1725 975 50  0000 C CNN
-F 1 "POWER" V 1100 1100 50  0000 C CNN
-F 2 "" V 1350 1000 50  0000 C CNN
-F 3 "" V 1350 1000 50  0000 C CNN
-	1    1400 1100
+P 1175 2000
+F 0 "P?" V 1500 1875 50  0000 C CNN
+F 1 "POWER" V 875 2000 50  0000 C CNN
+F 2 "" V 1125 1900 50  0000 C CNN
+F 3 "" V 1125 1900 50  0000 C CNN
+	1    1175 2000
 	0    -1   1    0
 $EndComp
@@
 L USB_A P?
 U 1 1 589C92E9
-P 1425 3250
-F 0 "P?" V 1625 3125 50  0000 C CNN
-F 1 "HOST" V 1125 3250 50  0000 C CNN
-F 2 "" V 1375 3150 50  0000 C CNN
-F 3 "" V 1375 3150 50  0000 C CNN
-	1    1425 3250
+P 1175 3800
+F 0 "P?" V 1375 3675 50  0000 C CNN
+F 1 "HOST" V 875 3800 50  0000 C CNN
+F 2 "" V 1125 3700 50  0000 C CNN
+F 3 "" V 1125 3700 50  0000 C CNN
+	1    1175 3800
 	0    -1   1    0
 $EndComp
@@
 L USB_OTG P?
 U 1 1 589C94AD
-P 1400 2150
-F 0 "P?" V 1700 2025 50  0000 C CNN
-F 1 "DEVICE" V 1100 2150 50  0000 C CNN
-F 2 "" V 1350 2050 50  0000 C CNN
-F 3 "" V 1350 2050 50  0000 C CNN
-	1    1400 2150
+P 1175 2900
+F 0 "P?" V 1475 2775 50  0000 C CNN
+F 1 "DEVICE" V 875 2900 50  0000 C CNN
+F 2 "" V 1125 2800 50  0000 C CNN
+F 3 "" V 1125 2800 50  0000 C CNN
+	1    1175 2900
 	0    -1   1    0
 $EndComp
@@
 L GNDD #PWR?
 U 1 1 589C99DB
-P 1700 1300
-F 0 "#PWR?" H 1700 1050 50  0001 C CNN
-F 1 "GNDD" H 1700 1150 50  0000 C CNN
-F 2 "" H 1700 1300 50  0000 C CNN
-F 3 "" H 1700 1300 50  0000 C CNN
-	1    1700 1300
+P 1475 2200
+F 0 "#PWR?" H 1475 1950 50  0001 C CNN
+F 1 "GNDD" H 1475 2050 50  0000 C CNN
+F 2 "" H 1475 2200 50  0000 C CNN
+F 3 "" H 1475 2200 50  0000 C CNN
+	1    1475 2200
 	1    0    0    -1
 $EndComp
@@
 L VDD_5V #PWR?
 U 1 1 589C99F5
-P 1700 900
-F 0 "#PWR?" H 1700 750 50  0001 C CNN
-F 1 "VDD_5V" V 1700 1175 50  0000 C CNN
-F 2 "" H 1700 900 50  0000 C CNN
-F 3 "" H 1700 900 50  0000 C CNN
-	1    1700 900
+P 1475 1800
+F 0 "#PWR?" H 1475 1650 50  0001 C CNN
+F 1 "VDD_5V" V 1475 2075 50  0000 C CNN
+F 2 "" H 1475 1800 50  0000 C CNN
+F 3 "" H 1475 1800 50  0000 C CNN
+	1    1475 1800
 	0    1    1    0
 $EndComp
-NoConn ~ 1700 1000
-NoConn ~ 1700 1100
-NoConn ~ 1700 1200
+NoConn ~ 1475 1900
+NoConn ~ 1475 2000
+NoConn ~ 1475 2100
 $Comp
 L GNDSHIELD #PWR?
 U 1 1 589C9AC7
-P 1300 1500
-F 0 "#PWR?" H 1300 1550 40  0001 C CNN
-F 1 "GNDSHIELD" H 1300 1440 25  0000 C CNN
-F 2 "" H 1300 1500 60  0001 C CNN
-F 3 "" H 1300 1500 60  0001 C CNN
-	1    1300 1500
+P 1075 2400
+F 0 "#PWR?" H 1075 2450 40  0001 C CNN
+F 1 "GNDSHIELD" H 1075 2340 25  0000 C CNN
+F 2 "" H 1075 2400 60  0001 C CNN
+F 3 "" H 1075 2400 60  0001 C CNN
+	1    1075 2400
 	1    0    0    -1
 $EndComp
@@
 L GNDSHIELD #PWR?
 U 1 1 589C9BDB
-P 1325 3550
-F 0 "#PWR?" H 1325 3600 40  0001 C CNN
-F 1 "GNDSHIELD" H 1325 3490 25  0000 C CNN
-F 2 "" H 1325 3550 60  0001 C CNN
-F 3 "" H 1325 3550 60  0001 C CNN
-	1    1325 3550
+P 1075 4100
+F 0 "#PWR?" H 1075 4150 40  0001 C CNN
+F 1 "GNDSHIELD" H 1075 4040 25  0000 C CNN
+F 2 "" H 1075 4100 60  0001 C CNN
+F 3 "" H 1075 4100 60  0001 C CNN
+	1    1075 4100
 	1    0    0    -1
 $EndComp
@@
 L GNDSHIELD #PWR?
 U 1 1 589C9C79
-P 1300 2550
-F 0 "#PWR?" H 1300 2600 40  0001 C CNN
-F 1 "GNDSHIELD" H 1300 2490 25  0000 C CNN
-F 2 "" H 1300 2550 60  0001 C CNN
-F 3 "" H 1300 2550 60  0001 C CNN
-	1    1300 2550
+P 1075 3300
+F 0 "#PWR?" H 1075 3350 40  0001 C CNN
+F 1 "GNDSHIELD" H 1075 3240 25  0000 C CNN
+F 2 "" H 1075 3300 60  0001 C CNN
+F 3 "" H 1075 3300 60  0001 C CNN
+	1    1075 3300
 	1    0    0    -1
 $EndComp
@@
 L GNDSHIELD #PWR?
 U 1 1 589C9CB7
-P 850 4000
-F 0 "#PWR?" H 850 4050 40  0001 C CNN
-F 1 "GNDSHIELD" H 850 3940 25  0000 C CNN
-F 2 "" H 850 4000 60  0001 C CNN
-F 3 "" H 850 4000 60  0001 C CNN
-	1    850  4000
+P 875 4475
+F 0 "#PWR?" H 875 4525 40  0001 C CNN
+F 1 "GNDSHIELD" H 875 4415 25  0000 C CNN
+F 2 "" H 875 4475 60  0001 C CNN
+F 3 "" H 875 4475 60  0001 C CNN
+	1    875  4475
 	1    0    0    -1
 $EndComp
@@
 L GNDD #PWR?
 U 1 1 589C9CCE
-P 1475 3950
-F 0 "#PWR?" H 1475 3700 50  0001 C CNN
-F 1 "GNDD" H 1475 3800 50  0000 C CNN
-F 2 "" H 1475 3950 50  0000 C CNN
-F 3 "" H 1475 3950 50  0000 C CNN
-	1    1475 3950
+P 1500 4425
+F 0 "#PWR?" H 1500 4175 50  0001 C CNN
+F 1 "GNDD" H 1500 4275 50  0000 C CNN
+F 2 "" H 1500 4425 50  0000 C CNN
+F 3 "" H 1500 4425 50  0000 C CNN
+	1    1500 4425
 	1    0    0    -1
 $EndComp
@@
 L R R?
 U 1 1 589C9CED
-P 1150 3900
-F 0 "R?" V 1230 3900 50  0000 C CNN
-F 1 "0.1" V 1150 3900 50  0000 C CNN
-F 2 "Resistors_SMD:R_0805" V 1080 3900 50  0001 C CNN
-F 3 "" H 1150 3900 50  0000 C CNN
-	1    1150 3900
+P 1175 4375
+F 0 "R?" V 1255 4375 50  0000 C CNN
+F 1 "0.1" V 1175 4375 50  0000 C CNN
+F 2 "Resistors_SMD:R_0805" V 1105 4375 50  0001 C CNN
+F 3 "" H 1175 4375 50  0000 C CNN
+	1    1175 4375
 	0    1    1    0
 $EndComp
 Wire Wire Line
-	1000 3900 850  3900
-Wire Wire Line
-	850  3900 850  4000
-Wire Wire Line
-	1300 3900 1475 3900
-Wire Wire Line
-	1475 3900 1475 3950
-$Sheet
-S 1325 5100 1175 1650
+	1025 4375 875  4375
+Wire Wire Line
+	875  4375 875  4475
+Wire Wire Line
+	1325 4375 1500 4375
+Wire Wire Line
+	1500 4375 1500 4425
+$Sheet
+S 2600 4200 1175 1650
 U 589E2993
 F0 "CPU Power" 60
@@
 F6 "MMC0_CMD" O R 8150 1450 60
 F7 "MMC0_CLK" O R 8150 1650 60
+F8 "USB1_OCn" I L 6900 2400 60
 $EndSheet
 $Comp
@@
 L USB_DC #PWR?
 U 1 1 58AEF700
-P 2100 1950
-F 0 "#PWR?" H 2100 1800 50  0001 C CNN
-F 1 "USB_DC" V 2100 2200 50  0000 C CNN
-F 2 "" H 2100 1950 50  0000 C CNN
-F 3 "" H 2100 1950 50  0000 C CNN
-	1    2100 1950
+P 1875 2700
+F 0 "#PWR?" H 1875 2550 50  0001 C CNN
+F 1 "USB_DC" V 1875 2950 50  0000 C CNN
+F 2 "" H 1875 2700 50  0000 C CNN
+F 3 "" H 1875 2700 50  0000 C CNN
+	1    1875 2700
 	0    1    1    0
 $EndComp
 $Sheet
-S 2600 2700 1250 1100
+S 2600 2700 1250 1200
 U 58AF1DA5
 F0 "USB" 60
 F1 "usb.sch" 60
-$EndSheet
-Wire Wire Line
-	1700 2050 2150 2050
-Text Label 2150 2250 2    60   ~ 0
+F2 "USB0_DP" B L 2600 2900 60
+F3 "USB0_DM" B L 2600 2800 60
+F4 "USB0_ID" B L 2600 3000 60
+F5 "USB1_DP" B L 2600 3800 60
+F6 "USB1_DM" B L 2600 3700 60
+F7 "USB1_VBUS" O L 2600 3600 60
+F8 "USB1_OCn" O R 3850 2800 60
+$EndSheet
+Wire Wire Line
+	1475 2800 2600 2800
+Text Label 1925 3000 2    60   ~ 0
 USB0_ID
 Wire Wire Line
-	2150 2250 1700 2250
-Text Label 2150 2050 2    60   ~ 0
+	1475 3000 2600 3000
+Text Label 1925 2800 2    60   ~ 0
 USB0_DM
 Wire Wire Line
-	1700 2150 2150 2150
-Text Label 2150 2150 2    60   ~ 0
+	1475 2900 2600 2900
+Text Label 1925 2900 2    60   ~ 0
 USB0_DP
 Wire Wire Line
-	2100 1950 1700 1950
+	1875 2700 1475 2700
 $Comp
 L GNDD #PWR?
 U 1 1 58AFBFA2
-P 1700 2350
-F 0 "#PWR?" H 1700 2100 50  0001 C CNN
-F 1 "GNDD" H 1700 2200 50  0000 C CNN
-F 2 "" H 1700 2350 50  0000 C CNN
-F 3 "" H 1700 2350 50  0000 C CNN
-	1    1700 2350
-	1    0    0    -1
-$EndComp
-Wire Wire Line
-	1725 3150 2175 3150
-Text Label 2175 3150 2    60   ~ 0
+P 1475 3100
+F 0 "#PWR?" H 1475 2850 50  0001 C CNN
+F 1 "GNDD" H 1475 2950 50  0000 C CNN
+F 2 "" H 1475 3100 50  0000 C CNN
+F 3 "" H 1475 3100 50  0000 C CNN
+	1    1475 3100
+	1    0    0    -1
+$EndComp
+Wire Wire Line
+	1475 3700 2600 3700
+Text Label 1925 3700 2    60   ~ 0
 USB1_DM
 Wire Wire Line
-	1725 3250 2175 3250
-Text Label 2175 3250 2    60   ~ 0
+	1475 3800 2600 3800
+Text Label 1925 3800 2    60   ~ 0
 USB1_DP
 Wire Wire Line
-	1725 3050 2175 3050
-Text Label 2175 3050 2    60   ~ 0
+	1475 3600 2600 3600
+Text Label 2025 3600 2    60   ~ 0
 USB1_VBUS
 $Comp
 L GNDD #PWR?
 U 1 1 58AFD11B
-P 1725 3350
-F 0 "#PWR?" H 1725 3100 50  0001 C CNN
-F 1 "GNDD" H 1725 3200 50  0000 C CNN
-F 2 "" H 1725 3350 50  0000 C CNN
-F 3 "" H 1725 3350 50  0000 C CNN
-	1    1725 3350
-	1    0    0    -1
-$EndComp
+P 1475 3900
+F 0 "#PWR?" H 1475 3650 50  0001 C CNN
+F 1 "GNDD" H 1475 3750 50  0000 C CNN
+F 2 "" H 1475 3900 50  0000 C CNN
+F 3 "" H 1475 3900 50  0000 C CNN
+	1    1475 3900
+	1    0    0    -1
+$EndComp
+Wire Wire Line
+	3850 2800 4400 2800
+Text Label 4400 2800 2    60   ~ 0
+USB1_OCn
+Wire Wire Line
+	6350 2400 6900 2400
+Text Label 6350 2400 0    60   ~ 0
+USB1_OCn
 $EndSCHEMATC

Commit message: hierarchical sheets defined
Parts:
- removed IC? (x6): AM335X_ZCZ, symbol AM335X_ZCZ
Changed lines of the file:
@@
 $Descr A4 11693 8268
 encoding utf-8
-Sheet 1 8
+Sheet 1 9
 Title ""
 Date ""
@@
 F1 "system.sch" 60
 $EndSheet
-$Comp
-L AM335X_ZCZ IC?
-U 5 1 58AC1D76
-P 13175 1850
-F 0 "IC?" V 13125 2150 60  0000 C CNN
-F 1 "AM335X_ZCZ" V 13125 1550 60  0000 C CNN
-F 2 "" H 13175 1850 60  0001 C CNN
-F 3 "" H 13175 1850 60  0001 C CNN
-	5    13175 1850
-	1    0    0    -1
-$EndComp
-$Comp
-L AM335X_ZCZ IC?
-U 7 1 58AC1E72
-P 11275 16175
-F 0 "IC?" V 11225 16475 60  0000 C CNN
-F 1 "AM335X_ZCZ" V 11225 15875 60  0000 C CNN
-F 2 "" H 11275 16175 60  0001 C CNN
-F 3 "" H 11275 16175 60  0001 C CNN
-	7    11275 16175
-	1    0    0    -1
-$EndComp
-$Comp
-L AM335X_ZCZ IC?
-U 8 1 58AC1F48
-P 11550 6225
-F 0 "IC?" V 11500 6525 60  0000 C CNN
-F 1 "AM335X_ZCZ" V 11500 5925 60  0000 C CNN
-F 2 "" H 11550 6225 60  0001 C CNN
-F 3 "" H 11550 6225 60  0001 C CNN
-	8    11550 6225
-	1    0    0    -1
-$EndComp
-$Comp
-L AM335X_ZCZ IC?
-U 9 1 58AC20AF
-P 11525 8400
-F 0 "IC?" V 11475 8700 60  0000 C CNN
-F 1 "AM335X_ZCZ" V 11475 8100 60  0000 C CNN
-F 2 "" H 11525 8400 60  0001 C CNN
-F 3 "" H 11525 8400 60  0001 C CNN
-	9    11525 8400
-	1    0    0    -1
-$EndComp
-$Comp
-L AM335X_ZCZ IC?
-U 13 1 58AC2482
-P 11250 14125
-F 0 "IC?" V 11200 14425 60  0000 C CNN
-F 1 "AM335X_ZCZ" V 11200 13825 60  0000 C CNN
-F 2 "" H 11250 14125 60  0001 C CNN
-F 3 "" H 11250 14125 60  0001 C CNN
-	13   11250 14125
-	1    0    0    -1
-$EndComp
-$Comp
-L AM335X_ZCZ IC?
-U 14 1 58AC2515
-P 11225 15275
-F 0 "IC?" V 11175 15575 60  0000 C CNN
-F 1 "AM335X_ZCZ" V 11175 14975 60  0000 C CNN
-F 2 "" H 11225 15275 60  0001 C CNN
-F 3 "" H 11225 15275 60  0001 C CNN
-	14   11225 15275
-	1    0    0    -1
-$EndComp
 $Sheet
 S 6900 850  1250 1650
@@
 $EndComp
 Wire Wire Line
-	3850 2800 4400 2800
+	3850 2800 6350 2800
 Text Label 4400 2800 2    60   ~ 0
 USB1_OCn
 Wire Wire Line
 	6350 2400 6900 2400
-Text Label 6350 2400 0    60   ~ 0
-USB1_OCn
+$Sheet
+S 6900 4550 1250 1550
+U 58AD6197
+F0 "Wi-Fi BLE" 60
+F1 "wifi.sch" 60
+$EndSheet
+Wire Wire Line
+	6350 2800 6350 2400
 $EndSCHEMATC

Commit message: system sheet
Connections:
- net GPIO-I2C-SPI-UART/MMC0_CD renamed MMC0_CD
Changed lines of the file:
@@
 LIBS:tpd4s012
 LIBS:tps2065cdgn
+LIBS:74lvc1g07dck
 LIBS:mateboard-cache
 EELAYER 25 0
@@
 F0 "CPU Power" 60
 F1 "cpu_power.sch" 60
-$EndSheet
-$Sheet
-S 4200 850  1725 1650
+F2 "VSS_RTC" B L 2600 5750 60
+$EndSheet
+$Sheet
+S 4400 850  1725 1650
 U 58AC1B74
 F0 "System" 60
 F1 "system.sch" 60
+F2 "NMIn" I L 4400 2000 60
+F3 "WAKEUP" I L 4400 1900 60
+F4 "VSS_RTC" B R 6125 1000 60
+F5 "POR" I L 4400 1700 60
+F6 "RTC_POR" I L 4400 1800 60
+F7 "SYS_RESETn" O R 6125 1200 60
+F8 "JTAG_EMU4" O R 6125 1100 60
+F9 "PMIC_POWER_EN" O L 4400 1000 60
+F10 "GPIO0_7" B R 6125 1300 60
 $EndSheet
 $Sheet
@@
 Wire Wire Line
 	6350 2800 6350 2400
+Wire Wire Line
+	4400 2000 3850 2000
+Wire Wire Line
+	4400 1900 3850 1900
+Wire Wire Line
+	2600 5750 2175 5750
+Text Label 2175 5750 0    60   ~ 0
+VSS_RTC
+Wire Wire Line
+	6125 1000 6675 1000
+Text Label 6675 1000 2    60   ~ 0
+VSS_RTC
+Wire Wire Line
+	3850 1700 4400 1700
+Wire Wire Line
+	4400 1800 3850 1800
+Text Label 8525 2100 0    60   ~ 0
+MMC0_CD
+Text Label 6675 1100 2    60   ~ 0
+MMC0_CD
+Wire Wire Line
+	6125 1100 6675 1100
+Text Label 6675 1200 2    60   ~ 0
+SYS_RESETn
+Wire Wire Line
+	6125 1200 6675 1200
+Wire Wire Line
+	4400 1000 3850 1000
 $EndSCHEMATC

Commit message: wip wl1835 lib
Parts:
- P? (x2): symbol USB_OTG -> USB_OTG-RESCUE-mateboard
- P?: symbol USB_A -> USB_A-RESCUE-mateboard
Other:
- note added: "References:\nhttp://processors.wiki.ti.com/index.php/AM335x_Hardware_Design_Guide\nhttp://processors.wiki.ti.com/index.php/AM335x_Schematic_Checklist\n"
Changed lines of the file:
@@
 EESchema Schematic File Version 2
+LIBS:mateboard-rescue
 LIBS:power
 LIBS:device
@@
 $EndSheet
 $Comp
-L USB_OTG P?
+L USB_OTG-RESCUE-mateboard P?
 U 1 1 589C9196
 P 1175 2000
@@
 $EndComp
 $Comp
-L USB_A P?
+L USB_A-RESCUE-mateboard P?
 U 1 1 589C92E9
 P 1175 3800
@@
 $EndComp
 $Comp
-L USB_OTG P?
+L USB_OTG-RESCUE-mateboard P?
 U 1 1 589C94AD
 P 1175 2900
@@
 Wire Wire Line
 	4400 1000 3850 1000
+Text Notes 575  7675 0    60   ~ 0
+References:\nhttp://processors.wiki.ti.com/index.php/AM335x_Hardware_Design_Guide\nhttp://processors.wiki.ti.com/index.php/AM335x_Schematic_Checklist\n
 $EndSCHEMATC
