File: mateboard.sch (KiCad schematic (older format))
At the start: 12 parts

Commit message: wifi bt done
Parts:
- added R?: 0R, symbol R
Connections:
- new net GPIO-I2C-SPI-UART/GPIO3_20: R?.1
- new net System/CLKOUT2: R?.2
Changed lines of the file:
@@
 LIBS:tps2065cdgn
 LIBS:74lvc1g07dck
+LIBS:wl1835modgbmoct
 LIBS:mateboard-cache
 EELAYER 25 0
@@
 F1 "io.sch" 60
 F2 "MMC0_CD" I R 8150 2850 60
+F3 "GPIO3_20" B L 6900 2850 60
 $EndSheet
 $Comp
@@
 F9 "PMIC_POWER_EN" O L 4400 1000 60
 F10 "GPIO0_7" B R 6125 1300 60
+F11 "CLKOUT2" O R 6125 2400 60
 $EndSheet
 $Sheet
@@
 Connection ~ 8950 775
 Wire Wire Line
-	8475 775  9150 775
+	8475 775  8550 775
+Wire Wire Line
+	8550 775  8650 775
+Wire Wire Line
+	8650 775  8750 775
+Wire Wire Line
+	8750 775  8850 775
+Wire Wire Line
+	8850 775  8950 775
+Wire Wire Line
+	8950 775  9050 775
+Wire Wire Line
+	9050 775  9150 775
 Wire Wire Line
 	9050 775  9050 900
@@
 	9150 1200 9150 1250
 Wire Wire Line
-	8150 1250 9225 1250
-Wire Wire Line
-	8150 1350 9225 1350
+	8150 1250 9150 1250
+Wire Wire Line
+	9150 1250 9225 1250
+Wire Wire Line
+	8150 1350 9050 1350
+Wire Wire Line
+	9050 1350 9225 1350
 Wire Wire Line
 	9050 1350 9050 1200
 Wire Wire Line
-	8150 1450 9225 1450
+	8150 1450 8950 1450
+Wire Wire Line
+	8950 1450 9225 1450
 Wire Wire Line
 	8950 1450 8950 1200
@@
 	8550 1550 8550 775
 Wire Wire Line
-	8150 1650 9225 1650
+	8150 1650 8850 1650
+Wire Wire Line
+	8850 1650 9225 1650
 Wire Wire Line
 	8850 1650 8850 1200
@@
 $EndComp
 Wire Wire Line
-	9150 1750 9150 2250
+	9150 1750 9150 2200
+Wire Wire Line
+	9150 2200 9150 2250
 Wire Wire Line
 	9150 1750 9225 1750
 Wire Wire Line
-	8150 1850 9225 1850
+	8150 1850 8750 1850
+Wire Wire Line
+	8750 1850 9225 1850
 Wire Wire Line
 	8750 1850 8750 1200
 Wire Wire Line
-	8150 1950 9225 1950
+	8150 1950 8650 1950
+Wire Wire Line
+	8650 1950 9225 1950
 Wire Wire Line
 	8650 1950 8650 1200
@@
 Connection ~ 8550 775
 Wire Wire Line
-	8475 1200 8475 2850
+	8475 1200 8475 2100
+Wire Wire Line
+	8475 2100 8475 2850
 Wire Wire Line
 	9225 2200 9150 2200
@@
 $EndComp
 Wire Wire Line
-	3850 2800 6350 2800
+	3850 2800 6375 2800
 Text Label 4400 2800 2    60   ~ 0
 USB1_OCn
 Wire Wire Line
-	6350 2400 6900 2400
+	6375 2400 6900 2400
 $Sheet
 S 6900 4550 1250 1550
@@
 F0 "Wi-Fi BLE" 60
 F1 "wifi.sch" 60
-$EndSheet
-Wire Wire Line
-	6350 2800 6350 2400
+F2 "CLKOUT2" I L 6900 4650 60
+$EndSheet
+Wire Wire Line
+	6375 2800 6375 2400
 Wire Wire Line
 	4400 2000 3850 2000
@@
 Text Notes 575  7675 0    60   ~ 0
 References:\nhttp://processors.wiki.ti.com/index.php/AM335x_Hardware_Design_Guide\nhttp://processors.wiki.ti.com/index.php/AM335x_Schematic_Checklist\n
+$Comp
+L R R?
+U 1 1 58BA190C
+P 6650 2850
+F 0 "R?" V 6730 2850 50  0000 C CNN
+F 1 "0R" V 6650 2850 50  0000 C CNN
+F 2 "" V 6580 2850 50  0001 C CNN
+F 3 "" H 6650 2850 50  0001 C CNN
+	1    6650 2850
+	0    1    1    0
+$EndComp
+Wire Wire Line
+	6800 2850 6900 2850
+Wire Wire Line
+	6500 2850 6275 2850
+Wire Wire Line
+	6275 2400 6275 2850
+Wire Wire Line
+	6275 2850 6275 4650
+Wire Wire Line
+	6275 2400 6125 2400
+Wire Wire Line
+	6275 4650 6900 4650
+Connection ~ 6275 2850
 $EndSCHEMATC
