File: mateboard.sch (KiCad schematic (older format))
At the start: 2 parts, among them J1 IO1, J2 IO2

Commit message: wip erc
Connections:
- net CLKOUT2: now also J1.16 (P16)
- net I2C0_SCL: now also J2.1 (P1)
- net I2C0_SDA: now also J2.3 (P3)
- net PWR_BUT: now also J1.6 (P6)
- net SYS_RESETn: now also J1.12 (P12)
- net VBAT: now also J1.5 (P5), J1.7 (P7)
- net VBAT_SENSE: now also J1.8 (P8)
- net VBAT_TEMP: now also J1.10 (P10)
- net VDD_5V: now reaches J1.1 (P1)
- net VDD_5V: now also J1.2 (P2), J1.3 (P3), J1.4 (P4)
- net USB_DC: now reaches J1.11 (P11)
- net USB0_DM: now reaches J1.13 (P13)
- net CLKOUT1: now reaches J1.14 (P14)
- net USB0_DP: now reaches J1.15 (P15)
- net USB0_ID: now reaches J1.17 (P17)
- net GNDD: now reaches J1.18 (P18)
- net GNDD: now also J1.19 (P19), J1.27 (P27), J1.36 (P36), J1.46 (P46), J1.69 (P69), J1.70 (P70), J1.9 (P9), J2.10 (P10), J2.11 (P11), J2.17 (P17), J2.18 (P18), J2.27 (P27), J2.44 (P44), J2.5 (P5), J2.61 (P61), J2.63 (P63), J2.69 (P69), J2.70 (P70)
- net SD_BOOT: now reaches J1.20 (P20)
- net USB1_VBUS: now reaches J1.21 (P21)
- net SD.CD: now reaches J1.22 (P22)
- net USB1_DM: now reaches J1.23 (P23)
- net SD.CLK: now reaches J1.24 (P24)
- net USB1_DP: now reaches J1.25 (P25)
- net SD.CMD: now reaches J1.26 (P26)
- net SD.D3: now reaches J1.28 (P28)
- net UART0_RXD: now reaches J1.29 (P29)
- net SD.D2: now reaches J1.30 (P30)
- net UART0_TXD: now reaches J1.31 (P31)
- net SD.D1: now reaches J1.32 (P32)
- net UART1_RXD: now reaches J1.33 (P33)
- net SD.D0: now reaches J1.34 (P34)
- net UART1_TXD: now reaches J1.35 (P35)
- net UART2_TXD: now reaches J1.37 (P37)
- net USR0: now reaches J1.38 (P38)
- net UART2_RXD: now reaches J1.39 (P39)
- net USR1: now reaches J1.40 (P40)
- net UART4_TXD: now reaches J1.41 (P41)
- net USR2: now reaches J1.42 (P42)
- net UART4_RXD: now reaches J1.43 (P43)
- net USR3: now reaches J1.44 (P44)
- net GPIO2_0: now reaches J1.45 (P45)
- net GPIO1_25: now reaches J1.47 (P47)
- net JTAG_EMU1: now reaches J1.48 (P48)
- net GPIO1_29: now reaches J1.49 (P49)
- net JTAG_EMU0: now reaches J1.50 (P50)
- net GPIO1_16: now reaches J1.51 (P51)
- net JTAG_TDO: now reaches J1.52 (P52)
- net GPIO1_15: now reaches J1.53 (P53)
- net JTAG_TCK: now reaches J1.54 (P54)
- net GPIO1_13: now reaches J1.55 (P55)
- net JTAG_TDI: now reaches J1.56 (P56)
- net GPIO1_14: now reaches J1.57 (P57)
- net JTAG_TMS: now reaches J1.58 (P58)
- net GPIO1_12: now reaches J1.59 (P59)
- net JTAG_TRSTn: now reaches J1.60 (P60)
- net GPIO0_27: now reaches J1.61 (P61)
- net TIMER4: now reaches J1.62 (P62)
- net GPIO0_26: now reaches J1.63 (P63)
- net TIMER5: now reaches J1.64 (P64)
- net GPIO2_1: now reaches J1.65 (P65)
- net TIMER6: now reaches J1.66 (P66)
- net GPIO1_28: now reaches J1.67 (P67)
- net TIMER7: now reaches J1.68 (P68)
- net GPIO0_7: now reaches J2.12 (P12)
- net I2C2_SCL: now reaches J2.13 (P13)
- net GPIO3_21: now reaches J2.14 (P14)
- net I2C2_SDA: now reaches J2.15 (P15)
- net GPIO3_19: now reaches J2.16 (P16)
- net LCD_DE: now reaches J2.19 (P19)
- net eHRPWM2B: now reaches J2.2 (P2)
- net GNDA: now reaches J2.20 (P20)
- net GNDA: now also J2.30 (P30), J2.40 (P40)
- net LCD_PCLK: now reaches J2.21 (P21)
- net AIN0: now reaches J2.22 (P22)
- net LCD_VSYNC: now reaches J2.23 (P23)
- net AIN1: now reaches J2.24 (P24)
- net LCD_HSYNC: now reaches J2.25 (P25)
- net AIN2: now reaches J2.26 (P26)
- net AIN3: now reaches J2.28 (P28)
- net LCD_DATA0: now reaches J2.29 (P29)
- net LCD_DATA1: now reaches J2.31 (P31)
- net AIN4: now reaches J2.32 (P32)
- net LCD_DATA2: now reaches J2.33 (P33)
- net AIN5: now reaches J2.34 (P34)
- net LCD_DATA3: now reaches J2.35 (P35)
- net AIN6: now reaches J2.36 (P36)
- net LCD_DATA4: now reaches J2.37 (P37)
- net AIN7: now reaches J2.38 (P38)
- net LCD_DATA5: now reaches J2.39 (P39)
- net eHRPWM2A: now reaches J2.4 (P4)
- net LCD_DATA6: now reaches J2.41 (P41)
- net VDD_ADC: now reaches J2.42 (P42)
- net LCD_DATA7: now reaches J2.43 (P43)
- net LCD_DATA8: now reaches J2.45 (P45)
- net SPI1_CLK: now reaches J2.46 (P46)
- net LCD_DATA9: now reaches J2.47 (P47)
- net SPI1_D0: now reaches J2.48 (P48)
- net LCD_DATA10: now reaches J2.49 (P49)
- net SPI1_D1: now reaches J2.50 (P50)
- net LCD_DATA11: now reaches J2.51 (P51)
- net SPI1_CS0: now reaches J2.52 (P52)
- net LCD_DATA12: now reaches J2.53 (P53)
- net LCD_DATA13: now reaches J2.55 (P55)
- net LCD_DATA14: now reaches J2.57 (P57)
- net LCD_DATA15: now reaches J2.59 (P59)
- net eHRPWM1B: now reaches J2.6 (P6)
- net VDD_3V3B: now reaches J2.65 (P65)
- net VDD_3V3B: now also J2.67 (P67)
- net SYS_5V: now reaches J2.66 (P66)
- net SYS_5V: now also J2.68 (P68)
- net I2C1_SDA: now reaches J2.7 (P7)
- net eHRPWM1A: now reaches J2.8 (P8)
- net I2C1_SCL: now reaches J2.9 (P9)
- no-connect marks 0 -> 6
Other:
- moved on the sheet: J1, J2

Commit message: erc passed
Connections:
- net AIN1: now also J2.26 (P26); no longer J2.24 (P24)
- net AIN2: now also J2.30 (P30); no longer J2.26 (P26)
- net AIN3: now also J2.34 (P34); no longer J2.28 (P28)
- net AIN4: now also J2.38 (P38); no longer J2.32 (P32)
- net AIN5: now also J2.42 (P42); no longer J2.34 (P34)
- net AIN6: now also J2.46 (P46); no longer J2.36 (P36)
- net AIN7: now also J2.50 (P50); no longer J2.38 (P38)
- net GNDA: now also J2.24 (P24), J2.28 (P28), J2.32 (P32), J2.36 (P36), J2.44 (P44), J2.48 (P48), J2.52 (P52); no longer J2.30 (P30)
- net GNDD: now also J2.56 (P56); no longer J2.44 (P44)
- net SPI1_CLK: now also J2.58 (P58); no longer J2.46 (P46)
- net SPI1_CS0: now also J2.64 (P64); no longer J2.52 (P52)
- net SPI1_D0: now also J2.60 (P60); no longer J2.48 (P48)
- net SPI1_D1: now also J2.62 (P62); no longer J2.50 (P50)
- net VDD_ADC: now also J2.54 (P54); no longer J2.42 (P42)
- no-connect marks 6 -> 0
