File: cpu_power.sch (KiCad schematic (older format))
At the start: 81 parts

Commit message: emmc nand and micro sd
Changed lines of the file:
@@
 LIBS:tl1963adcqr
 LIBS:ddr3_sdram
+LIBS:nand_4gb
+LIBS:microsd
 LIBS:mateboard-cache
 EELAYER 25 0
@@
 $Descr A4 11693 8268
 encoding utf-8
-Sheet 5 6
+Sheet 5 8
 Title ""
 Date ""
@@
 	4700 3500 4700 3400
 Wire Wire Line
-	4800 3400 4700 3400
+	4700 3400 4800 3400
 Wire Wire Line
 	4800 3200 4800 3500
@@
 	8850 3500 8850 3400
 Wire Wire Line
-	8950 3400 8850 3400
+	8850 3400 8950 3400
 Wire Wire Line
 	8950 1825 8950 3500

Commit message: system sheet
Connections:
- net VSS_RTC: now reaches IC?.A5 (xVSS_RTC), R?.1
Changed lines of the file:
@@
 LIBS:tpd4s012
 LIBS:tps2065cdgn
+LIBS:74lvc1g07dck
 LIBS:mateboard-cache
 EELAYER 25 0
@@
 Connection ~ 7950 5950
 Connection ~ 7350 6325
+Text HLabel 7150 6300 0    60   BiDi ~ 0
+VSS_RTC
+Wire Wire Line
+	7150 6300 7250 6300
+Wire Wire Line
+	7250 6300 7250 5950
+Wire Wire Line
+	7250 5950 7350 5950
+Connection ~ 7350 5950
 $EndSCHEMATC
