File: cpu_power.sch (KiCad schematic (older format))
At the start: 6 parts, among them IC1 OSD335x, J15 VDDS_PLL, J16 VDDS_DDR, J17 VDD_MPU, J18 VDD_CORE

Commit message: sch updated
Signed-off-by: Pablo Ridolfi <pabloridolfi@outlook.com>
Parts:
- added J20: VDD_RTC, Measurement_Points:Measurement_Point_Round-SMD-Pad_Small, symbol TEST_1P
Connections:
- net VRTC: no longer names the net of IC1.N6 (VDD_RTC4)
- net VRTC: now also J20.1
Other:
- moved on the sheet: R30
Changed lines of the file:
@@
 LIBS:osd335x
 LIBS:mateboard-cache
-EELAYER 25 0
+EELAYER 26 0
 EELAYER END
 $Descr A4 11693 8268
 encoding utf-8
 Sheet 4 6
-Title ""
-Date ""
-Rev ""
-Comp ""
-Comment1 ""
-Comment2 ""
-Comment3 ""
+Title "Mateboard"
+Date "2017-06-21"
+Rev "1.00"
+Comp "DPLab@UTN-FRBA"
+Comment1 "Director: Alejandro Furfaro"
+Comment2 "Revisor: Nicolás Dassieu Blanchet"
+Comment3 "Autor: Pablo Ridolfi"
 Comment4 ""
 $EndDescr
@@
 	6900 5000 7000 5000
 $Comp
-L GNDD #PWR094
+L GNDD #PWR092
 U 1 1 58E11DA7
 P 6900 5100
-F 0 "#PWR094" H 6900 4850 50  0001 C CNN
+F 0 "#PWR092" H 6900 4850 50  0001 C CNN
 F 1 "GNDD" H 6900 4950 50  0000 C CNN
 F 2 "" H 6900 5100 50  0001 C CNN
@@
 	10300 5000 10200 5000
 $Comp
-L GNDD #PWR095
+L GNDD #PWR093
 U 1 1 58E11EBE
 P 10300 5100
-F 0 "#PWR095" H 10300 4850 50  0001 C CNN
+F 0 "#PWR093" H 10300 4850 50  0001 C CNN
 F 1 "GNDD" H 10300 4950 50  0000 C CNN
 F 2 "" H 10300 5100 50  0001 C CNN
@@
 Connection ~ 7900 5600
 Wire Wire Line
-	8000 5500 8000 5600
+	8000 5600 8000 5500
 Connection ~ 8000 5600
 Wire Wire Line
-	8100 5500 8100 5600
+	8100 5600 8100 5500
 Connection ~ 8100 5600
 Wire Wire Line
-	8200 5500 8200 5600
+	8200 5600 8200 5500
 Connection ~ 8200 5600
 Wire Wire Line
-	8300 5500 8300 5600
+	8300 5600 8300 5500
 Connection ~ 8300 5600
 Wire Wire Line
-	8400 5500 8400 5600
+	8400 5600 8400 5500
 Connection ~ 8400 5600
 Wire Wire Line
-	8500 5500 8500 5600
+	8500 5600 8500 5500
 Connection ~ 8500 5600
 Wire Wire Line
-	8600 5500 8600 5600
+	8600 5600 8600 5500
 Connection ~ 8600 5600
 Wire Wire Line
-	8700 5500 8700 5600
+	8700 5600 8700 5500
 Connection ~ 8700 5600
 Wire Wire Line
-	8900 5500 8900 5600
+	8900 5600 8900 5500
 Connection ~ 8900 5600
 Wire Wire Line
-	9000 5500 9000 5600
+	9000 5600 9000 5500
 Connection ~ 9000 5600
 Wire Wire Line
-	9100 5500 9100 5600
+	9100 5600 9100 5500
 Connection ~ 9100 5600
 Wire Wire Line
-	9200 5500 9200 5600
+	9200 5600 9200 5500
 Connection ~ 9200 5600
 Wire Wire Line
-	9300 5500 9300 5600
+	9300 5600 9300 5500
 Connection ~ 9300 5600
 Wire Wire Line
-	9400 5500 9400 5600
+	9400 5600 9400 5500
 Connection ~ 9400 5600
 Wire Wire Line
@@
 	7800 5500 7800 5650
 $Comp
-L GNDD #PWR096
+L GNDD #PWR094
 U 1 1 58E12353
 P 7800 5650
-F 0 "#PWR096" H 7800 5400 50  0001 C CNN
+F 0 "#PWR094" H 7800 5400 50  0001 C CNN
 F 1 "GNDD" H 7800 5500 50  0000 C CNN
 F 2 "" H 7800 5650 50  0001 C CNN
@@
 Connection ~ 7800 5600
 $Comp
-L GNDA #PWR097
+L GNDA #PWR095
 U 1 1 58E12456
 P 9700 5600
-F 0 "#PWR097" H 9700 5350 50  0001 C CNN
+F 0 "#PWR095" H 9700 5350 50  0001 C CNN
 F 1 "GNDA" H 9700 5450 50  0000 C CNN
 F 2 "" H 9700 5600 50  0001 C CNN
@@
 Connection ~ 1600 2950
 $Comp
-L VDD_3V3A #PWR098
+L VDD_3V3A #PWR096
 U 1 1 58E148B3
 P 1400 2850
-F 0 "#PWR098" H 1400 2700 50  0001 C CNN
+F 0 "#PWR096" H 1400 2700 50  0001 C CNN
 F 1 "VDD_3V3A" V 1400 3150 50  0000 C CNN
 F 2 "" H 1400 2850 50  0000 C CNN
@@
 	1550 3750 1700 3750
 $Comp
-L VDD_ADC #PWR099
+L VDD_ADC #PWR097
 U 1 1 58E14B9C
 P 1400 5050
-F 0 "#PWR099" H 1400 4900 50  0001 C CNN
+F 0 "#PWR097" H 1400 4900 50  0001 C CNN
 F 1 "VDD_ADC" V 1400 5325 50  0000 C CNN
 F 2 "" H 1400 5050 50  0000 C CNN
@@
 NoConn ~ 4700 3650
 Wire Wire Line
-	4850 4650 4700 4650
+	4700 4650 4950 4650
 $Comp
 L R R30
 U 1 1 58E1536B
-P 5350 4350
-F 0 "R30" V 5430 4350 50  0000 C CNN
-F 1 "10k 1%" V 5275 4350 50  0000 C CNN
-F 2 "Resistors_SMD:R_0402" V 5280 4350 50  0001 C CNN
-F 3 "" H 5350 4350 50  0001 C CNN
-	1    5350 4350
-	1    0    0    -1
-$EndComp
-$Comp
-L GNDD #PWR0100
+P 5750 4350
+F 0 "R30" V 5830 4350 50  0000 C CNN
+F 1 "10k 1%" V 5675 4350 50  0000 C CNN
+F 2 "Resistors_SMD:R_0402" V 5680 4350 50  0001 C CNN
+F 3 "" H 5750 4350 50  0001 C CNN
+	1    5750 4350
+	1    0    0    -1
+$EndComp
+$Comp
+L GNDD #PWR098
 U 1 1 58E153CC
-P 5350 4500
-F 0 "#PWR0100" H 5350 4250 50  0001 C CNN
-F 1 "GNDD" H 5350 4350 50  0000 C CNN
-F 2 "" H 5350 4500 50  0001 C CNN
-F 3 "" H 5350 4500 50  0001 C CNN
-	1    5350 4500
-	1    0    0    -1
-$EndComp
-Wire Wire Line
-	5350 4200 5350 4150
-Wire Wire Line
-	5350 4150 4700 4150
+P 5750 4500
+F 0 "#PWR098" H 5750 4250 50  0001 C CNN
+F 1 "GNDD" H 5750 4350 50  0000 C CNN
+F 2 "" H 5750 4500 50  0001 C CNN
+F 3 "" H 5750 4500 50  0001 C CNN
+	1    5750 4500
+	1    0    0    -1
+$EndComp
+Wire Wire Line
+	5750 4200 5750 4150
+Wire Wire Line
+	5750 4150 4700 4150
 NoConn ~ 1700 1550
 NoConn ~ 1700 1650
@@
 NoConn ~ 4700 5850
 $Comp
-L VDD_1V8 #PWR0101
+L VDD_1V8 #PWR099
 U 1 1 58E16271
 P 4850 3950
-F 0 "#PWR0101" H 4850 3800 50  0001 C CNN
+F 0 "#PWR099" H 4850 3800 50  0001 C CNN
 F 1 "VDD_1V8" V 4850 4225 50  0000 C CNN
 F 2 "" H 4850 3950 50  0000 C CNN
@@
 Connection ~ 4800 3950
 $Comp
-L PWR_FLAG #FLG0102
+L PWR_FLAG #FLG0100
 U 1 1 58DCC8EE
 P 9700 5550
-F 0 "#FLG0102" H 9700 5625 50  0001 C CNN
+F 0 "#FLG0100" H 9700 5625 50  0001 C CNN
 F 1 "PWR_FLAG" H 9700 5700 50  0001 C CNN
 F 2 "" H 9700 5550 50  0001 C CNN
@@
 $EndComp
 $Comp
-L PWR_FLAG #FLG0103
+L PWR_FLAG #FLG0101
 U 1 1 58DD740C
 P 1600 2850
-F 0 "#FLG0103" H 1600 2925 50  0001 C CNN
+F 0 "#FLG0101" H 1600 2925 50  0001 C CNN
 F 1 "PWR_FLAG" H 1600 3000 50  0001 C CNN
 F 2 "" H 1600 2850 50  0001 C CNN
@@
 $EndComp
 $Comp
-L PWR_FLAG #FLG0104
+L PWR_FLAG #FLG0102
 U 1 1 58DD798F
 P 7800 5600
-F 0 "#FLG0104" H 7800 5675 50  0001 C CNN
+F 0 "#FLG0102" H 7800 5675 50  0001 C CNN
 F 1 "PWR_FLAG" H 7800 5750 50  0001 C CNN
 F 2 "" H 7800 5600 50  0001 C CNN
@@
 $EndComp
 $Comp
-L VRTC #PWR0105
-U 1 1 58E1525D
-P 4850 4650
-F 0 "#PWR0105" H 4850 4500 50  0001 C CNN
-F 1 "VRTC" V 4850 4850 50  0000 C CNN
-F 2 "" H 4850 4650 50  0000 C CNN
-F 3 "" H 4850 4650 50  0000 C CNN
-	1    4850 4650
-	0    1    1    0
-$EndComp
-$Comp
 L TEST_1P J18
 U 1 1 58DDEA58
@@
 	0    1    1    0
 $EndComp
+$Comp
+L TEST_1P J20
+U 1 1 5924D28B
+P 4950 4650
+F 0 "J20" V 4900 4700 50  0000 C CNN
+F 1 "VDD_RTC" V 4950 4975 50  0000 C CNN
+F 2 "Measurement_Points:Measurement_Point_Round-SMD-Pad_Small" H 5150 4650 50  0001 C CNN
+F 3 "" H 5150 4650 50  0001 C CNN
+	1    4950 4650
+	0    1    1    0
+$EndComp

Commit message: sch updated
Signed-off-by: Pablo Ridolfi <pabloridolfi@outlook.com>
Parts:
- removed IC1: OSD335x, footprints:OSD3358-BAS-BGA400, symbol OSD335x-RESCUE-mateboard
- added IC1: OSD335x, GHI-SoMs-Processors_OSD3358, symbol OSD335x
Connections:
- net GNDA: now also IC1.E8 (AGND)
- net GNDD: now also IC1.A1 (DGND1), IC1.A18 (DGND2), IC1.E19 (DGND3), IC1.E20 (DGND4), IC1.F19 (DGND6), IC1.F8 (DGND5), IC1.G11 (DGND9), IC1.G12 (DGND10), IC1.G19 (DGND11), IC1.G8 (DGND7), IC1.G9 (DGND8), IC1.H10 (DGND16), IC1.H12 (DGND17), IC1.H19 (DGND18), IC1.H6 (DGND12), IC1.H7 (DGND13), IC1.H8 (DGND14), IC1.H9 (DGND15), IC1.J10 (DGND23), IC1.J11 (DGND24), IC1.J19 (DGND25), IC1.J20 (DGND26), IC1.J6 (DGND19), IC1.J7 (DGND20), IC1.J8 (DGND21), IC1.J9 (DGND22), IC1.K10 (DGND29), IC1.K11 (DGND30), IC1.K19 (DGND31), IC1.K7 (DGND27), IC1.K9 (DGND28), IC1.L10 (DGND32), IC1.L11 (DGND33), IC1.L12 (DGND34), IC1.L13 (DGND35), IC1.L19 (DGND36), IC1.M10 (DGND42), IC1.M12 (DGND43), IC1.M14 (DGND44), IC1.M19 (DGND45), IC1.M6 (DGND38), IC1.M7 (DGND39), IC1.M8 (DGND40), IC1.M9 (DGND41), IC1.N10 (DGND47), IC1.N11 (DGND48), IC1.N14 (DGND49), IC1.N19 (DGND50), IC1.N20 (DGND51), IC1.N7 (DGND46), IC1.P19 (DGND52), IC1.P20 (DGND53), IC1.R19 (DGND54), IC1.R20 (DGND55), IC1.T19 (DGND56), IC1.T20 (DGND57), IC1.U19 (DGND58), IC1.V1 (DGND59), IC1.V18 (DGND60), IC1.V19 (DGND61), IC1.W10 (DGND70), IC1.W11 (DGND71), IC1.W12 (DGND72), IC1.W13 (DGND73), IC1.W14 (DGND74), IC1.W15 (DGND75), IC1.W16 (DGND76), IC1.W17 (DGND77), IC1.W18 (DGND78), IC1.W19 (DGND79), IC1.W2 (DGND62), IC1.W20 (DGND80), IC1.W3 (DGND63), IC1.W5 (DGND65), IC1.W6 (DGND66), IC1.W7 (DGND67), IC1.W8 (DGND68), IC1.W9 (DGND69), IC1.Y10 (DGND83), IC1.Y12 (DGND84), IC1.Y15 (DGND85), IC1.Y18 (DGND86), IC1.Y7 (DGND82)
- net VDD_1V8: now also IC1.D10 (VDD_1V84), IC1.E9 (VDD_1V83)
- net VDD_3V3A: now also IC1.N5 (VDD_3V3A18), IC1.P5 (VDD_3V3A17), IC1.P6 (VDD_3V3A16), IC1.P7 (VDD_3V3A15)
- net VDD_ADC: now also IC1.D8 (VDDA_ADC)
- net at J15.1: now also IC1.E7 (VDD_PLL1)
- net at J16.1: now also IC1.H5 (VDDS_DDR4)
- net at J17.1: now also IC1.F10 (VDD_MPU0)
- net at J18.1: now also IC1.F6 (VDD_CORE1)
- net at R30.1: now also IC1.B4 (RTC_KALDO_ENN)
- net VDD_RTC: now reaches J20.1
- net VDD_RTC: now also IC1.N6 (VDD_RTC4)
Other:
- moved on the sheet: J20, R30
Changed lines of the file:
@@
 Comment4 ""
 $EndDescr
-$Comp
-L OSD335x-RESCUE-mateboard IC1
-U 5 1 58DDF956
-P 3200 3550
-AR Path="/58DDF956" Ref="IC1"  Part="5"
-AR Path="/589E2993/58DDF956" Ref="IC1"  Part="5"
-F 0 "IC1" H 3125 3575 45  0000 L BNN
-F 1 "OSD335x" H 3050 3475 45  0000 L BNN
-F 2 "footprints:OSD3358-BAS-BGA400" H 3230 3700 20  0001 C CNN
-F 3 "" H 3200 3550 60  0001 C CNN
-	5    3200 3550
-	1    0    0    -1
-$EndComp
-$Comp
-L OSD335x-RESCUE-mateboard IC1
-U 6 1 58DDF9B7
-P 8600 3700
-AR Path="/58DDF9B7" Ref="IC1"  Part="6"
-AR Path="/589E2993/58DDF9B7" Ref="IC1"  Part="6"
-F 0 "IC1" H 8525 3725 45  0000 L BNN
-F 1 "OSD335x" H 8450 3625 45  0000 L BNN
-F 2 "footprints:OSD3358-BAS-BGA400" H 8630 3850 20  0001 C CNN
-F 3 "" H 8600 3700 60  0001 C CNN
-	6    8600 3700
-	1    0    0    -1
-$EndComp
 Wire Wire Line
 	7000 2500 6900 2500
@@
 	10300 4900 10200 4900
 Wire Wire Line
-	10300 5000 10200 5000
+	10200 5000 10350 5000
 $Comp
 L GNDD #PWR093
@@
 NoConn ~ 4700 3650
 Wire Wire Line
-	4700 4650 4950 4650
+	4700 4650 5325 4650
 $Comp
 L R R30
 U 1 1 58E1536B
-P 5750 4350
-F 0 "R30" V 5830 4350 50  0000 C CNN
-F 1 "10k 1%" V 5675 4350 50  0000 C CNN
-F 2 "Resistors_SMD:R_0402" V 5680 4350 50  0001 C CNN
-F 3 "" H 5750 4350 50  0001 C CNN
-	1    5750 4350
+P 6275 4350
+F 0 "R30" V 6355 4350 50  0000 C CNN
+F 1 "10k 1%" V 6200 4350 50  0000 C CNN
+F 2 "Resistors_SMD:R_0402" V 6205 4350 50  0001 C CNN
+F 3 "" H 6275 4350 50  0001 C CNN
+	1    6275 4350
 	1    0    0    -1
 $EndComp
@@
 L GNDD #PWR098
 U 1 1 58E153CC
-P 5750 4500
-F 0 "#PWR098" H 5750 4250 50  0001 C CNN
-F 1 "GNDD" H 5750 4350 50  0000 C CNN
-F 2 "" H 5750 4500 50  0001 C CNN
-F 3 "" H 5750 4500 50  0001 C CNN
-	1    5750 4500
-	1    0    0    -1
-$EndComp
-Wire Wire Line
-	5750 4200 5750 4150
-Wire Wire Line
-	5750 4150 4700 4150
+P 6275 4500
+F 0 "#PWR098" H 6275 4250 50  0001 C CNN
+F 1 "GNDD" H 6275 4350 50  0000 C CNN
+F 2 "" H 6275 4500 50  0001 C CNN
+F 3 "" H 6275 4500 50  0001 C CNN
+	1    6275 4500
+	1    0    0    -1
+$EndComp
+Wire Wire Line
+	6275 4200 6275 4150
+Wire Wire Line
+	6275 4150 4700 4150
 NoConn ~ 1700 1550
 NoConn ~ 1700 1650
@@
 Connection ~ 4800 3950
 $Comp
-L PWR_FLAG #FLG0100
-U 1 1 58DCC8EE
-P 9700 5550
-F 0 "#FLG0100" H 9700 5625 50  0001 C CNN
-F 1 "PWR_FLAG" H 9700 5700 50  0001 C CNN
-F 2 "" H 9700 5550 50  0001 C CNN
-F 3 "" H 9700 5550 50  0001 C CNN
-	1    9700 5550
-	0    1    1    0
-$EndComp
-Connection ~ 9700 5550
-$Comp
 L TEST_1P J15
 U 1 1 58DD0E89
@@
 $EndComp
 $Comp
-L PWR_FLAG #FLG0101
+L PWR_FLAG #FLG0100
 U 1 1 58DD740C
 P 1600 2850
-F 0 "#FLG0101" H 1600 2925 50  0001 C CNN
+F 0 "#FLG0100" H 1600 2925 50  0001 C CNN
 F 1 "PWR_FLAG" H 1600 3000 50  0001 C CNN
 F 2 "" H 1600 2850 50  0001 C CNN
@@
 	1    1600 2850
 	1    0    0    -1
-$EndComp
-$Comp
-L PWR_FLAG #FLG0102
-U 1 1 58DD798F
-P 7800 5600
-F 0 "#FLG0102" H 7800 5675 50  0001 C CNN
-F 1 "PWR_FLAG" H 7800 5750 50  0001 C CNN
-F 2 "" H 7800 5600 50  0001 C CNN
-F 3 "" H 7800 5600 50  0001 C CNN
-	1    7800 5600
-	0    -1   -1   0
 $EndComp
 $Comp
@@
 L TEST_1P J20
 U 1 1 5924D28B
-P 4950 4650
-F 0 "J20" V 4900 4700 50  0000 C CNN
-F 1 "VDD_RTC" V 4950 4975 50  0000 C CNN
-F 2 "Measurement_Points:Measurement_Point_Round-SMD-Pad_Small" H 5150 4650 50  0001 C CNN
-F 3 "" H 5150 4650 50  0001 C CNN
-	1    4950 4650
+P 5325 4650
+F 0 "J20" V 5275 4700 50  0000 C CNN
+F 1 "VDD_RTC" V 5325 4975 50  0000 C CNN
+F 2 "Measurement_Points:Measurement_Point_Round-SMD-Pad_Small" H 5525 4650 50  0001 C CNN
+F 3 "" H 5525 4650 50  0001 C CNN
+	1    5325 4650
 	0    1    1    0
 $EndComp
+Text Label 4850 4650 0    60   ~ 0
+VDD_RTC
+$Comp
+L OSD335x IC1
+U 5 1 594BE01D
+P 3200 3550
+AR Path="/594BE01D" Ref="IC1"  Part="5"
+AR Path="/589E2993/594BE01D" Ref="IC1"  Part="5"
+F 0 "IC1" H 3200 5904 45  0000 C CNN
+F 1 "OSD335x" H 3200 5820 45  0000 C CNN
+F 2 "GHI-SoMs-Processors_OSD3358" H 3230 3700 20  0001 C CNN
+F 3 "" H 3200 3550 60  0001 C CNN
+	5    3200 3550
+	1    0    0    -1
+$EndComp
+$Comp
+L OSD335x IC1
+U 6 1 594BE1D2
+P 8600 3700
+AR Path="/594BE1D2" Ref="IC1"  Part="6"
+AR Path="/589E2993/594BE1D2" Ref="IC1"  Part="6"
+F 0 "IC1" H 7275 5050 45  0000 C CNN
+F 1 "OSD335x" H 7575 5050 45  0000 C CNN
+F 2 "GHI-SoMs-Processors_OSD3358" H 8630 3850 20  0001 C CNN
+F 3 "" H 8600 3700 60  0001 C CNN
+	6    8600 3700
+	1    0    0    -1
+$EndComp
+$Comp
+L PWR_FLAG #FLG0101
+U 1 1 594D55BF
+P 9750 5550
+F 0 "#FLG0101" H 9750 5625 50  0001 C CNN
+F 1 "PWR_FLAG" H 9750 5700 50  0001 C CNN
+F 2 "" H 9750 5550 50  0001 C CNN
+F 3 "" H 9750 5550 50  0001 C CNN
+	1    9750 5550
+	0    1    1    0
+$EndComp
+Wire Wire Line
+	9750 5550 9700 5550
+Connection ~ 9700 5550
+$Comp
+L PWR_FLAG #FLG0102
+U 1 1 594D6177
+P 10350 5000
+F 0 "#FLG0102" H 10350 5075 50  0001 C CNN
+F 1 "PWR_FLAG" H 10350 5150 50  0001 C CNN
+F 2 "" H 10350 5000 50  0001 C CNN
+F 3 "" H 10350 5000 50  0001 C CNN
+	1    10350 5000
+	0    1    1    0
+$EndComp

Commit message: footprints updated, add power led
Signed-off-by: Pablo Ridolfi <pabloridolfi@outlook.com>
Parts:
- IC1: footprint GHI-SoMs-Processors_OSD3358 -> footprints:OSD3358-BAS-BGA400
Changed lines of the file:
@@
 F 0 "IC1" H 3200 5904 45  0000 C CNN
 F 1 "OSD335x" H 3200 5820 45  0000 C CNN
-F 2 "GHI-SoMs-Processors_OSD3358" H 3230 3700 20  0001 C CNN
+F 2 "footprints:OSD3358-BAS-BGA400" H 3230 3700 20  0001 C CNN
 F 3 "" H 3200 3550 60  0001 C CNN
 	5    3200 3550
@@
 F 0 "IC1" H 7275 5050 45  0000 C CNN
 F 1 "OSD335x" H 7575 5050 45  0000 C CNN
-F 2 "GHI-SoMs-Processors_OSD3358" H 8630 3850 20  0001 C CNN
+F 2 "footprints:OSD3358-BAS-BGA400" H 8630 3850 20  0001 C CNN
 F 3 "" H 8600 3700 60  0001 C CNN
 	6    8600 3700

Commit message: gerbers updated, bom using kicost
Signed-off-by: Pablo Ridolfi <pabloridolfi@outlook.com>
Parts:
- R30: manf# (none) -> RC0402FR-0710KL
Changed lines of the file:
@@
 	6900 5000 7000 5000
 $Comp
-L GNDD #PWR92
+L GNDD #PWR092
 U 1 1 58E11DA7
 P 6900 5100
-F 0 "#PWR92" H 6900 4850 50  0001 C CNN
+F 0 "#PWR092" H 6900 4850 50  0001 C CNN
 F 1 "GNDD" H 6900 4950 50  0000 C CNN
 F 2 "" H 6900 5100 50  0001 C CNN
@@
 	10200 5000 10350 5000
 $Comp
-L GNDD #PWR95
+L GNDD #PWR095
 U 1 1 58E11EBE
 P 10300 5100
-F 0 "#PWR95" H 10300 4850 50  0001 C CNN
+F 0 "#PWR095" H 10300 4850 50  0001 C CNN
 F 1 "GNDD" H 10300 4950 50  0000 C CNN
 F 2 "" H 10300 5100 50  0001 C CNN
@@
 	7800 5500 7800 5650
 $Comp
-L GNDD #PWR93
+L GNDD #PWR093
 U 1 1 58E12353
 P 7800 5650
-F 0 "#PWR93" H 7800 5400 50  0001 C CNN
+F 0 "#PWR093" H 7800 5400 50  0001 C CNN
 F 1 "GNDD" H 7800 5500 50  0000 C CNN
 F 2 "" H 7800 5650 50  0001 C CNN
@@
 Connection ~ 7800 5600
 $Comp
-L GNDA #PWR94
+L GNDA #PWR094
 U 1 1 58E12456
 P 9700 5600
-F 0 "#PWR94" H 9700 5350 50  0001 C CNN
+F 0 "#PWR094" H 9700 5350 50  0001 C CNN
 F 1 "GNDA" H 9700 5450 50  0000 C CNN
 F 2 "" H 9700 5600 50  0001 C CNN
@@
 Connection ~ 1600 2950
 $Comp
-L VDD_3V3A #PWR88
+L VDD_3V3A #PWR088
 U 1 1 58E148B3
 P 1400 2850
-F 0 "#PWR88" H 1400 2700 50  0001 C CNN
+F 0 "#PWR088" H 1400 2700 50  0001 C CNN
 F 1 "VDD_3V3A" V 1400 3150 50  0000 C CNN
 F 2 "" H 1400 2850 50  0000 C CNN
@@
 	1550 3750 1700 3750
 $Comp
-L VDD_ADC #PWR89
+L VDD_ADC #PWR089
 U 1 1 58E14B9C
 P 1400 5050
-F 0 "#PWR89" H 1400 4900 50  0001 C CNN
+F 0 "#PWR089" H 1400 4900 50  0001 C CNN
 F 1 "VDD_ADC" V 1400 5325 50  0000 C CNN
 F 2 "" H 1400 5050 50  0000 C CNN
@@
 F 2 "Resistors_SMD:R_0402" V 6205 4350 50  0001 C CNN
 F 3 "" H 6275 4350 50  0001 C CNN
+F 4 "RC0402FR-0710KL" V 6275 4350 60  0001 C CNN "manf#"
 	1    6275 4350
 	1    0    0    -1
 $EndComp
 $Comp
-L GNDD #PWR91
+L GNDD #PWR091
 U 1 1 58E153CC
 P 6275 4500
-F 0 "#PWR91" H 6275 4250 50  0001 C CNN
+F 0 "#PWR091" H 6275 4250 50  0001 C CNN
 F 1 "GNDD" H 6275 4350 50  0000 C CNN
 F 2 "" H 6275 4500 50  0001 C CNN
@@
 NoConn ~ 4700 5850
 $Comp
-L VDD_1V8 #PWR90
+L VDD_1V8 #PWR090
 U 1 1 58E16271
 P 4850 3950
-F 0 "#PWR90" H 4850 3800 50  0001 C CNN
+F 0 "#PWR090" H 4850 3800 50  0001 C CNN
 F 1 "VDD_1V8" V 4850 4225 50  0000 C CNN
 F 2 "" H 4850 3950 50  0000 C CNN
@@
 $EndComp
 $Comp
-L PWR_FLAG #FLG5
+L PWR_FLAG #FLG05
 U 1 1 58DD740C
 P 1600 2850
-F 0 "#FLG5" H 1600 2925 50  0001 C CNN
+F 0 "#FLG05" H 1600 2925 50  0001 C CNN
 F 1 "PWR_FLAG" H 1600 3000 50  0001 C CNN
 F 2 "" H 1600 2850 50  0001 C CNN
@@
 $EndComp
 $Comp
-L PWR_FLAG #FLG6
+L PWR_FLAG #FLG06
 U 1 1 594D55BF
 P 9750 5550
-F 0 "#FLG6" H 9750 5625 50  0001 C CNN
+F 0 "#FLG06" H 9750 5625 50  0001 C CNN
 F 1 "PWR_FLAG" H 9750 5700 50  0001 C CNN
 F 2 "" H 9750 5550 50  0001 C CNN
@@
 Connection ~ 9700 5550
 $Comp
-L PWR_FLAG #FLG7
+L PWR_FLAG #FLG07
 U 1 1 594D6177
 P 10350 5000
-F 0 "#FLG7" H 10350 5075 50  0001 C CNN
+F 0 "#FLG07" H 10350 5075 50  0001 C CNN
 F 1 "PWR_FLAG" H 10350 5150 50  0001 C CNN
 F 2 "" H 10350 5000 50  0001 C CNN
