File: mmc.sch (KiCad schematic (older format))
At the start: 18 parts

Commit message: usb
Connections:
- net USB1_OCn: now reaches IC?.T16 (xGPMC_A10-GMII2_RXD1-RGMII2_RD1-RMII2_RXD1-GPMC_A26-PR1_MII1_RXDV-McASP0_AXR0-GPIO1_26)
Changed lines of the file:
@@
 LIBS:nand_4gb
 LIBS:microsd
+LIBS:tpd4s012
+LIBS:tps2065cdgn
 LIBS:mateboard-cache
 EELAYER 25 0
@@
 Wire Wire Line
 	5825 5175 5600 5175
+Wire Wire Line
+	5600 1700 6150 1700
+Text HLabel 6150 1700 2    60   Input ~ 0
+USB1_OCn
 $EndSCHEMATC

Commit message: wip gpio
Connections:
- net GPIO1_16: now reaches IC?.R13 (xGPMC_A0-GMII2_TXEn-RGMII2_TCTL-RMII2_TXEn-GPMC_A16-PR1_MII_MT1_CLK-eHRPWM1_TRIPZONE_INPUT-GPIO1_16)
- net eHRPWM2B: now reaches IC?.T10 (GPMC_AD9-LCD_DATA22-MMC1_DAT1-MMC2_DAT5-eHRPWM2B-PR1_MII0_COL-GPIO0_23)
- net eHRPWM1B: now reaches IC?.T14 (xGPMC_A3-GMII2_TXD2-RGMII2_TD2-MMC2_DAT2-GPMC_A19-PR1_MII1_TXD1-eHRPWM1B-GPIO1_19)
- net USR2: now reaches IC?.T15 (xGPMC_A7-GMII2_RXCLK-RGMII2_RCLK-MMC2_DAT5-GPMC_A23-PR1_MII1_RXD1-eQEP1_STROBE-GPIO1_23)
- net eHRPWM2A: now reaches IC?.U10 (GPMC_AD8-LCD_DATA23-MMC1_DAT0-MMC2_DAT4-eHRPWM2A-PR1_MII_MT0_CLK-GPIO0_22)
- net eHRPWM1A: now reaches IC?.U14 (xGPMC_A2-GMII2_TXD3-RGMII2_TD3-MMC2_DAT1-GPMC_A18-PR1_MII1_TXD2-eHRPWM1A-GPIO1_18)
- net USR1: now reaches IC?.U15 (xGPMC_A6-GMII2_TXCLK-RGMII2_TCLK-MMC2_DAT4-GPMC_A22-PR1_MII1_RXD2-eQEP1_INDEX-GPIO1_22)
- net GPIO1_25: now reaches IC?.U16 (xGPMC_A9-GMII2_RXD2-RGMII2_RD2-MMC2_DAT7-GPMC_A25-PR1_MII_MR1_CLK-McASP0_FSX-GPIO1_25)
- net GPIO1_17: now reaches IC?.V14 (xGPMC_A1-GMII2_RXDV-RGMII2_RCTL-MMC2_DAT0-GPMC_A17-PR1_MII1_TXD3-eHRPWM0_SYNCO-GPIO1_17)
- net USR0: now reaches IC?.V15 (xGPMC_A5-GMII2_TXD0-RGMII2_TD0-RMII2_TXD0-GPMC_A21-PR1_MII1_RXD3-eQEP1B_IN-GPIO1_21)
- net USR3: now reaches IC?.V16 (xGPMC_A8-GMII2_RXD3-RGMII2_RD3-MMC2_DAT6-GPMC_A24-PR1_MII1_RXD0-McASP0_ACLKX-GPIO1_24)
- net GPIO1_27: now reaches IC?.V17 (xGPMC_A11-GMII2_RXD0-RGMII2_RD0-RMII2_RXD0-GPMC_A27-PR1_MII1_RXER-McASP0_AXR1-GPIO1_27)
Changed lines of the file:
@@
 $Descr A4 11693 8268
 encoding utf-8
-Sheet 7 10
+Sheet 6 10
 Title ""
 Date ""
@@
 U 6 1 58ABE3EA
 P 600 2700
-F 0 "IC?" V 550 3000 60  0000 C CNN
-F 1 "AM335X_ZCZ" V 550 2400 60  0000 C CNN
+F 0 "IC?" H 700 4850 60  0000 C CNN
+F 1 "AM335X_ZCZ" H 1500 4850 60  0000 C CNN
 F 2 "" H 600 2700 60  0001 C CNN
 F 3 "" H 600 2700 60  0001 C CNN
@@
 AR Path="/58ACF85A" Ref="IC?"  Part="10"
 AR Path="/58ABDF44/58ACF85A" Ref="IC?"  Part="10"
-F 0 "IC?" V 1250 5625 60  0000 C CNN
-F 1 "AM335X_ZCZ" V 1250 5025 60  0000 C CNN
+F 0 "IC?" H 1400 5725 60  0000 C CNN
+F 1 "AM335X_ZCZ" H 2225 5725 60  0000 C CNN
 F 2 "" H 1300 5325 60  0001 C CNN
 F 3 "" H 1300 5325 60  0001 C CNN
@@
 Text HLabel 6150 1700 2    60   Input ~ 0
 USB1_OCn
+Text HLabel 6150 700  2    60   BiDi ~ 0
+GPIO1_16
+Wire Wire Line
+	6150 700  5600 700
+Text HLabel 6150 800  2    60   BiDi ~ 0
+GPIO1_17
+Wire Wire Line
+	6150 800  5600 800
+Wire Wire Line
+	5600 900  6150 900
+Text HLabel 6150 900  2    60   Output ~ 0
+eHRPWM1A
+Wire Wire Line
+	5600 1000 6150 1000
+Text HLabel 6150 1000 2    60   Output ~ 0
+eHRPWM1B
+Wire Wire Line
+	5600 2750 6150 2750
+Text HLabel 6150 2750 2    60   Output ~ 0
+eHRPWM2A
+Wire Wire Line
+	5600 2850 6150 2850
+Text HLabel 6150 2850 2    60   Output ~ 0
+eHRPWM2B
+Wire Wire Line
+	5600 1200 6150 1200
+Text HLabel 6150 1200 2    60   Output ~ 0
+USR0
+Wire Wire Line
+	5600 1300 6150 1300
+Text HLabel 6150 1300 2    60   Output ~ 0
+USR1
+Wire Wire Line
+	5600 1400 6150 1400
+Text HLabel 6150 1400 2    60   Output ~ 0
+USR2
+Wire Wire Line
+	5600 1500 6150 1500
+Text HLabel 6150 1500 2    60   Output ~ 0
+USR3
+Text HLabel 6150 1600 2    60   BiDi ~ 0
+GPIO1_25
+Wire Wire Line
+	6150 1600 5600 1600
+Wire Wire Line
+	5600 1800 6150 1800
+Text HLabel 6150 1800 2    60   BiDi ~ 0
+GPIO1_27
 $EndSCHEMATC

Commit message: gpio assignment done
Connections:
- net GPIO1_13: now reaches IC?.R12 (GPMC_AD13-LCD_DATA18-MMC1_DAT5-MMC2_DAT1-eQEP2B_IN-PR1_MII0_TXD1-PR1_PRU0_PRU_R30_15-GPIO1_13)
- net TIMER4: now reaches IC?.R7 (GPMC_ADVn_ALE-TIMER4-GPIO2_2)
- net GPIO0_26: now reaches IC?.T11 (GPMC_AD10-LCD_DATA21-MMC1_DAT2-MMC2_DAT6-eHRPWM2_TRIPZONE_INPUT-PR1_MII0_TXEn-GPIO0_26)
- net GPIO1_12: now reaches IC?.T12 (GPMC_AD12-LCD_DATA19-MMC1_DAT4-MMC2_DAT0-eQEP2A_IN-PR1_MII0_TXD2-PR1_PRU0_PRU_R30_14-GPIO1_12)
- net GPIO2_0: now reaches IC?.T13 (GPMC_CSn3-MMC2_CMD-PR1_MII0_CRS-PR1_MDIO_DATA-EMU4-GPIO2_0)
- net UART4_RXD: now reaches IC?.T17 (GPMC_WAIT0-GMII2_CRS-GPMC_CSN4-RMII2_CRS_DV-MMC1_SDCD-PR1_MII1_COL-UART4_RXD-GPIO0_30)
- net TIMER5: now reaches IC?.T6 (GPMC_BE0n_CLE-TIMER5-GPIO2_5)
- net TIMER7: now reaches IC?.T7 (GPMC_OEn_REn-TIMER7-GPIO2_3)
- net GPIO0_27: now reaches IC?.U12 (GPMC_AD11-LCD_DATA20-MMC1_DAT3-MMC2_DAT7-eHRPWM0_SYNCO-PR1_MII0_TXD3-GPIO0_27)
- net GPIO1_15: now reaches IC?.U13 (GPMC_AD15-LCD_DATA16-MMC1_DAT7-MMC2_DAT3-eQEP2_STROBE-PR1_eCAP0_eCAP_CAPIN_APWM_O-PR1_PRU0_PRU_R31_15-GPIO1_15)
- net UART4_TXD: now reaches IC?.U17 (GPMC_WPn-GMII2_RXERR-GPMC_CSN5-RMII2_RXERR-MMC2_SDCD-PR1_MII1_TXEn-UART4_TXD-GPIO0_31)
- net GPIO1_28: now reaches IC?.U18 (GPMC_BE1n-GMII2_COL-GPMC_CSN6-MMC2_DAT3-GPMC_DIR-PR1_MII1_RXLINK-McASP0_ACLKR-GPIO1_28)
- net TIMER6: now reaches IC?.U6 (GPMC_WEn-TIMER6-GPIO2_4)
- net GPIO2_1: now reaches IC?.V12 (GPMC_CLK-LCD_MEMORY_CLK-GPMC_WAIT1-MMC2_CLK-PR1_MII1_CRS-PR1_MDIO_MDCLK-McASP0_FSR-GPIO2_1)
- net GPIO1_14: now reaches IC?.V13 (GPMC_AD14-LCD_DATA17-MMC1_DAT6-MMC2_DAT2-eQEP2_INDEX-PR1_MII0_TXD0-PR1_PRU0_PRU_R31_14-GPIO1_14)
- net GPIO1_29: now reaches IC?.V6 (GPMC_CSn0-GPIO1_29)
Changed lines of the file:
@@
 Text HLabel 6150 1800 2    60   BiDi ~ 0
 GPIO1_27
+Wire Wire Line
+	5600 4000 6150 4000
+Text HLabel 6150 4000 2    60   Output ~ 0
+TIMER7
+Wire Wire Line
+	5600 4100 6150 4100
+Text HLabel 6150 4100 2    60   Output ~ 0
+TIMER6
+Wire Wire Line
+	5600 3600 6150 3600
+Text HLabel 6150 3600 2    60   Output ~ 0
+TIMER4
+Wire Wire Line
+	5600 3700 6150 3700
+Text HLabel 6150 3700 2    60   Output ~ 0
+TIMER5
+Wire Wire Line
+	5600 3800 6150 3800
+Text HLabel 6150 3800 2    60   BiDi ~ 0
+GPIO1_28
+Wire Wire Line
+	5600 3900 6150 3900
+Text HLabel 6150 3900 2    60   BiDi ~ 0
+GPIO2_1
+Wire Wire Line
+	5600 4200 6150 4200
+Text HLabel 6150 4200 2    60   Output ~ 0
+UART4_TXD
+Wire Wire Line
+	5600 4300 6150 4300
+Text HLabel 6150 4300 2    60   Input ~ 0
+UART4_RXD
+Wire Wire Line
+	5600 4400 6150 4400
+Text HLabel 6150 4400 2    60   BiDi ~ 0
+GPIO1_29
+Wire Wire Line
+	5600 4700 6150 4700
+Text HLabel 6150 4700 2    60   BiDi ~ 0
+GPIO2_0
+Wire Wire Line
+	5600 2950 6150 2950
+Text HLabel 6150 2950 2    60   BiDi ~ 0
+GPIO0_26
+Wire Wire Line
+	5600 3050 6150 3050
+Text HLabel 6150 3050 2    60   BiDi ~ 0
+GPIO0_27
+Wire Wire Line
+	5600 3150 6150 3150
+Text HLabel 6150 3150 2    60   BiDi ~ 0
+GPIO1_12
+Wire Wire Line
+	5600 3250 6150 3250
+Text HLabel 6150 3250 2    60   BiDi ~ 0
+GPIO1_13
+Wire Wire Line
+	5600 3350 6150 3350
+Text HLabel 6150 3350 2    60   BiDi ~ 0
+GPIO1_14
+Wire Wire Line
+	5600 3450 6150 3450
+Text HLabel 6150 3450 2    60   BiDi ~ 0
+GPIO1_15
 $EndSCHEMATC
