File: mmc.sch (KiCad schematic (older format))
At the start: 18 parts

Commit message: gpio connectors
Parts:
- IC?: footprint (none) -> footprints:WFBGA153
Changed lines of the file:
@@
 F 0 "IC?" H 8950 2225 60  0000 C CNN
 F 1 "NAND_4GB" H 9125 925 60  0000 C CNN
-F 2 "" H 8875 1625 60  0001 C CNN
+F 2 "footprints:WFBGA153" H 8875 1625 60  0001 C CNN
 F 3 "" H 8875 1625 60  0001 C CNN
 	1    8875 1625

Commit message: annotation, wip erc
Parts:
- gave numbers to parts that had none: 17
Changed lines of the file:
@@
 $EndDescr
 $Comp
-L AM335X_ZCZ IC?
+L AM335X_ZCZ IC2
 U 6 1 58ABE3EA
 P 600 2700
-F 0 "IC?" H 700 4850 60  0000 C CNN
+F 0 "IC2" H 700 4850 60  0000 C CNN
 F 1 "AM335X_ZCZ" H 1500 4850 60  0000 C CNN
 F 2 "" H 600 2700 60  0001 C CNN
@@
 $EndComp
 $Comp
-L NAND_4GB IC?
+L NAND_4GB IC4
 U 1 1 58AC77E5
 P 8875 1625
-F 0 "IC?" H 8950 2225 60  0000 C CNN
+F 0 "IC4" H 8950 2225 60  0000 C CNN
 F 1 "NAND_4GB" H 9125 925 60  0000 C CNN
 F 2 "footprints:WFBGA153" H 8875 1625 60  0001 C CNN
@@
 $EndComp
 $Comp
-L VDD_3V3B #PWR?
+L VDD_3V3B #PWR247
 U 1 1 58AC7A07
 P 9875 775
-F 0 "#PWR?" H 9875 625 50  0001 C CNN
+F 0 "#PWR247" H 9875 625 50  0001 C CNN
 F 1 "VDD_3V3B" H 9875 925 50  0000 C CNN
 F 2 "" H 9875 775 50  0000 C CNN
@@
 	9475 825  10275 825
 $Comp
-L C C?
+L C C124
 U 1 1 58AC7ACC
 P 10725 850
-F 0 "C?" H 10750 950 50  0000 L CNN
+F 0 "C124" H 10750 950 50  0000 L CNN
 F 1 "2.2uF/6.3V" H 10750 750 50  0000 L CNN
 F 2 "" H 10763 700 50  0000 C CNN
@@
 $EndComp
 $Comp
-L GNDD #PWR?
+L GNDD #PWR249
 U 1 1 58AC7B05
 P 10725 1000
-F 0 "#PWR?" H 10725 750 50  0001 C CNN
+F 0 "#PWR249" H 10725 750 50  0001 C CNN
 F 1 "GNDD" H 10725 850 50  0000 C CNN
 F 2 "" H 10725 1000 50  0000 C CNN
@@
 	10450 700  10725 700
 $Comp
-L GNDD #PWR?
+L GNDD #PWR248
 U 1 1 58AC7B50
 P 9875 2575
-F 0 "#PWR?" H 9875 2325 50  0001 C CNN
+F 0 "#PWR248" H 9875 2325 50  0001 C CNN
 F 1 "GNDD" H 9875 2425 50  0000 C CNN
 F 2 "" H 9875 2575 50  0000 C CNN
@@
 	9475 2525 10275 2525
 $Comp
-L R R?
+L R R47
 U 1 1 58AC80C4
 P 7900 950
-F 0 "R?" V 7850 1100 50  0000 C CNN
+F 0 "R47" V 7850 1100 50  0000 C CNN
 F 1 "10k" V 7900 950 50  0000 C CNN
 F 2 "" V 7830 950 50  0000 C CNN
@@
 $EndComp
 $Comp
-L R R?
+L R R49
 U 1 1 58AC81C6
 P 8000 950
-F 0 "R?" V 7950 1100 50  0000 C CNN
+F 0 "R49" V 7950 1100 50  0000 C CNN
 F 1 "10k" V 8000 950 50  0000 C CNN
 F 2 "" V 7930 950 50  0000 C CNN
@@
 $EndComp
 $Comp
-L R R?
+L R R50
 U 1 1 58AC8209
 P 8100 950
-F 0 "R?" V 8050 1100 50  0000 C CNN
+F 0 "R50" V 8050 1100 50  0000 C CNN
 F 1 "10k" V 8100 950 50  0000 C CNN
 F 2 "" V 8030 950 50  0000 C CNN
@@
 $EndComp
 $Comp
-L R R?
+L R R51
 U 1 1 58AC820F
 P 8200 950
-F 0 "R?" V 8150 1100 50  0000 C CNN
+F 0 "R51" V 8150 1100 50  0000 C CNN
 F 1 "10k" V 8200 950 50  0000 C CNN
 F 2 "" V 8130 950 50  0000 C CNN
@@
 $EndComp
 $Comp
-L R R?
+L R R43
 U 1 1 58AC82D4
 P 7500 950
-F 0 "R?" V 7450 1100 50  0000 C CNN
+F 0 "R43" V 7450 1100 50  0000 C CNN
 F 1 "10k" V 7500 950 50  0000 C CNN
 F 2 "" V 7430 950 50  0000 C CNN
@@
 $EndComp
 $Comp
-L R R?
+L R R44
 U 1 1 58AC82DA
 P 7600 950
-F 0 "R?" V 7550 1100 50  0000 C CNN
+F 0 "R44" V 7550 1100 50  0000 C CNN
 F 1 "10k" V 7600 950 50  0000 C CNN
 F 2 "" V 7530 950 50  0000 C CNN
@@
 $EndComp
 $Comp
-L R R?
+L R R45
 U 1 1 58AC82E0
 P 7700 950
-F 0 "R?" V 7650 1100 50  0000 C CNN
+F 0 "R45" V 7650 1100 50  0000 C CNN
 F 1 "10k" V 7700 950 50  0000 C CNN
 F 2 "" V 7630 950 50  0000 C CNN
@@
 $EndComp
 $Comp
-L R R?
+L R R46
 U 1 1 58AC82E6
 P 7800 950
-F 0 "R?" V 7750 1100 50  0000 C CNN
+F 0 "R46" V 7750 1100 50  0000 C CNN
 F 1 "10k" V 7800 950 50  0000 C CNN
 F 2 "" V 7730 950 50  0000 C CNN
@@
 $EndComp
 $Comp
-L R R?
+L R R40
 U 1 1 58AC833F
 P 7200 950
-F 0 "R?" V 7150 1100 50  0000 C CNN
+F 0 "R40" V 7150 1100 50  0000 C CNN
 F 1 "10k" V 7200 950 50  0000 C CNN
 F 2 "" V 7130 950 50  0000 C CNN
@@
 $EndComp
 $Comp
-L R R?
+L R R41
 U 1 1 58AC8345
 P 7300 950
-F 0 "R?" V 7250 1100 50  0000 C CNN
+F 0 "R41" V 7250 1100 50  0000 C CNN
 F 1 "10k" V 7300 950 50  0000 C CNN
 F 2 "" V 7230 950 50  0000 C CNN
@@
 $EndComp
 $Comp
-L R R?
+L R R42
 U 1 1 58AC834B
 P 7400 950
-F 0 "R?" V 7350 1100 50  0000 C CNN
+F 0 "R42" V 7350 1100 50  0000 C CNN
 F 1 "10k" V 7400 950 50  0000 C CNN
 F 2 "" V 7330 950 50  0000 C CNN
@@
 $EndComp
 $Comp
-L VDD_3V3B #PWR?
+L VDD_3V3B #PWR245
 U 1 1 58AC8663
 P 7600 675
-F 0 "#PWR?" H 7600 525 50  0001 C CNN
+F 0 "#PWR245" H 7600 525 50  0001 C CNN
 F 1 "VDD_3V3B" H 7600 825 50  0000 C CNN
 F 2 "" H 7600 675 50  0000 C CNN
@@
 	6150 4500 5600 4500
 $Comp
-L 74AHC1G14 U?
+L 74AHC1G14 U5
 U 1 1 58ACBE41
 P 7350 3000
-F 0 "U?" H 7500 2900 50  0000 C CNN
+F 0 "U5" H 7500 2900 50  0000 C CNN
 F 1 "SN74LVC1G06DCK" H 7650 2800 50  0000 C CNN
 F 2 "" H 7445 2865 50  0000 C CNN
@@
 $EndComp
 $Comp
-L R R?
+L R R48
 U 1 1 58ACC029
 P 7950 3000
-F 0 "R?" V 8030 3000 50  0000 C CNN
+F 0 "R48" V 8030 3000 50  0000 C CNN
 F 1 "0R" V 7950 3000 50  0000 C CNN
 F 2 "" V 7880 3000 50  0000 C CNN
@@
 $EndComp
 $Comp
-L VDD_3V3A #PWR?
+L VDD_3V3A #PWR243
 U 1 1 58ACC796
 P 7300 2625
-F 0 "#PWR?" H 7300 2475 50  0001 C CNN
+F 0 "#PWR243" H 7300 2475 50  0001 C CNN
 F 1 "VDD_3V3A" H 7300 2775 50  0000 C CNN
 F 2 "" H 7300 2625 50  0000 C CNN
@@
 $EndComp
 $Comp
-L GNDD #PWR?
+L GNDD #PWR244
 U 1 1 58ACC7CA
 P 7300 3200
-F 0 "#PWR?" H 7300 2950 50  0001 C CNN
+F 0 "#PWR244" H 7300 2950 50  0001 C CNN
 F 1 "GNDD" H 7300 3050 50  0000 C CNN
 F 2 "" H 7300 3200 50  0000 C CNN
@@
 $EndComp
 $Comp
-L C C?
+L C C123
 U 1 1 58ACCFD2
 P 7500 2725
-F 0 "C?" V 7325 2575 50  0000 L CNN
+F 0 "C123" V 7325 2575 50  0000 L CNN
 F 1 "100nF/6.3V" V 7400 2225 50  0000 L CNN
 F 2 "" H 7538 2575 50  0000 C CNN
@@
 $EndComp
 $Comp
-L GNDD #PWR?
+L GNDD #PWR246
 U 1 1 58ACCFD9
 P 7650 2725
-F 0 "#PWR?" H 7650 2475 50  0001 C CNN
+F 0 "#PWR246" H 7650 2475 50  0001 C CNN
 F 1 "GNDD" V 7650 2525 50  0000 C CNN
 F 2 "" H 7650 2725 50  0000 C CNN
@@
 P 1300 5325
 AR Path="/58ACF85A" Ref="IC?"  Part="10"
-AR Path="/58ABDF44/58ACF85A" Ref="IC?"  Part="10"
-F 0 "IC?" H 1400 5725 60  0000 C CNN
+AR Path="/58ABDF44/58ACF85A" Ref="IC2"  Part="10"
+F 0 "IC2" H 1400 5725 60  0000 C CNN
 F 1 "AM335X_ZCZ" H 2225 5725 60  0000 C CNN
 F 2 "" H 1300 5325 60  0001 C CNN

Commit message: erc passed, sch first version
Changed lines of the file:
@@
 $EndComp
 $Comp
-L VDD_3V3B #PWR247
+L VDD_3V3B #PWR0261
 U 1 1 58AC7A07
 P 9875 775
-F 0 "#PWR247" H 9875 625 50  0001 C CNN
+F 0 "#PWR0261" H 9875 625 50  0001 C CNN
 F 1 "VDD_3V3B" H 9875 925 50  0000 C CNN
 F 2 "" H 9875 775 50  0000 C CNN
@@
 $EndComp
 $Comp
-L GNDD #PWR249
+L GNDD #PWR0262
 U 1 1 58AC7B05
 P 10725 1000
-F 0 "#PWR249" H 10725 750 50  0001 C CNN
+F 0 "#PWR0262" H 10725 750 50  0001 C CNN
 F 1 "GNDD" H 10725 850 50  0000 C CNN
 F 2 "" H 10725 1000 50  0000 C CNN
@@
 $EndComp
 Wire Wire Line
-	10450 875  10450 700
+	10450 675  10450 875
 Wire Wire Line
 	10450 700  10725 700
 $Comp
-L GNDD #PWR248
+L GNDD #PWR0263
 U 1 1 58AC7B50
 P 9875 2575
-F 0 "#PWR248" H 9875 2325 50  0001 C CNN
+F 0 "#PWR0263" H 9875 2325 50  0001 C CNN
 F 1 "GNDD" H 9875 2425 50  0000 C CNN
 F 2 "" H 9875 2575 50  0000 C CNN
@@
 $EndComp
 $Comp
-L VDD_3V3B #PWR245
+L VDD_3V3B #PWR0264
 U 1 1 58AC8663
 P 7600 675
-F 0 "#PWR245" H 7600 525 50  0001 C CNN
+F 0 "#PWR0264" H 7600 525 50  0001 C CNN
 F 1 "VDD_3V3B" H 7600 825 50  0000 C CNN
 F 2 "" H 7600 675 50  0000 C CNN
@@
 $EndComp
 $Comp
-L VDD_3V3A #PWR243
+L VDD_3V3A #PWR0265
 U 1 1 58ACC796
 P 7300 2625
-F 0 "#PWR243" H 7300 2475 50  0001 C CNN
+F 0 "#PWR0265" H 7300 2475 50  0001 C CNN
 F 1 "VDD_3V3A" H 7300 2775 50  0000 C CNN
 F 2 "" H 7300 2625 50  0000 C CNN
@@
 $EndComp
 $Comp
-L GNDD #PWR244
+L GNDD #PWR0266
 U 1 1 58ACC7CA
 P 7300 3200
-F 0 "#PWR244" H 7300 2950 50  0001 C CNN
+F 0 "#PWR0266" H 7300 2950 50  0001 C CNN
 F 1 "GNDD" H 7300 3050 50  0000 C CNN
 F 2 "" H 7300 3200 50  0000 C CNN
@@
 $EndComp
 $Comp
-L GNDD #PWR246
+L GNDD #PWR0267
 U 1 1 58ACCFD9
 P 7650 2725
-F 0 "#PWR246" H 7650 2475 50  0001 C CNN
+F 0 "#PWR0267" H 7650 2475 50  0001 C CNN
 F 1 "GNDD" V 7650 2525 50  0000 C CNN
 F 2 "" H 7650 2725 50  0000 C CNN
@@
 Text HLabel 6150 3450 2    60   BiDi ~ 0
 GPIO1_15
+$Comp
+L PWR_FLAG #FLG0268
+U 1 1 58C83D42
+P 10450 675
+F 0 "#FLG0268" H 10450 750 50  0001 C CNN
+F 1 "PWR_FLAG" H 10450 825 50  0001 C CNN
+F 2 "" H 10450 675 50  0001 C CNN
+F 3 "" H 10450 675 50  0001 C CNN
+	1    10450 675
+	1    0    0    -1
+$EndComp
+Connection ~ 10450 700
 $EndSCHEMATC

Commit message: wip sch
Parts:
- removed unit 10 of IC2
Connections:
- net labels removed: MMC0_CLK, MMC0_CMD, MMC0_DAT0, MMC0_DAT1, MMC0_DAT2, MMC0_DAT3, eHRPWM1A, eHRPWM1B, eHRPWM2A, eHRPWM2B
- wire segments 106 -> 100
Changed lines of the file:
@@
 LIBS:74lvc1g07dck
 LIBS:wl1835modgbmoct
+LIBS:osd335x
 LIBS:mateboard-cache
 EELAYER 25 0
@@
 Wire Wire Line
 	6900 1100 6900 3000
-$Comp
-L AM335X_ZCZ IC?
-U 10 1 58ACF85A
-P 1300 5325
-AR Path="/58ACF85A" Ref="IC?"  Part="10"
-AR Path="/58ABDF44/58ACF85A" Ref="IC2"  Part="10"
-F 0 "IC2" H 1400 5725 60  0000 C CNN
-F 1 "AM335X_ZCZ" H 2225 5725 60  0000 C CNN
-F 2 "" H 1300 5325 60  0001 C CNN
-F 3 "" H 1300 5325 60  0001 C CNN
-	10   1300 5325
-	1    0    0    -1
-$EndComp
 Wire Wire Line
 	8100 3000 8100 2175
 Connection ~ 8100 2175
-Text HLabel 5825 5475 2    60   BiDi ~ 0
-MMC0_DAT2
-Wire Wire Line
-	5825 5475 5600 5475
-Text HLabel 5825 5575 2    60   BiDi ~ 0
-MMC0_DAT3
-Wire Wire Line
-	5825 5575 5600 5575
-Text HLabel 5825 5275 2    60   BiDi ~ 0
-MMC0_DAT0
-Text HLabel 5825 5375 2    60   BiDi ~ 0
-MMC0_DAT1
-Wire Wire Line
-	5825 5275 5600 5275
-Wire Wire Line
-	5825 5375 5600 5375
-Text HLabel 5825 5075 2    60   Output ~ 0
-MMC0_CMD
-Text HLabel 5825 5175 2    60   Output ~ 0
-MMC0_CLK
-Wire Wire Line
-	5825 5075 5600 5075
-Wire Wire Line
-	5825 5175 5600 5175
 Wire Wire Line
 	5600 1700 6150 1700
@@
 Wire Wire Line
 	5600 900  6150 900
-Text HLabel 6150 900  2    60   Output ~ 0
-eHRPWM1A
 Wire Wire Line
 	5600 1000 6150 1000
-Text HLabel 6150 1000 2    60   Output ~ 0
-eHRPWM1B
 Wire Wire Line
 	5600 2750 6150 2750
-Text HLabel 6150 2750 2    60   Output ~ 0
-eHRPWM2A
 Wire Wire Line
 	5600 2850 6150 2850
-Text HLabel 6150 2850 2    60   Output ~ 0
-eHRPWM2B
 Wire Wire Line
 	5600 1200 6150 1200
@@
 Wire Wire Line
 	5600 4000 6150 4000
-Text HLabel 6150 4000 2    60   Output ~ 0
+Text HLabel 7950 4000 2    60   Output ~ 0
 TIMER7
 Wire Wire Line
 	5600 4100 6150 4100
-Text HLabel 6150 4100 2    60   Output ~ 0
+Text HLabel 7950 4100 2    60   Output ~ 0
 TIMER6
 Wire Wire Line
 	5600 3600 6150 3600
-Text HLabel 6150 3600 2    60   Output ~ 0
+Text HLabel 7950 3775 2    60   Output ~ 0
 TIMER4
 Wire Wire Line
 	5600 3700 6150 3700
-Text HLabel 6150 3700 2    60   Output ~ 0
+Text HLabel 7950 3875 2    60   Output ~ 0
 TIMER5
 Wire Wire Line
