File: system.sch (KiCad schematic (older format))
At the start: 1 part

Commit message: system sheet
Parts:
- added C? (x4): 18pF/50V, symbol C
- added C?: 2.2uF/10V, symbol C
- added C? (x2): 100nF/10V, symbol C
- added P?: JTAG, symbol CONN_02X10
- added R? (x4): 4.75k, symbol R
- added R?: 1M, symbol R
- added R? (x2): 10k, symbol R
- added R?: 0R, symbol R
- added S?: Reset Button, symbol PushButton
- added U?: 74LVC1G07DCK, symbol 74LVC1G07DCK
- added W?: TESTOUT, symbol TEST_1P
- added Y?: 24MHz, symbol Crystal
- added Y?: 32.768kHz MC-306, symbol Crystal_GND23
Connections:
- net SYS_RESETn: now reaches IC?.A10 (WARMRSTn-nRESETIN_OUT)
- net SYS_RESETn: now also C?.1, C?.1, P?.15 (P15), R?.2, S?.2, U?.4
- net JTAG_TDO: now reaches IC?.A11 (TDO)
- net JTAG_TDO: now also P?.7 (P7)
- net JTAG_TCK: now reaches IC?.A12 (TCK)
- net JTAG_TCK: now also P?.11 (P11), P?.9 (P9)
- net JTAG_EMU2: now reaches IC?.A15 (xDMA_EVENT_INTR0-TIMER4-CLKOUT1-SPI1_CS1-PR1_PRU1_PRU_R31_16-EMU2-GPIO0_19)
- net JTAG_EMU2: now also P?.17 (P17)
- net at IC?.A3 (RSVD-TESTOUT): now also W?.1
- net at IC?.A4 (RTC_XTALOUT): now also C?.1, Y?.4
- net at IC?.A6 (RTC_XTALIN): now also C?.1, Y?.1
- net JTAG_TRSTn: now reaches IC?.B10 (TRSTn)
- net JTAG_TRSTn: now also P?.2 (P2), R?.1
- net JTAG_TDI: now reaches IC?.B11 (TDI)
- net JTAG_TDI: now also P?.3 (P3)
- net JTAG_EMU1: now reaches IC?.B14 (EMU1-GPIO3_8)
- net JTAG_EMU1: now also P?.14 (P14), R?.2
- net POR: now reaches IC?.B15 (PWRONRSTn)
- net POR: now also U?.2
- net NMIn: now reaches IC?.B18 (NMIn-EXTINTn)
- net at IC?.B4 (RTC_KALDO_ENn): now also R?.2
- net RTC_POR: now reaches IC?.B5 (RTC_PWRONRSTn)
- net JTAG_TMS: now reaches IC?.C11 (TMS)
- net JTAG_TMS: now also P?.1 (P1)
- net JTAG_EMU0: now reaches IC?.C14 (EMU0-GPIO3_7)
- net JTAG_EMU0: now also P?.13 (P13), R?.2
- net at IC?.C18 (eCAP0_IN_PWM0_OUT-UART3_TXD-SPI1_CS1-PR1_eCAP0_eCAP_CAPIN_APWM_O-SPI1_SCLK-MMC0_SDWP-XDMA_EVENT_INTR2-GPIO0_7): now also R?.2
- net WAKEUP: now reaches IC?.C5 (EXT_WAKEUP)
- net WAKEUP: now also R?.2
- net PMIC_POWER_EN: now reaches IC?.C6 (PMIC_POWER_EN)
- net JTAG_EMU3: now reaches IC?.D14 (xDMA_EVENT_INTR1-TCLKIN-CLKOUT2-TIMER7-PR1_PRU0_PRU_R31_16-EMU3-GPIO0_20)
- net JTAG_EMU3: now also P?.18 (P18)
- net at IC?.U11 (XTALOUT): now also C?.1, R?.2, Y?.2
- net at IC?.V10 (XTALIN): now also C?.1, R?.1, Y?.1
- new net GNDD: C?.2, C?.2, C?.2, P?.10 (P10), P?.12 (P12), P?.16 (P16), P?.20 (P20), P?.4 (P4), P?.8 (P8), R?.1, R?.2, S?.1, U?.3 (GND)
- new net GND_OSC: C?.2, C?.2
- new net GPIO0_7: R?.1
- new net JTAG_EMU4: P?.19 (P19)
- new net VDD_3V3A: R?.1
- new net VDD_3V3B: C?.1, P?.5 (P5), R?.1, R?.1
- new net VIO: U?.5 (VCC)
- new net VRTC: R?.1
- new net VSS_RTC: C?.2, C?.2
- no-connect marks 0 -> 3
Other:
- moved on the sheet: IC?D

Commit message: wifi bt done
Parts:
- added L?: BLM15AG102SN1D, symbol L
Connections:
- net JTAG_EMU3: now also L?.2
- new net CLKOUT2: L?.1
Changed lines of the file:
@@
 LIBS:tps2065cdgn
 LIBS:74lvc1g07dck
+LIBS:wl1835modgbmoct
 LIBS:mateboard-cache
 EELAYER 25 0
@@
 JTAG_EMU2
 Wire Wire Line
-	5725 4375 6200 4375
+	5725 4375 6350 4375
 Text Label 6200 4375 2    60   ~ 0
 JTAG_EMU3
@@
 Wire Wire Line
 	6225 4775 6100 4775
+$Comp
+L L L?
+U 1 1 58B9CB53
+P 6500 4375
+F 0 "L?" V 6450 4375 50  0000 C CNN
+F 1 "BLM15AG102SN1D" V 6575 4375 50  0000 C CNN
+F 2 "" H 6500 4375 50  0001 C CNN
+F 3 "" H 6500 4375 50  0001 C CNN
+	1    6500 4375
+	0    1    1    0
+$EndComp
+Text HLabel 6900 4375 2    60   Output ~ 0
+CLKOUT2
+Wire Wire Line
+	6900 4375 6650 4375
 $EndSCHEMATC

Commit message: annotation, wip erc
Parts:
- gave numbers to parts that had none: 23
Changed lines of the file:
@@
 P 1225 3125
 AR Path="/58AC1D57" Ref="IC?"  Part="4"
-AR Path="/58AC1B74/58AC1D57" Ref="IC?"  Part="4"
-F 0 "IC?" V 1175 3425 60  0000 C CNN
+AR Path="/58AC1B74/58AC1D57" Ref="IC2"  Part="4"
+F 0 "IC2" V 1175 3425 60  0000 C CNN
 F 1 "AM335X_ZCZ" V 1175 2825 60  0000 C CNN
 F 2 "" H 1225 3125 60  0001 C CNN
@@
 	6250 1475 5725 1475
 $Comp
-L R R?
+L R R35
 U 1 1 58AF48BD
 P 5800 1275
-F 0 "R?" V 5880 1275 50  0000 C CNN
+F 0 "R35" V 5880 1275 50  0000 C CNN
 F 1 "4.75k" V 5800 1275 50  0000 C CNN
 F 2 "" V 5730 1275 50  0000 C CNN
@@
 	5725 1675 6250 1675
 $Comp
-L VRTC #PWR?
+L VRTC #PWR235
 U 1 1 58AF4983
 P 5800 1125
-F 0 "#PWR?" H 5800 975 50  0001 C CNN
+F 0 "#PWR235" H 5800 975 50  0001 C CNN
 F 1 "VRTC" H 5800 1275 50  0000 C CNN
 F 2 "" H 5800 1125 50  0000 C CNN
@@
 WAKEUP
 $Comp
-L Crystal Y?
+L Crystal Y1
 U 1 1 58AF5252
 P 6350 2025
-F 0 "Y?" V 6325 2250 50  0000 C CNN
+F 0 "Y1" V 6325 2250 50  0000 C CNN
 F 1 "24MHz" V 6400 2250 50  0000 C CNN
 F 2 "" H 6350 2025 50  0000 C CNN
@@
 	5725 2175 6650 2175
 $Comp
-L R R?
+L R R36
 U 1 1 58AF52F6
 P 5900 2025
-F 0 "R?" V 5980 2025 50  0000 C CNN
+F 0 "R36" V 5980 2025 50  0000 C CNN
 F 1 "1M" V 5900 2025 50  0000 C CNN
 F 2 "" V 5830 2025 50  0000 C CNN
@@
 Connection ~ 5900 2175
 $Comp
-L C C?
+L C C118
 U 1 1 58AF5351
 P 6800 1875
-F 0 "C?" V 6925 1725 50  0000 L CNN
+F 0 "C118" V 6925 1725 50  0000 L CNN
 F 1 "18pF/50V" V 6850 1425 50  0000 L CNN
 F 2 "" H 6838 1725 50  0000 C CNN
@@
 	7275 2175 6950 2175
 $Comp
-L GND_OSC #PWR?
+L GND_OSC #PWR237
 U 1 1 58AF548A
 P 7275 2225
-F 0 "#PWR?" H 7275 2225 30  0001 C CNN
+F 0 "#PWR237" H 7275 2225 30  0001 C CNN
 F 1 "GND_OSC" H 7275 2155 30  0000 C CNN
 F 2 "" H 7275 2225 60  0001 C CNN
@@
 Connection ~ 7275 2175
 $Comp
-L Crystal_GND23 Y?
+L Crystal_GND23 Y2
 U 1 1 58AF6150
 P 6350 2475
-F 0 "Y?" V 6325 2725 50  0000 L CNN
+F 0 "Y2" V 6325 2725 50  0000 L CNN
 F 1 "32.768kHz MC-306" V 6400 2725 50  0000 L CNN
 F 2 "" H 6350 2475 50  0000 C CNN
@@
 NoConn ~ 6150 2475
 $Comp
-L C C?
+L C C119
 U 1 1 58AF6403
 P 6800 2175
-F 0 "C?" V 6925 2025 50  0000 L CNN
+F 0 "C119" V 6925 2025 50  0000 L CNN
 F 1 "18pF/50V" V 6850 1725 50  0000 L CNN
 F 2 "" H 6838 2025 50  0000 C CNN
@@
 $EndComp
 $Comp
-L C C?
+L C C120
 U 1 1 58AF664D
 P 7450 2325
-F 0 "C?" V 7575 2175 50  0000 L CNN
+F 0 "C120" V 7575 2175 50  0000 L CNN
 F 1 "18pF/50V" V 7500 1875 50  0000 L CNN
 F 2 "" H 7488 2175 50  0000 C CNN
@@
 Connection ~ 7925 2625
 $Comp
-L C C?
+L C C121
 U 1 1 58AF665E
 P 7450 2625
-F 0 "C?" V 7575 2475 50  0000 L CNN
+F 0 "C121" V 7575 2475 50  0000 L CNN
 F 1 "18pF/50V" V 7500 2175 50  0000 L CNN
 F 2 "" H 7488 2475 50  0000 C CNN
@@
 VSS_RTC
 $Comp
-L PushButton S?
+L PushButton S2
 U 1 1 58AFBFEC
 P 9275 3675
-F 0 "S?" H 9275 3475 60  0000 C CNN
+F 0 "S2" H 9275 3475 60  0000 C CNN
 F 1 "Reset Button" H 9300 3575 60  0000 C CNN
 F 2 "" H 9275 3675 60  0001 C CNN
@@
 $EndComp
 $Comp
-L GNDD #PWR?
+L GNDD #PWR242
 U 1 1 58AFBFF3
 P 9625 3675
-F 0 "#PWR?" H 9625 3425 50  0001 C CNN
+F 0 "#PWR242" H 9625 3425 50  0001 C CNN
 F 1 "GNDD" V 9625 3475 50  0000 C CNN
 F 2 "" H 9625 3675 50  0000 C CNN
@@
 POR
 $Comp
-L 74LVC1G07DCK U?
+L 74LVC1G07DCK U4
 U 1 1 58AFDB30
 P 7450 3275
-F 0 "U?" H 7645 3390 50  0000 C CNN
+F 0 "U4" H 7645 3390 50  0000 C CNN
 F 1 "74LVC1G07DCK" H 7750 3125 50  0000 C CNN
 F 2 "" H 7450 3275 50  0000 C CNN
@@
 	5725 3275 7000 3275
 $Comp
-L GNDD #PWR?
+L GNDD #PWR239
 U 1 1 58AFE459
 P 7500 3475
-F 0 "#PWR?" H 7500 3225 50  0001 C CNN
+F 0 "#PWR239" H 7500 3225 50  0001 C CNN
 F 1 "GNDD" H 7500 3325 50  0000 C CNN
 F 2 "" H 7500 3475 50  0000 C CNN
@@
 $EndComp
 $Comp
-L VIO #PWR?
+L VIO #PWR238
 U 1 1 58AFE60F
 P 7500 3000
-F 0 "#PWR?" H 7500 2850 50  0001 C CNN
+F 0 "#PWR238" H 7500 2850 50  0001 C CNN
 F 1 "VIO" H 7500 3150 50  0000 C CNN
 F 2 "" H 7500 3000 50  0000 C CNN
@@
 Connection ~ 6350 3275
 $Comp
-L C C?
+L C C122
 U 1 1 58AFEEE9
 P 8525 3850
-F 0 "C?" H 8550 3950 50  0000 L CNN
+F 0 "C122" H 8550 3950 50  0000 L CNN
 F 1 "2.2uF/10V" H 8550 3750 50  0000 L CNN
 F 2 "" H 8563 3700 50  0000 C CNN
@@
 $EndComp
 $Comp
-L R R?
+L R R39
 U 1 1 58AFF009
 P 8525 3500
-F 0 "R?" V 8605 3500 50  0000 C CNN
+F 0 "R39" V 8605 3500 50  0000 C CNN
 F 1 "10k" V 8525 3500 50  0000 C CNN
 F 2 "" V 8455 3500 50  0000 C CNN
@@
 Connection ~ 8525 3675
 $Comp
-L VDD_3V3A #PWR?
+L VDD_3V3A #PWR240
 U 1 1 58AFF28A
 P 8525 3350
-F 0 "#PWR?" H 8525 3200 50  0001 C CNN
+F 0 "#PWR240" H 8525 3200 50  0001 C CNN
 F 1 "VDD_3V3A" H 8525 3500 50  0000 C CNN
 F 2 "" H 8525 3350 50  0000 C CNN
@@
 $EndComp
 $Comp
-L GNDD #PWR?
+L GNDD #PWR241
 U 1 1 58AFF2DD
 P 8525 4000
-F 0 "#PWR?" H 8525 3750 50  0001 C CNN
+F 0 "#PWR241" H 8525 3750 50  0001 C CNN
 F 1 "GNDD" H 8525 3850 50  0000 C CNN
 F 2 "" H 8525 4000 50  0000 C CNN
@@
 	6250 2925 5725 2925
 $Comp
-L CONN_02X10 P?
+L CONN_02X10 P5
 U 1 1 58B00233
 P 3650 5900
-F 0 "P?" H 3650 6450 50  0000 C CNN
+F 0 "P5" H 3650 6450 50  0000 C CNN
 F 1 "JTAG" V 3650 5900 50  0000 C CNN
 F 2 "" H 3650 4700 50  0000 C CNN
@@
 	2825 5550 3400 5550
 $Comp
-L VDD_3V3B #PWR?
+L VDD_3V3B #PWR230
 U 1 1 58B00DF7
 P 3325 5300
-F 0 "#PWR?" H 3325 5150 50  0001 C CNN
+F 0 "#PWR230" H 3325 5150 50  0001 C CNN
 F 1 "VDD_3V3B" H 3325 5450 50  0000 C CNN
 F 2 "" H 3325 5300 50  0000 C CNN
@@
 	2400 6150 3400 6150
 $Comp
-L C C?
+L C C116
 U 1 1 58B02147
 P 2400 6300
-F 0 "C?" H 2425 6400 50  0000 L CNN
+F 0 "C116" H 2425 6400 50  0000 L CNN
 F 1 "100nF/10V" H 2425 6200 50  0000 L CNN
 F 2 "" H 2438 6150 50  0000 C CNN
@@
 $EndComp
 $Comp
-L GNDD #PWR?
+L GNDD #PWR229
 U 1 1 58B0214D
 P 2400 6450
-F 0 "#PWR?" H 2400 6200 50  0001 C CNN
+F 0 "#PWR229" H 2400 6200 50  0001 C CNN
 F 1 "GNDD" H 2400 6300 50  0000 C CNN
 F 2 "" H 2400 6450 50  0000 C CNN
@@
 $EndComp
 $Comp
-L C C?
+L C C117
 U 1 1 58B022AB
 P 3325 6550
-F 0 "C?" H 3350 6650 50  0000 L CNN
+F 0 "C117" H 3350 6650 50  0000 L CNN
 F 1 "100nF/10V" H 3350 6450 50  0000 L CNN
 F 2 "" H 3363 6400 50  0000 C CNN
@@
 $EndComp
 $Comp
-L GNDD #PWR?
+L GNDD #PWR231
 U 1 1 58B022B1
 P 3325 6700
-F 0 "#PWR?" H 3325 6450 50  0001 C CNN
+F 0 "#PWR231" H 3325 6450 50  0001 C CNN
 F 1 "GNDD" H 3325 6550 50  0000 C CNN
 F 2 "" H 3325 6700 50  0000 C CNN
@@
 	4825 6250 3900 6250
 $Comp
-L R R?
+L R R32
 U 1 1 58B02D3C
 P 2400 5900
-F 0 "R?" V 2480 5900 50  0000 C CNN
+F 0 "R32" V 2480 5900 50  0000 C CNN
 F 1 "4.75k" V 2400 5900 50  0000 C CNN
 F 2 "" V 2330 5900 50  0000 C CNN
@@
 $EndComp
 $Comp
-L VDD_3V3B #PWR?
+L VDD_3V3B #PWR228
 U 1 1 58B02FB2
 P 2400 5750
-F 0 "#PWR?" H 2400 5600 50  0001 C CNN
+F 0 "#PWR228" H 2400 5600 50  0001 C CNN
 F 1 "VDD_3V3B" H 2400 5900 50  0000 C CNN
 F 2 "" H 2400 5750 50  0000 C CNN
@@
 	3900 6050 5000 6050
 $Comp
-L R R?
+L R R34
 U 1 1 58B0647B
 P 5000 5900
-F 0 "R?" V 5080 5900 50  0000 C CNN
+F 0 "R34" V 5080 5900 50  0000 C CNN
 F 1 "4.75k" V 5000 5900 50  0000 C CNN
 F 2 "" V 4930 5900 50  0000 C CNN
@@
 $EndComp
 $Comp
-L VDD_3V3B #PWR?
+L VDD_3V3B #PWR234
 U 1 1 58B06481
 P 5000 5750
-F 0 "#PWR?" H 5000 5600 50  0001 C CNN
+F 0 "#PWR234" H 5000 5600 50  0001 C CNN
 F 1 "VDD_3V3B" H 5000 5900 50  0000 C CNN
 F 2 "" H 5000 5750 50  0000 C CNN
@@
 $EndComp
 $Comp
-L R R?
+L R R33
 U 1 1 58B064FD
 P 3950 6550
-F 0 "R?" V 4030 6550 50  0000 C CNN
+F 0 "R33" V 4030 6550 50  0000 C CNN
 F 1 "4.75k" V 3950 6550 50  0000 C CNN
 F 2 "" V 3880 6550 50  0000 C CNN
@@
 Connection ~ 3950 5450
 $Comp
-L GNDD #PWR?
+L GNDD #PWR232
 U 1 1 58B06ADB
 P 3950 6700
-F 0 "#PWR?" H 3950 6450 50  0001 C CNN
+F 0 "#PWR232" H 3950 6450 50  0001 C CNN
 F 1 "GNDD" H 3950 6550 50  0000 C CNN
 F 2 "" H 3950 6700 50  0000 C CNN
@@
 	4200 5550 4200 6700
 $Comp
-L GNDD #PWR?
+L GNDD #PWR233
 U 1 1 58B06BC7
 P 4200 6700
-F 0 "#PWR?" H 4200 6450 50  0001 C CNN
+F 0 "#PWR233" H 4200 6450 50  0001 C CNN
 F 1 "GNDD" H 4200 6550 50  0000 C CNN
 F 2 "" H 4200 6700 50  0000 C CNN
@@
 JTAG_EMU4
 $Comp
-L R R?
+L R R38
 U 1 1 58B0F772
 P 5975 2825
-F 0 "R?" V 5925 2975 50  0000 C CNN
+F 0 "R38" V 5925 2975 50  0000 C CNN
 F 1 "10k" V 5975 2825 50  0000 C CNN
 F 2 "" V 5905 2825 50  0000 C CNN
@@
 	5825 2825 5725 2825
 $Comp
-L GNDD #PWR?
+L GNDD #PWR236
 U 1 1 58B0F970
 P 6125 2825
-F 0 "#PWR?" H 6125 2575 50  0001 C CNN
+F 0 "#PWR236" H 6125 2575 50  0001 C CNN
 F 1 "GNDD" V 6125 2600 50  0000 C CNN
 F 2 "" H 6125 2825 50  0000 C CNN
@@
 	6250 3175 5725 3175
 $Comp
-L TEST_1P W?
+L TEST_1P W2
 U 1 1 58B13012
 P 5725 4575
-F 0 "W?" V 5725 4800 50  0000 C CNN
+F 0 "W2" V 5725 4800 50  0000 C CNN
 F 1 "TESTOUT" V 5725 5075 50  0000 C CNN
 F 2 "" H 5925 4575 50  0000 C CNN
@@
 $EndComp
 $Comp
-L R R?
+L R R37
 U 1 1 58B13994
 P 5950 4775
-F 0 "R?" V 6030 4775 50  0000 C CNN
+F 0 "R37" V 6030 4775 50  0000 C CNN
 F 1 "0R" V 5950 4775 50  0000 C CNN
 F 2 "" V 5880 4775 50  0000 C CNN
@@
 	6225 4775 6100 4775
 $Comp
-L L L?
+L L L8
 U 1 1 58B9CB53
 P 6500 4375
-F 0 "L?" V 6450 4375 50  0000 C CNN
+F 0 "L8" V 6450 4375 50  0000 C CNN
 F 1 "BLM15AG102SN1D" V 6575 4375 50  0000 C CNN
 F 2 "" H 6500 4375 50  0001 C CNN
