File: system.sch (KiCad schematic (older format))
At the start: 38 parts, among them IC1 OSD335x, IC3 NAND_4GB, U8 SN74LVC1G06DCK, U9 74LVC1G07DCK, Y1 24MHz, Y2 32.768kHz

Commit message: wip footprint assoc
Parts:
- C16, C17, C18, C19, C20, C26, C27, C28: footprint (none) -> Capacitors_SMD:C_0402
- C21, C22, C23, C24: footprint (none) -> Capacitors_SMD:C_0603
- C25: footprint (none) -> Capacitors_SMD:C_0805
- IC1: footprint GHI-SoMs-Processors_OSD3358 -> footprints:OSD3358-BAS-BGA400
- L4, L5, R31, R32, R33, R34, R35, R36, R37, R38, R39, R40, R41, R42, R43, R44, R45, R46, R47: footprint (none) -> Resistors_SMD:R_0402
Changed lines of the file:
@@
 F 0 "Y1" V 1650 1150 50  0000 C CNN
 F 1 "24MHz" V 1725 1150 50  0000 C CNN
-F 2 "" H 1675 925 50  0000 C CNN
+F 2 "" H 1675 925 50  0001 C CNN
 F 3 "" H 1675 925 50  0000 C CNN
 	1    1675 925
@@
 F 0 "R31" V 2205 925 50  0000 C CNN
 F 1 "1M" V 2125 925 50  0000 C CNN
-F 2 "" V 2055 925 50  0000 C CNN
+F 2 "Resistors_SMD:R_0402" V 2055 925 50  0001 C CNN
 F 3 "" H 2125 925 50  0000 C CNN
 	1    2125 925
@@
 F 0 "C16" V 1350 625 50  0000 L CNN
 F 1 "18pF/50V" V 1275 325 50  0000 L CNN
-F 2 "" H 1263 625 50  0000 C CNN
+F 2 "Capacitors_SMD:C_0402" H 1263 625 50  0001 C CNN
 F 3 "" H 1225 775 50  0000 C CNN
 	1    1225 775
@@
 F 0 "C17" V 1350 925 50  0000 L CNN
 F 1 "18pF/50V" V 1275 625 50  0000 L CNN
-F 2 "" H 1263 925 50  0000 C CNN
+F 2 "Capacitors_SMD:C_0402" H 1263 925 50  0001 C CNN
 F 3 "" H 1225 1075 50  0000 C CNN
 	1    1225 1075
@@
 F 0 "U9" H 8070 1090 50  0000 C CNN
 F 1 "74LVC1G07DCK" H 8175 825 50  0000 C CNN
-F 2 "" H 7875 975 50  0000 C CNN
+F 2 "" H 7875 975 50  0001 C CNN
 F 3 "" H 7875 975 50  0000 C CNN
 	1    7875 975
@@
 F 0 "C21" H 8975 1650 50  0000 L CNN
 F 1 "2.2uF/6.3V" H 8975 1450 50  0000 L CNN
-F 2 "" H 8988 1400 50  0000 C CNN
+F 2 "Capacitors_SMD:C_0603" H 8988 1400 50  0001 C CNN
 F 3 "" H 8950 1550 50  0000 C CNN
 	1    8950 1550
@@
 F 0 "R47" V 9030 1200 50  0000 C CNN
 F 1 "10k" V 8950 1200 50  0000 C CNN
-F 2 "" V 8880 1200 50  0000 C CNN
+F 2 "Resistors_SMD:R_0402" V 8880 1200 50  0001 C CNN
 F 3 "" H 8950 1200 50  0000 C CNN
 	1    8950 1200
@@
 F 0 "L5" V 5800 1625 50  0000 C CNN
 F 1 "BLM15AG102SN1D" V 5700 1600 50  0000 C CNN
-F 2 "" H 5750 1475 50  0001 C CNN
+F 2 "Resistors_SMD:R_0402" H 5750 1475 50  0001 C CNN
 F 3 "" H 5750 1475 50  0001 C CNN
 	1    5750 1475
@@
 F 0 "IC1" H 3700 3100 45  0000 L BNN
 F 1 "OSD335x" H 3625 3000 45  0000 L BNN
-F 2 "GHI-SoMs-Processors_OSD3358" H 3805 3225 20  0001 C CNN
+F 2 "footprints:OSD3358-BAS-BGA400" H 3805 3225 20  0001 C CNN
 F 3 "" H 3775 3075 60  0001 C CNN
 	1    3775 3075
@@
 F 0 "Y2" V 1600 1675 50  0000 C CNN
 F 1 "32.768kHz" V 1700 1750 50  0000 C CNN
-F 2 "" H 1675 1425 50  0000 C CNN
+F 2 "" H 1675 1425 50  0001 C CNN
 F 3 "" H 1675 1425 50  0000 C CNN
 	1    1675 1425
@@
 F 0 "R32" V 2205 1425 50  0000 C CNN
 F 1 "DNP 1M" V 2025 1425 50  0000 C CNN
-F 2 "" V 2055 1425 50  0000 C CNN
+F 2 "Resistors_SMD:R_0402" V 2055 1425 50  0001 C CNN
 F 3 "" H 2125 1425 50  0000 C CNN
 	1    2125 1425
@@
 F 0 "C18" V 1275 1125 50  0000 L CNN
 F 1 "18pF/50V" V 1175 850 50  0000 L CNN
-F 2 "" H 1263 1125 50  0000 C CNN
+F 2 "Capacitors_SMD:C_0402" H 1263 1125 50  0001 C CNN
 F 3 "" H 1225 1275 50  0000 C CNN
 	1    1225 1275
@@
 F 0 "C19" V 1275 1425 50  0000 L CNN
 F 1 "18pF/50V" V 1175 1125 50  0000 L CNN
-F 2 "" H 1263 1425 50  0000 C CNN
+F 2 "Capacitors_SMD:C_0402" H 1263 1425 50  0001 C CNN
 F 3 "" H 1225 1575 50  0000 C CNN
 	1    1225 1575
@@
 F 0 "C25" H 10150 2550 50  0000 L CNN
 F 1 "4.7uF/6.3V" H 10150 2350 50  0000 L CNN
-F 2 "" H 10163 2300 50  0000 C CNN
+F 2 "Capacitors_SMD:C_0805" H 10163 2300 50  0001 C CNN
 F 3 "" H 10125 2450 50  0000 C CNN
 	1    10125 2450
@@
 F 0 "R42" V 7250 2700 50  0000 C CNN
 F 1 "10k" V 7300 2550 50  0000 C CNN
-F 2 "" V 7230 2550 50  0000 C CNN
+F 2 "Resistors_SMD:R_0402" V 7230 2550 50  0001 C CNN
 F 3 "" H 7300 2550 50  0000 C CNN
 	1    7300 2550
@@
 F 0 "R44" V 7350 2700 50  0000 C CNN
 F 1 "10k" V 7400 2550 50  0000 C CNN
-F 2 "" V 7330 2550 50  0000 C CNN
+F 2 "Resistors_SMD:R_0402" V 7330 2550 50  0001 C CNN
 F 3 "" H 7400 2550 50  0000 C CNN
 	1    7400 2550
@@
 F 0 "R45" V 7450 2700 50  0000 C CNN
 F 1 "10k" V 7500 2550 50  0000 C CNN
-F 2 "" V 7430 2550 50  0000 C CNN
+F 2 "Resistors_SMD:R_0402" V 7430 2550 50  0001 C CNN
 F 3 "" H 7500 2550 50  0000 C CNN
 	1    7500 2550
@@
 F 0 "R46" V 7550 2700 50  0000 C CNN
 F 1 "10k" V 7600 2550 50  0000 C CNN
-F 2 "" V 7530 2550 50  0000 C CNN
+F 2 "Resistors_SMD:R_0402" V 7530 2550 50  0001 C CNN
 F 3 "" H 7600 2550 50  0000 C CNN
 	1    7600 2550
@@
 F 0 "R38" V 6850 2700 50  0000 C CNN
 F 1 "10k" V 6900 2550 50  0000 C CNN
-F 2 "" V 6830 2550 50  0000 C CNN
+F 2 "Resistors_SMD:R_0402" V 6830 2550 50  0001 C CNN
 F 3 "" H 6900 2550 50  0000 C CNN
 	1    6900 2550
@@
 F 0 "R39" V 6950 2700 50  0000 C CNN
 F 1 "10k" V 7000 2550 50  0000 C CNN
-F 2 "" V 6930 2550 50  0000 C CNN
+F 2 "Resistors_SMD:R_0402" V 6930 2550 50  0001 C CNN
 F 3 "" H 7000 2550 50  0000 C CNN
 	1    7000 2550
@@
 F 0 "R40" V 7050 2700 50  0000 C CNN
 F 1 "10k" V 7100 2550 50  0000 C CNN
-F 2 "" V 7030 2550 50  0000 C CNN
+F 2 "Resistors_SMD:R_0402" V 7030 2550 50  0001 C CNN
 F 3 "" H 7100 2550 50  0000 C CNN
 	1    7100 2550
@@
 F 0 "R41" V 7150 2700 50  0000 C CNN
 F 1 "10k" V 7200 2550 50  0000 C CNN
-F 2 "" V 7130 2550 50  0000 C CNN
+F 2 "Resistors_SMD:R_0402" V 7130 2550 50  0001 C CNN
 F 3 "" H 7200 2550 50  0000 C CNN
 	1    7200 2550
@@
 F 0 "R35" V 6550 2700 50  0000 C CNN
 F 1 "10k" V 6600 2550 50  0000 C CNN
-F 2 "" V 6530 2550 50  0000 C CNN
+F 2 "Resistors_SMD:R_0402" V 6530 2550 50  0001 C CNN
 F 3 "" H 6600 2550 50  0000 C CNN
 	1    6600 2550
@@
 F 0 "R36" V 6650 2700 50  0000 C CNN
 F 1 "10k" V 6700 2550 50  0000 C CNN
-F 2 "" V 6630 2550 50  0000 C CNN
+F 2 "Resistors_SMD:R_0402" V 6630 2550 50  0001 C CNN
 F 3 "" H 6700 2550 50  0000 C CNN
 	1    6700 2550
@@
 F 0 "R37" V 6750 2700 50  0000 C CNN
 F 1 "10k" V 6800 2550 50  0000 C CNN
-F 2 "" V 6730 2550 50  0000 C CNN
+F 2 "Resistors_SMD:R_0402" V 6730 2550 50  0001 C CNN
 F 3 "" H 6800 2550 50  0000 C CNN
 	1    6800 2550
@@
 F 0 "U8" H 6900 4975 50  0000 C CNN
 F 1 "SN74LVC1G06DCK" H 7050 4875 50  0000 C CNN
-F 2 "" H 6845 4940 50  0000 C CNN
+F 2 "" H 6845 4940 50  0001 C CNN
 F 3 "" H 6895 5190 50  0000 C CNN
 	1    6750 5075
@@
 F 0 "R43" V 7430 5075 50  0000 C CNN
 F 1 "0R" V 7350 5075 50  0000 C CNN
-F 2 "" V 7280 5075 50  0000 C CNN
+F 2 "Resistors_SMD:R_0402" V 7280 5075 50  0001 C CNN
 F 3 "" H 7350 5075 50  0000 C CNN
 	1    7350 5075
@@
 F 0 "C20" V 6725 4650 50  0000 L CNN
 F 1 "100nF/6.3V" V 6800 4300 50  0000 L CNN
-F 2 "" H 6938 4650 50  0000 C CNN
+F 2 "Capacitors_SMD:C_0402" H 6938 4650 50  0001 C CNN
 F 3 "" H 6900 4800 50  0000 C CNN
 	1    6900 4800
@@
 F 0 "R33" V 5250 1325 50  0000 C CNN
 F 1 "0 1%" V 5200 1175 50  0000 C CNN
-F 2 "" V 5130 1175 50  0001 C CNN
+F 2 "Resistors_SMD:R_0402" V 5130 1175 50  0001 C CNN
 F 3 "" H 5200 1175 50  0001 C CNN
 	1    5200 1175
@@
 F 0 "L4" V 5775 1425 50  0000 C CNN
 F 1 "BLM15AG102SN1D" V 5675 1400 50  0000 C CNN
-F 2 "" H 5725 1275 50  0001 C CNN
+F 2 "Resistors_SMD:R_0402" H 5725 1275 50  0001 C CNN
 F 3 "" H 5725 1275 50  0001 C CNN
 	1    5725 1275
@@
 F 0 "C28" H 10675 2550 50  0000 L CNN
 F 1 "100nF/6.3V" H 10675 2350 50  0000 L CNN
-F 2 "" H 10688 2300 50  0000 C CNN
+F 2 "Capacitors_SMD:C_0402" H 10688 2300 50  0001 C CNN
 F 3 "" H 10650 2450 50  0000 C CNN
 	1    10650 2450
@@
 F 0 "C22" H 10125 3300 50  0000 L CNN
 F 1 "2.2uF/6.3V" H 10125 3100 50  0000 L CNN
-F 2 "" H 10138 3050 50  0000 C CNN
+F 2 "Capacitors_SMD:C_0603" H 10138 3050 50  0001 C CNN
 F 3 "" H 10100 3200 50  0000 C CNN
 	1    10100 3200
@@
 F 0 "C26" H 10600 3300 50  0000 L CNN
 F 1 "100nF/6.3V" H 10600 3100 50  0000 L CNN
-F 2 "" H 10613 3050 50  0000 C CNN
+F 2 "Capacitors_SMD:C_0402" H 10613 3050 50  0001 C CNN
 F 3 "" H 10575 3200 50  0000 C CNN
 	1    10575 3200
@@
 F 0 "R34" V 5300 4625 50  0000 C CNN
 F 1 "0R" V 5250 4775 50  0000 C CNN
-F 2 "" V 5180 4775 50  0001 C CNN
+F 2 "Resistors_SMD:R_0402" V 5180 4775 50  0001 C CNN
 F 3 "" H 5250 4775 50  0001 C CNN
 	1    5250 4775
@@
 F 0 "C23" H 10125 4025 50  0000 L CNN
 F 1 "2.2uF/6.3V" H 10125 3825 50  0000 L CNN
-F 2 "" H 10138 3775 50  0000 C CNN
+F 2 "Capacitors_SMD:C_0603" H 10138 3775 50  0001 C CNN
 F 3 "" H 10100 3925 50  0000 C CNN
 	1    10100 3925
@@
 F 0 "C24" H 10125 4725 50  0000 L CNN
 F 1 "2.2uF/6.3V" H 10125 4525 50  0000 L CNN
-F 2 "" H 10138 4475 50  0000 C CNN
+F 2 "Capacitors_SMD:C_0603" H 10138 4475 50  0001 C CNN
 F 3 "" H 10100 4625 50  0000 C CNN
 	1    10100 4625
@@
 F 0 "C27" H 10600 4025 50  0000 L CNN
 F 1 "100nF/6.3V" H 10600 3825 50  0000 L CNN
-F 2 "" H 10613 3775 50  0000 C CNN
+F 2 "Capacitors_SMD:C_0402" H 10613 3775 50  0001 C CNN
 F 3 "" H 10575 3925 50  0000 C CNN
 	1    10575 3925
