File: system.sch (KiCad schematic (older format))
At the start: 38 parts, among them IC1 OSD335x, IC3 NAND_4GB, U8 SN74LVC1G06DCK, U9 74LVC1G07DCK, Y1 24MHz, Y2 32.768kHz

Commit message: wip footprint assoc
Parts:
- U8, U9: footprint (none) -> TO_SOT_Packages_SMD:SOT-353_SC-70-5
- Y1: footprint (none) -> Crystals:Crystal_SMD_5032-2pin_5.0x3.2mm
- Y2: footprint (none) -> Crystals:Crystal_SMD_3215-2pin_3.2x1.5mm
Changed lines of the file:
@@
 F 0 "Y1" V 1650 1150 50  0000 C CNN
 F 1 "24MHz" V 1725 1150 50  0000 C CNN
-F 2 "" H 1675 925 50  0001 C CNN
+F 2 "Crystals:Crystal_SMD_5032-2pin_5.0x3.2mm" H 1675 925 50  0001 C CNN
 F 3 "" H 1675 925 50  0000 C CNN
 	1    1675 925
@@
 F 0 "U9" H 8070 1090 50  0000 C CNN
 F 1 "74LVC1G07DCK" H 8175 825 50  0000 C CNN
-F 2 "" H 7875 975 50  0001 C CNN
+F 2 "TO_SOT_Packages_SMD:SOT-353_SC-70-5" H 7875 975 50  0001 C CNN
 F 3 "" H 7875 975 50  0000 C CNN
 	1    7875 975
@@
 F 0 "Y2" V 1600 1675 50  0000 C CNN
 F 1 "32.768kHz" V 1700 1750 50  0000 C CNN
-F 2 "" H 1675 1425 50  0001 C CNN
+F 2 "Crystals:Crystal_SMD_3215-2pin_3.2x1.5mm" H 1675 1425 50  0001 C CNN
 F 3 "" H 1675 1425 50  0000 C CNN
 	1    1675 1425
@@
 F 0 "U8" H 6900 4975 50  0000 C CNN
 F 1 "SN74LVC1G06DCK" H 7050 4875 50  0000 C CNN
-F 2 "" H 6845 4940 50  0001 C CNN
+F 2 "TO_SOT_Packages_SMD:SOT-353_SC-70-5" H 6845 4940 50  0001 C CNN
 F 3 "" H 6895 5190 50  0000 C CNN
 	1    6750 5075

Commit message: wip routing
Connections:
- net GPIO1_28: no longer IC1.V14 (GPIO1_17), IC1.V17 ((HDMICLK_DISN)GPIO1_27)
- new net GPIO1_17: IC1.V14 (GPIO1_17)
- new net GPIO1_27: IC1.V17 ((HDMICLK_DISN)GPIO1_27)
Changed lines of the file:
@@
 	4975 975  7425 975
 $Comp
-L GNDD #PWR0106
+L GNDD #PWR0104
 U 1 1 58AFE459
 P 7925 1175
-F 0 "#PWR0106" H 7925 925 50  0001 C CNN
+F 0 "#PWR0104" H 7925 925 50  0001 C CNN
 F 1 "GNDD" H 7925 1025 50  0000 C CNN
 F 2 "" H 7925 1175 50  0000 C CNN
@@
 Connection ~ 8950 1375
 $Comp
-L VDD_3V3A #PWR0107
+L VDD_3V3A #PWR0105
 U 1 1 58AFF28A
 P 8950 1050
-F 0 "#PWR0107" H 8950 900 50  0001 C CNN
+F 0 "#PWR0105" H 8950 900 50  0001 C CNN
 F 1 "VDD_3V3A" H 8950 1200 50  0000 C CNN
 F 2 "" H 8950 1050 50  0000 C CNN
@@
 $EndComp
 $Comp
-L GNDD #PWR0108
+L GNDD #PWR0106
 U 1 1 58AFF2DD
 P 8950 1700
-F 0 "#PWR0108" H 8950 1450 50  0001 C CNN
+F 0 "#PWR0106" H 8950 1450 50  0001 C CNN
 F 1 "GNDD" H 8950 1550 50  0000 C CNN
 F 2 "" H 8950 1700 50  0000 C CNN
@@
 $EndComp
 $Comp
-L VDD_3V3B #PWR0109
+L VDD_3V3B #PWR0107
 U 1 1 58D48CDC
 P 9275 2375
-F 0 "#PWR0109" H 9275 2225 50  0001 C CNN
+F 0 "#PWR0107" H 9275 2225 50  0001 C CNN
 F 1 "VDD_3V3B" H 9275 2525 50  0000 C CNN
 F 2 "" H 9275 2375 50  0000 C CNN
@@
 $EndComp
 $Comp
-L GNDD #PWR0110
+L GNDD #PWR0108
 U 1 1 58D48CFA
 P 10125 2600
-F 0 "#PWR0110" H 10125 2350 50  0001 C CNN
+F 0 "#PWR0108" H 10125 2350 50  0001 C CNN
 F 1 "GNDD" H 10125 2450 50  0000 C CNN
 F 2 "" H 10125 2600 50  0000 C CNN
@@
 	9850 2300 10650 2300
 $Comp
-L GNDD #PWR0111
+L GNDD #PWR0109
 U 1 1 58D48D02
 P 9275 4175
-F 0 "#PWR0111" H 9275 3925 50  0001 C CNN
+F 0 "#PWR0109" H 9275 3925 50  0001 C CNN
 F 1 "GNDD" H 9275 4025 50  0000 C CNN
 F 2 "" H 9275 4175 50  0000 C CNN
@@
 $EndComp
 $Comp
-L VDD_3V3B #PWR0112
+L VDD_3V3B #PWR0110
 U 1 1 58D48D66
 P 7000 2275
-F 0 "#PWR0112" H 7000 2125 50  0001 C CNN
+F 0 "#PWR0110" H 7000 2125 50  0001 C CNN
 F 1 "VDD_3V3B" H 7000 2425 50  0000 C CNN
 F 2 "" H 7000 2275 50  0000 C CNN
@@
 $EndComp
 $Comp
-L VDD_3V3A #PWR0113
+L VDD_3V3A #PWR0111
 U 1 1 58D48DB0
 P 6700 4700
-F 0 "#PWR0113" H 6700 4550 50  0001 C CNN
+F 0 "#PWR0111" H 6700 4550 50  0001 C CNN
 F 1 "VDD_3V3A" H 6700 4850 50  0000 C CNN
 F 2 "" H 6700 4700 50  0000 C CNN
@@
 $EndComp
 $Comp
-L GNDD #PWR0114
+L GNDD #PWR0112
 U 1 1 58D48DB6
 P 6700 5275
-F 0 "#PWR0114" H 6700 5025 50  0001 C CNN
+F 0 "#PWR0112" H 6700 5025 50  0001 C CNN
 F 1 "GNDD" H 6700 5125 50  0000 C CNN
 F 2 "" H 6700 5275 50  0000 C CNN
@@
 $EndComp
 $Comp
-L GNDD #PWR0115
+L GNDD #PWR0113
 U 1 1 58D48DC3
 P 7050 4800
-F 0 "#PWR0115" H 7050 4550 50  0001 C CNN
+F 0 "#PWR0113" H 7050 4550 50  0001 C CNN
 F 1 "GNDD" V 7050 4600 50  0000 C CNN
 F 2 "" H 7050 4800 50  0000 C CNN
@@
 Connection ~ 7500 3775
 $Comp
-L PWR_FLAG #FLG0116
+L PWR_FLAG #FLG0114
 U 1 1 58D48DD0
 P 9850 2275
-F 0 "#FLG0116" H 9850 2350 50  0001 C CNN
+F 0 "#FLG0114" H 9850 2350 50  0001 C CNN
 F 1 "PWR_FLAG" H 9850 2425 50  0001 C CNN
 F 2 "" H 9850 2275 50  0001 C CNN
@@
 	5950 875  4975 875
 $Comp
-L VDD_1V8 #PWR0117
+L VDD_1V8 #PWR0115
 U 1 1 58DA59D5
 P 7925 700
-F 0 "#PWR0117" H 7925 550 50  0001 C CNN
+F 0 "#PWR0115" H 7925 550 50  0001 C CNN
 F 1 "VDD_1V8" H 7925 850 50  0000 C CNN
 F 2 "" H 7925 700 50  0000 C CNN
@@
 $EndComp
 $Comp
-L GNDD #PWR0118
+L GNDD #PWR0116
 U 1 1 58DADD35
 P 10650 2600
-F 0 "#PWR0118" H 10650 2350 50  0001 C CNN
+F 0 "#PWR0116" H 10650 2350 50  0001 C CNN
 F 1 "GNDD" H 10650 2450 50  0000 C CNN
 F 2 "" H 10650 2600 50  0000 C CNN
@@
 $EndComp
 $Comp
-L GNDD #PWR0119
+L GNDD #PWR0117
 U 1 1 58DAEBBD
 P 10100 3350
-F 0 "#PWR0119" H 10100 3100 50  0001 C CNN
+F 0 "#PWR0117" H 10100 3100 50  0001 C CNN
 F 1 "GNDD" H 10100 3200 50  0000 C CNN
 F 2 "" H 10100 3350 50  0000 C CNN
@@
 $EndComp
 $Comp
-L GNDD #PWR0120
+L GNDD #PWR0118
 U 1 1 58DAEC64
 P 10575 3350
-F 0 "#PWR0120" H 10575 3100 50  0001 C CNN
+F 0 "#PWR0118" H 10575 3100 50  0001 C CNN
 F 1 "GNDD" H 10575 3200 50  0000 C CNN
 F 2 "" H 10575 3350 50  0000 C CNN
@@
 	4975 4875 5250 4875
 Text HLabel 5250 4875 2    60   BiDi ~ 0
-GPIO1_28
+GPIO1_17
 Wire Wire Line
 	4975 4975 5250 4975
 Text HLabel 5250 4975 2    60   BiDi ~ 0
-GPIO1_28
+GPIO1_27
 Text HLabel 5250 3875 2    60   BiDi ~ 0
 GPIO1_29
@@
 	5400 4775 5700 4775
 $Comp
-L VDD_3V3B #PWR0121
+L VDD_3V3B #PWR0119
 U 1 1 58DB0C91
 P 10100 3050
-F 0 "#PWR0121" H 10100 2900 50  0001 C CNN
+F 0 "#PWR0119" H 10100 2900 50  0001 C CNN
 F 1 "VDD_3V3B" H 10100 3200 50  0000 C CNN
 F 2 "" H 10100 3050 50  0000 C CNN
@@
 $EndComp
 $Comp
-L VDD_3V3B #PWR0122
+L VDD_3V3B #PWR0120
 U 1 1 58DB0D28
 P 10575 3050
-F 0 "#PWR0122" H 10575 2900 50  0001 C CNN
+F 0 "#PWR0120" H 10575 2900 50  0001 C CNN
 F 1 "VDD_3V3B" H 10575 3200 50  0000 C CNN
 F 2 "" H 10575 3050 50  0000 C CNN
@@
 $EndComp
 $Comp
-L GNDD #PWR0123
+L GNDD #PWR0121
 U 1 1 58DB0E3C
 P 10100 4075
-F 0 "#PWR0123" H 10100 3825 50  0001 C CNN
+F 0 "#PWR0121" H 10100 3825 50  0001 C CNN
 F 1 "GNDD" H 10100 3925 50  0000 C CNN
 F 2 "" H 10100 4075 50  0000 C CNN
@@
 $EndComp
 $Comp
-L VDD_3V3B #PWR0124
+L VDD_3V3B #PWR0122
 U 1 1 58DB0E42
 P 10100 3775
-F 0 "#PWR0124" H 10100 3625 50  0001 C CNN
+F 0 "#PWR0122" H 10100 3625 50  0001 C CNN
 F 1 "VDD_3V3B" H 10100 3925 50  0000 C CNN
 F 2 "" H 10100 3775 50  0000 C CNN
@@
 $EndComp
 $Comp
-L GNDD #PWR0125
+L GNDD #PWR0123
 U 1 1 58DB0EE7
 P 10100 4775
-F 0 "#PWR0125" H 10100 4525 50  0001 C CNN
+F 0 "#PWR0123" H 10100 4525 50  0001 C CNN
 F 1 "GNDD" H 10100 4625 50  0000 C CNN
 F 2 "" H 10100 4775 50  0000 C CNN
@@
 $EndComp
 $Comp
-L VDD_3V3B #PWR0126
+L VDD_3V3B #PWR0124
 U 1 1 58DB0EED
 P 10100 4475
-F 0 "#PWR0126" H 10100 4325 50  0001 C CNN
+F 0 "#PWR0124" H 10100 4325 50  0001 C CNN
 F 1 "VDD_3V3B" H 10100 4625 50  0000 C CNN
 F 2 "" H 10100 4475 50  0000 C CNN
@@
 $EndComp
 $Comp
-L GNDD #PWR0127
+L GNDD #PWR0125
 U 1 1 58DB11F2
 P 10575 4075
-F 0 "#PWR0127" H 10575 3825 50  0001 C CNN
+F 0 "#PWR0125" H 10575 3825 50  0001 C CNN
 F 1 "GNDD" H 10575 3925 50  0000 C CNN
 F 2 "" H 10575 4075 50  0000 C CNN
@@
 $EndComp
 $Comp
-L VDD_3V3B #PWR0128
+L VDD_3V3B #PWR0126
 U 1 1 58DB11F8
 P 10575 3775
-F 0 "#PWR0128" H 10575 3625 50  0001 C CNN
+F 0 "#PWR0126" H 10575 3625 50  0001 C CNN
 F 1 "VDD_3V3B" H 10575 3925 50  0000 C CNN
 F 2 "" H 10575 3775 50  0000 C CNN

Commit message: sch updated
Signed-off-by: Pablo Ridolfi <pabloridolfi@outlook.com>
Parts:
- removed IC1: OSD335x, footprints:OSD3358-BAS-BGA400, symbol OSD335x-RESCUE-mateboard
- added IC1: OSD335x, GHI-SoMs-Processors_OSD3358, symbol OSD335x
Connections:
- net GPIO0_26: now also IC1.T11 (GPIO0_26)
- net GPIO0_27: now also IC1.U12 (GPIO0_27)
- net GPIO1_12: now also IC1.T12 (GPIO1_12)
- net GPIO1_13: now also IC1.R12 (GPIO1_13)
- net GPIO1_14: now also IC1.V13 (GPIO1_14)
- net GPIO1_15: now also IC1.U13 (GPIO1_15)
- net GPIO1_17: now also IC1.V14 (GPIO1_17)
- net GPIO1_25: now also IC1.U16 ((HDMI_INT)GPIO1_25)
- net GPIO1_27: now also IC1.V17 ((HDMICLK_DISN)GPIO1_27)
- net GPIO1_28: now also IC1.U18 (GPIO1_28)
- net GPIO1_29: now also IC1.V6 (GPIO1_29)
- net GPIO2_0: now also IC1.T13 (GPIO2_0)
- net GPIO2_1: now also IC1.V12 (GPIO2_1)
- net JTAG_EMU0: now also IC1.C14 (JTAG_EMU0)
- net JTAG_EMU1: now also IC1.B14 (JTAG_EMU1)
- net JTAG_TCK: now also IC1.A12 (JTAG_TCK)
- net JTAG_TDI: now also IC1.B11 (JTAG_TDI)
- net JTAG_TDO: now also IC1.A11 (JTAG_TDO)
- net JTAG_TMS: now also IC1.C11 (JTAG_TMS)
- net JTAG_TRSTn: now also IC1.B10 (JTAG_TRSTN)
- net LDO_PGOOD: now also IC1.B5 (RTC_PORZ)
- net MMC1_CLK: now also IC1.U9 (MMC1_CLK)
- net MMC1_CMD: now also IC1.V9 (MMC1_CMD)
- net MMC1_DAT0: now also IC1.U7 (MMC1_DAT0)
- net MMC1_DAT1: now also IC1.V7 (MMC1_DAT1)
- net MMC1_DAT2: now also IC1.R8 (MMC1_DAT2)
- net MMC1_DAT3: now also IC1.T8 (MMC1_DAT3)
- net MMC1_DAT4: now also IC1.U8 (MMC1_DAT4)
- net MMC1_DAT5: now also IC1.V8 (MMC1_DAT5)
- net MMC1_DAT6: now also IC1.R9 (MMC1_DAT6)
- net MMC1_DAT7: now also IC1.T9 (MMC1_DAT7)
- net PMIC_INT: now also IC1.B18 (EXTIN)
- net PMIC_PGOOD: now also IC1.B15 (PORZ)
- net PMIC_nWAKEUP: now also IC1.C5 (EXT_WAKEUP)
- net SD.CD: now also IC1.C15 (MMC0_CD)
- net SD.CLK: now also IC1.G17 (MMC0_CLK0)
- net SD.CMD: now also IC1.G18 (MMC0_CMD)
- net SD.D0: now also IC1.G16 (MMC0_DAT0)
- net SD.D1: now also IC1.G15 (MMC0_DAT1)
- net SD.D2: now also IC1.F18 (MMC0_DAT2)
- net SD.D3: now also IC1.F17 (MMC0_DAT3)
- net SYS_RESETn: now also IC1.A10 (SYS_RESETN)
- net TIMER4: now also IC1.R7 (TIMER4)
- net TIMER5: now also IC1.T6 (TIMER5)
- net TIMER6: now also IC1.U6 (TIMER6)
- net TIMER7: now also IC1.T7 (TIMER7)
- net UART4_RXD: now also IC1.T17 (UART4_RXD)
- net UART4_TXD: now also IC1.U17 (UART4_TXD)
- net USB1_OCn: now also IC1.T16 ((USB1_OCN)GPIO1_26)
- net USR0: now also IC1.V15 (USR0)
- net USR1: now also IC1.U15 (USR1)
- net USR2: now also IC1.T15 (USR2)
- net USR3: now also IC1.V16 (USR3)
- net eHRPWM1A: now also IC1.U14 (EHRPWM1A)
- net eHRPWM1B: now also IC1.T14 (EHRPWM1B)
- net eHRPWM2A: now also IC1.U10 (EHRPWM2A)
- net eHRPWM2B: now also IC1.T10 (EHRPWM2B)
- net at C16.1, R31.1, Y1.1: now also IC1.M20 (OSC0_IN)
- net at C17.1, R31.2, Y1.2: now also IC1.K20 (OSC0_OUT)
- net at C16.2, C17.2: now also IC1.L20 (DGND0)
- net at L5.2: now also IC1.D14 (CLKOUT2)
- net at L4.2: now also IC1.A15 (CLKOUT1)
- net at R33.2: now also IC1.D13 (GPIO3_20)
- net at C19.1, R32.2, Y2.2: now also IC1.F20 (OSC1_OUT)
- net at C18.2, C19.2: now also IC1.G20 (DGND1)
- net at C18.1, R32.1, Y2.1: now also IC1.H20 (OSC1_IN)
- net at R34.2: now also IC1.R13 (GPIO1_16)
- net at U8.2: now also IC1.R14 ((EMMC_RSTN)GPIO1_20)
Changed lines of the file:
@@
 Wire Wire Line
 	5900 1475 6400 1475
-$Comp
-L OSD335x-RESCUE-mateboard IC1
-U 1 1 58D2CE56
-P 3775 3075
-AR Path="/58D2CE56" Ref="IC1"  Part="1"
-AR Path="/58AC1B74/58D2CE56" Ref="IC1"  Part="1"
-F 0 "IC1" H 3700 3100 45  0000 L BNN
-F 1 "OSD335x" H 3625 3000 45  0000 L BNN
-F 2 "footprints:OSD3358-BAS-BGA400" H 3805 3225 20  0001 C CNN
-F 3 "" H 3775 3075 60  0001 C CNN
-	1    3775 3075
-	1    0    0    -1
-$EndComp
 Wire Wire Line
 	750  1175 2575 1175
@@
 Text HLabel 5250 5275 2    60   BiDi ~ 0
 GPIO2_0
+$Comp
+L OSD335x IC1
+U 1 1 594B5AA6
+P 3775 3075
+AR Path="/594B5AA6" Ref="IC1"  Part="1"
+AR Path="/58AC1B74/594B5AA6" Ref="IC1"  Part="1"
+F 0 "IC1" H 3775 5529 45  0000 C CNN
+F 1 "OSD335x" H 3775 5445 45  0000 C CNN
+F 2 "GHI-SoMs-Processors_OSD3358" H 3805 3225 20  0001 C CNN
+F 3 "" H 3775 3075 60  0001 C CNN
+	1    3775 3075
+	1    0    0    -1
+$EndComp
 $EndSCHEMATC

Commit message: footprints updated, add power led
Signed-off-by: Pablo Ridolfi <pabloridolfi@outlook.com>
Parts:
- IC1: footprint GHI-SoMs-Processors_OSD3358 -> footprints:OSD3358-BAS-BGA400
- IC3: footprint footprints:WFBGA153 -> footprints:BeagleBone_Blue-GHI-IC_MICRON_EMMC_153_MODIFICADO
Changed lines of the file:
@@
 F 0 "IC3" H 8350 3825 60  0000 C CNN
 F 1 "NAND_4GB" H 8525 2525 60  0000 C CNN
-F 2 "footprints:WFBGA153" H 8275 3225 60  0001 C CNN
+F 2 "footprints:BeagleBone_Blue-GHI-IC_MICRON_EMMC_153_MODIFICADO" H 8275 3225 60  0001 C CNN
 F 3 "" H 8275 3225 60  0001 C CNN
 	1    8275 3225
@@
 F 0 "IC1" H 3775 5529 45  0000 C CNN
 F 1 "OSD335x" H 3775 5445 45  0000 C CNN
-F 2 "GHI-SoMs-Processors_OSD3358" H 3805 3225 20  0001 C CNN
+F 2 "footprints:OSD3358-BAS-BGA400" H 3805 3225 20  0001 C CNN
 F 3 "" H 3775 3075 60  0001 C CNN
 	1    3775 3075
