File: ddr.sch (KiCad schematic (older format))
At the start: 27 parts, among them IC2 AM335X_ZCZ, IC3 DDR3_SDRAM

Commit message: erc passed, sch first version
Changed lines of the file:
@@
 DDR_D15
 $Comp
-L VDDS_DDR #PWR100
+L VDDS_DDR #PWR0104
 U 1 1 58AC4CB7
 P 5900 1750
-F 0 "#PWR100" H 5900 1600 50  0001 C CNN
+F 0 "#PWR0104" H 5900 1600 50  0001 C CNN
 F 1 "VDDS_DDR" H 5900 1900 50  0000 C CNN
 F 2 "" H 5900 1750 50  0000 C CNN
@@
 DDR_A15
 $Comp
-L GNDD #PWR101
+L GNDD #PWR0105
 U 1 1 58AC5047
 P 5900 5725
-F 0 "#PWR101" H 5900 5475 50  0001 C CNN
+F 0 "#PWR0105" H 5900 5475 50  0001 C CNN
 F 1 "GNDD" H 5900 5575 50  0000 C CNN
 F 2 "" H 5900 5725 50  0000 C CNN
@@
 $EndComp
 $Comp
-L VDDS_DDR #PWR106
+L VDDS_DDR #PWR0106
 U 1 1 58AC6BD8
 P 8000 4400
-F 0 "#PWR106" H 8000 4250 50  0001 C CNN
+F 0 "#PWR0106" H 8000 4250 50  0001 C CNN
 F 1 "VDDS_DDR" V 8000 4725 50  0000 C CNN
 F 2 "" H 8000 4400 50  0000 C CNN
@@
 $EndComp
 $Comp
-L GNDD #PWR99
+L GNDD #PWR0107
 U 1 1 58AC6E23
 P 3875 4600
-F 0 "#PWR99" H 3875 4350 50  0001 C CNN
+F 0 "#PWR0107" H 3875 4350 50  0001 C CNN
 F 1 "GNDD" V 3875 4375 50  0000 C CNN
 F 2 "" H 3875 4600 50  0000 C CNN
@@
 $EndComp
 $Comp
-L GNDD #PWR103
+L GNDD #PWR0108
 U 1 1 58AC7DFA
 P 7450 5050
-F 0 "#PWR103" H 7450 4800 50  0001 C CNN
+F 0 "#PWR0108" H 7450 4800 50  0001 C CNN
 F 1 "GNDD" V 7450 4825 50  0000 C CNN
 F 2 "" H 7450 5050 50  0000 C CNN
@@
 $EndComp
 $Comp
-L DDR_VREF #PWR114
+L DDR_VREF #PWR0109
 U 1 1 58AB68A2
 P 8825 4625
-F 0 "#PWR114" H 8825 4475 50  0001 C CNN
+F 0 "#PWR0109" H 8825 4475 50  0001 C CNN
 F 1 "DDR_VREF" H 8825 4775 50  0000 C CNN
 F 2 "" H 8825 4625 50  0000 C CNN
@@
 Connection ~ 8100 4650
 $Comp
-L GNDD #PWR107
+L GNDD #PWR0110
 U 1 1 58AB6B33
 P 8100 5000
-F 0 "#PWR107" H 8100 4750 50  0001 C CNN
+F 0 "#PWR0110" H 8100 4750 50  0001 C CNN
 F 1 "GNDD" H 8100 4850 50  0000 C CNN
 F 2 "" H 8100 5000 50  0000 C CNN
@@
 Connection ~ 8675 4650
 $Comp
-L GNDD #PWR110
+L GNDD #PWR0111
 U 1 1 58AB6D24
 P 8675 5000
-F 0 "#PWR110" H 8675 4750 50  0001 C CNN
+F 0 "#PWR0111" H 8675 4750 50  0001 C CNN
 F 1 "GNDD" H 8675 4850 50  0000 C CNN
 F 2 "" H 8675 5000 50  0000 C CNN
@@
 $EndComp
 $Comp
-L GNDD #PWR115
+L GNDD #PWR0112
 U 1 1 58AB6FFD
 P 8975 5000
-F 0 "#PWR115" H 8975 4750 50  0001 C CNN
+F 0 "#PWR0112" H 8975 4750 50  0001 C CNN
 F 1 "GNDD" H 8975 4850 50  0000 C CNN
 F 2 "" H 8975 5000 50  0000 C CNN
@@
 Connection ~ 8975 4650
 $Comp
-L VDDS_DDR #PWR122
+L VDDS_DDR #PWR0113
 U 1 1 58AB71F0
 P 9775 4650
-F 0 "#PWR122" H 9775 4500 50  0001 C CNN
+F 0 "#PWR0113" H 9775 4500 50  0001 C CNN
 F 1 "VDDS_DDR" H 9775 4800 50  0000 C CNN
 F 2 "" H 9775 4650 50  0000 C CNN
@@
 $EndComp
 $Comp
-L GNDD #PWR104
+L GNDD #PWR0114
 U 1 1 58AB7EB8
 P 7475 1500
-F 0 "#PWR104" H 7475 1250 50  0001 C CNN
+F 0 "#PWR0114" H 7475 1250 50  0001 C CNN
 F 1 "GNDD" H 7475 1350 50  0000 C CNN
 F 2 "" H 7475 1500 50  0000 C CNN
@@
 $EndComp
 $Comp
-L GNDD #PWR105
+L GNDD #PWR0115
 U 1 1 58AB7EBE
 P 7800 1500
-F 0 "#PWR105" H 7800 1250 50  0001 C CNN
+F 0 "#PWR0115" H 7800 1250 50  0001 C CNN
 F 1 "GNDD" H 7800 1350 50  0000 C CNN
 F 2 "" H 7800 1500 50  0000 C CNN
@@
 $EndComp
 $Comp
-L GNDD #PWR102
+L GNDD #PWR0116
 U 1 1 58AB7EC4
 P 7150 1500
-F 0 "#PWR102" H 7150 1250 50  0001 C CNN
+F 0 "#PWR0116" H 7150 1250 50  0001 C CNN
 F 1 "GNDD" H 7150 1350 50  0000 C CNN
 F 2 "" H 7150 1500 50  0000 C CNN
@@
 $EndComp
 $Comp
-L GNDD #PWR108
+L GNDD #PWR0117
 U 1 1 58AB7ECA
 P 8125 1500
-F 0 "#PWR108" H 8125 1250 50  0001 C CNN
+F 0 "#PWR0117" H 8125 1250 50  0001 C CNN
 F 1 "GNDD" H 8125 1350 50  0000 C CNN
 F 2 "" H 8125 1500 50  0000 C CNN
@@
 $EndComp
 $Comp
-L GNDD #PWR116
+L GNDD #PWR0118
 U 1 1 58AB7ED0
 P 9100 1500
-F 0 "#PWR116" H 9100 1250 50  0001 C CNN
+F 0 "#PWR0118" H 9100 1250 50  0001 C CNN
 F 1 "GNDD" H 9100 1350 50  0000 C CNN
 F 2 "" H 9100 1500 50  0000 C CNN
@@
 $EndComp
 $Comp
-L GNDD #PWR119
+L GNDD #PWR0119
 U 1 1 58AB7ED6
 P 9425 1500
-F 0 "#PWR119" H 9425 1250 50  0001 C CNN
+F 0 "#PWR0119" H 9425 1250 50  0001 C CNN
 F 1 "GNDD" H 9425 1350 50  0000 C CNN
 F 2 "" H 9425 1500 50  0000 C CNN
@@
 $EndComp
 $Comp
-L GNDD #PWR109
+L GNDD #PWR0120
 U 1 1 58AB7EDC
 P 8450 1500
-F 0 "#PWR109" H 8450 1250 50  0001 C CNN
+F 0 "#PWR0120" H 8450 1250 50  0001 C CNN
 F 1 "GNDD" H 8450 1350 50  0000 C CNN
 F 2 "" H 8450 1500 50  0000 C CNN
@@
 $EndComp
 $Comp
-L GNDD #PWR112
+L GNDD #PWR0121
 U 1 1 58AB7EE2
 P 8775 1500
-F 0 "#PWR112" H 8775 1250 50  0001 C CNN
+F 0 "#PWR0121" H 8775 1250 50  0001 C CNN
 F 1 "GNDD" H 8775 1350 50  0000 C CNN
 F 2 "" H 8775 1500 50  0000 C CNN
@@
 $EndComp
 $Comp
-L GNDD #PWR124
+L GNDD #PWR0122
 U 1 1 58AB7EE8
 P 10075 1500
-F 0 "#PWR124" H 10075 1250 50  0001 C CNN
+F 0 "#PWR0122" H 10075 1250 50  0001 C CNN
 F 1 "GNDD" H 10075 1350 50  0000 C CNN
 F 2 "" H 10075 1500 50  0000 C CNN
@@
 $EndComp
 $Comp
-L GNDD #PWR126
+L GNDD #PWR0123
 U 1 1 58AB7EEE
 P 10400 1500
-F 0 "#PWR126" H 10400 1250 50  0001 C CNN
+F 0 "#PWR0123" H 10400 1250 50  0001 C CNN
 F 1 "GNDD" H 10400 1350 50  0000 C CNN
 F 2 "" H 10400 1500 50  0000 C CNN
@@
 $EndComp
 $Comp
-L GNDD #PWR121
+L GNDD #PWR0124
 U 1 1 58AB7EF4
 P 9750 1500
-F 0 "#PWR121" H 9750 1250 50  0001 C CNN
+F 0 "#PWR0124" H 9750 1250 50  0001 C CNN
 F 1 "GNDD" H 9750 1350 50  0000 C CNN
 F 2 "" H 9750 1500 50  0000 C CNN
@@
 Connection ~ 8450 1100
 $Comp
-L VDDS_DDR #PWR111
+L VDDS_DDR #PWR0125
 U 1 1 58AB90C3
 P 8775 1050
-F 0 "#PWR111" H 8775 900 50  0001 C CNN
+F 0 "#PWR0125" H 8775 900 50  0001 C CNN
 F 1 "VDDS_DDR" H 8775 1200 50  0000 C CNN
 F 2 "" H 8775 1050 50  0000 C CNN
@@
 	2225 6200 2100 6200
 $Comp
-L GNDD #PWR96
+L GNDD #PWR0126
 U 1 1 58AB9DDF
 P 2225 6575
-F 0 "#PWR96" H 2225 6325 50  0001 C CNN
+F 0 "#PWR0126" H 2225 6325 50  0001 C CNN
 F 1 "GNDD" H 2225 6425 50  0000 C CNN
 F 2 "" H 2225 6575 50  0000 C CNN
@@
 $EndComp
 $Comp
-L GNDD #PWR97
+L GNDD #PWR0127
 U 1 1 58ABA2AF
 P 2750 6400
-F 0 "#PWR97" H 2750 6150 50  0001 C CNN
+F 0 "#PWR0127" H 2750 6150 50  0001 C CNN
 F 1 "GNDD" H 2750 6250 50  0000 C CNN
 F 2 "" H 2750 6400 50  0000 C CNN
@@
 $EndComp
 Wire Wire Line
-	2750 6100 2750 6050
+	2750 6025 2750 6100
 Wire Wire Line
 	2100 6050 2800 6050
 $Comp
-L DDR_VREF #PWR98
+L DDR_VREF #PWR0128
 U 1 1 58ABA60D
 P 2800 6050
-F 0 "#PWR98" H 2800 5900 50  0001 C CNN
+F 0 "#PWR0128" H 2800 5900 50  0001 C CNN
 F 1 "DDR_VREF" V 2800 6350 50  0000 C CNN
 F 2 "" H 2800 6050 50  0000 C CNN
@@
 $EndComp
 $Comp
-L GNDD #PWR113
+L GNDD #PWR0129
 U 1 1 58ABC703
 P 8800 2475
-F 0 "#PWR113" H 8800 2225 50  0001 C CNN
+F 0 "#PWR0129" H 8800 2225 50  0001 C CNN
 F 1 "GNDD" H 8800 2325 50  0000 C CNN
 F 2 "" H 8800 2475 50  0000 C CNN
@@
 $EndComp
 $Comp
-L GNDD #PWR118
+L GNDD #PWR0130
 U 1 1 58ABC709
 P 9100 2475
-F 0 "#PWR118" H 9100 2225 50  0001 C CNN
+F 0 "#PWR0130" H 9100 2225 50  0001 C CNN
 F 1 "GNDD" H 9100 2325 50  0000 C CNN
 F 2 "" H 9100 2475 50  0000 C CNN
@@
 $EndComp
 $Comp
-L GNDD #PWR125
+L GNDD #PWR0131
 U 1 1 58ABC70F
 P 10125 2475
-F 0 "#PWR125" H 10125 2225 50  0001 C CNN
+F 0 "#PWR0131" H 10125 2225 50  0001 C CNN
 F 1 "GNDD" H 10125 2325 50  0000 C CNN
 F 2 "" H 10125 2475 50  0000 C CNN
@@
 $EndComp
 $Comp
-L GNDD #PWR120
+L GNDD #PWR0132
 U 1 1 58ABC715
 P 9475 2475
-F 0 "#PWR120" H 9475 2225 50  0001 C CNN
+F 0 "#PWR0132" H 9475 2225 50  0001 C CNN
 F 1 "GNDD" H 9475 2325 50  0000 C CNN
 F 2 "" H 9475 2475 50  0000 C CNN
@@
 $EndComp
 $Comp
-L GNDD #PWR123
+L GNDD #PWR0133
 U 1 1 58ABC71B
 P 9800 2475
-F 0 "#PWR123" H 9800 2225 50  0001 C CNN
+F 0 "#PWR0133" H 9800 2225 50  0001 C CNN
 F 1 "GNDD" H 9800 2325 50  0000 C CNN
 F 2 "" H 9800 2475 50  0000 C CNN
@@
 Connection ~ 9800 2050
 $Comp
-L VDDS_DDR #PWR117
+L VDDS_DDR #PWR0134
 U 1 1 58ABCEAC
 P 9100 2000
-F 0 "#PWR117" H 9100 1850 50  0001 C CNN
+F 0 "#PWR0134" H 9100 1850 50  0001 C CNN
 F 1 "VDDS_DDR" H 9100 2150 50  0000 C CNN
 F 2 "" H 9100 2000 50  0000 C CNN
@@
 Text Notes 8325 5350 0    60   ~ 0
 high precision resistors, see am335x datasheet
+$Comp
+L PWR_FLAG #FLG0135
+U 1 1 58C6871C
+P 2750 6025
+F 0 "#FLG0135" H 2750 6100 50  0001 C CNN
+F 1 "PWR_FLAG" H 2750 6175 50  0001 C CNN
+F 2 "" H 2750 6025 50  0001 C CNN
+F 3 "" H 2750 6025 50  0001 C CNN
+	1    2750 6025
+	1    0    0    -1
+$EndComp
 $EndSCHEMATC
