File: sysboot.sch (KiCad schematic (older format))
At the start: 19 parts

Commit message: gpio assignment done
Other:
- note added: "0 1 2 3 4 5 6 7 8 9 0 1 2 3 4 5\n0 0 x 1 1 1 0 0 0 0 0 0 0 0 1 0"
Changed lines of the file:
@@
 $Descr A4 11693 8268
 encoding utf-8
-Sheet 10 10
+Sheet 9 10
 Title ""
 Date ""
@@
 Wire Wire Line
 	6250 4350 6150 4350
+Text Notes 8550 4425 0    60   ~ 0
+0 1 2 3 4 5 6 7 8 9 0 1 2 3 4 5\n0 0 x 1 1 1 0 0 0 0 0 0 0 0 1 0
 $EndSCHEMATC

Commit message: annotation, wip erc
Parts:
- gave numbers to parts that had none: 19
Changed lines of the file:
@@
 AR Path="/58BD44E1" Ref="IC?"  Part="8"
 AR Path="/589C7F89/58BD44E1" Ref="IC?"  Part="8"
-AR Path="/58BD360A/58BD44E1" Ref="IC?"  Part="8"
-F 0 "IC?" H 1250 4500 60  0000 C CNN
+AR Path="/58BD360A/58BD44E1" Ref="IC2"  Part="8"
+F 0 "IC2" H 1250 4500 60  0000 C CNN
 F 1 "AM335X_ZCZ" H 1925 4500 60  0000 C CNN
 F 2 "" H 1150 3400 60  0001 C CNN
@@
 SYS_BOOT0
 $Comp
-L R R?
+L R R93
 U 1 1 58BD4B7B
 P 6800 4600
-F 0 "R?" V 6750 4750 50  0000 C CNN
+F 0 "R93" V 6750 4750 50  0000 C CNN
 F 1 "100k" V 6800 4600 50  0000 C CNN
 F 2 "" V 6730 4600 50  0001 C CNN
@@
 $EndComp
 $Comp
-L R R?
+L R R94
 U 1 1 58BD5FFA
 P 6900 4600
-F 0 "R?" V 6850 4750 50  0000 C CNN
+F 0 "R94" V 6850 4750 50  0000 C CNN
 F 1 "100k" V 6900 4600 50  0000 C CNN
 F 2 "" V 6830 4600 50  0001 C CNN
@@
 $EndComp
 $Comp
-L R R?
+L R R95
 U 1 1 58BD60B0
 P 7000 2200
-F 0 "R?" V 6950 2350 50  0000 C CNN
+F 0 "R95" V 6950 2350 50  0000 C CNN
 F 1 "100k" V 7000 2200 50  0000 C CNN
 F 2 "" V 6930 2200 50  0001 C CNN
@@
 $EndComp
 $Comp
-L R R?
+L R R96
 U 1 1 58BD60BC
 P 7100 2200
-F 0 "R?" V 7050 2350 50  0000 C CNN
+F 0 "R96" V 7050 2350 50  0000 C CNN
 F 1 "100k" V 7100 2200 50  0000 C CNN
 F 2 "" V 7030 2200 50  0001 C CNN
@@
 $EndComp
 $Comp
-L R R?
+L R R98
 U 1 1 58BD6460
 P 7300 2200
-F 0 "R?" V 7250 2350 50  0000 C CNN
+F 0 "R98" V 7250 2350 50  0000 C CNN
 F 1 "100k" V 7300 2200 50  0000 C CNN
 F 2 "" V 7230 2200 50  0001 C CNN
@@
 $EndComp
 $Comp
-L R R?
+L R R99
 U 1 1 58BD6472
 P 7400 4600
-F 0 "R?" V 7350 4750 50  0000 C CNN
+F 0 "R99" V 7350 4750 50  0000 C CNN
 F 1 "100k" V 7400 4600 50  0000 C CNN
 F 2 "" V 7330 4600 50  0001 C CNN
@@
 $EndComp
 $Comp
-L R R?
+L R R100
 U 1 1 58BD6478
 P 7500 4600
-F 0 "R?" V 7450 4750 50  0000 C CNN
+F 0 "R100" V 7450 4750 50  0000 C CNN
 F 1 "100k" V 7500 4600 50  0000 C CNN
 F 2 "" V 7430 4600 50  0001 C CNN
@@
 $EndComp
 $Comp
-L R R?
+L R R97
 U 1 1 58BD647E
 P 7200 2200
-F 0 "R?" V 7150 2350 50  0000 C CNN
+F 0 "R97" V 7150 2350 50  0000 C CNN
 F 1 "100k" V 7200 2200 50  0000 C CNN
 F 2 "" V 7130 2200 50  0001 C CNN
@@
 $EndComp
 $Comp
-L R R?
+L R R101
 U 1 1 58BD69A4
 P 7600 4600
-F 0 "R?" V 7550 4750 50  0000 C CNN
+F 0 "R101" V 7550 4750 50  0000 C CNN
 F 1 "100k" V 7600 4600 50  0000 C CNN
 F 2 "" V 7530 4600 50  0001 C CNN
@@
 $EndComp
 $Comp
-L R R?
+L R R102
 U 1 1 58BD69B0
 P 7700 4600
-F 0 "R?" V 7650 4750 50  0000 C CNN
+F 0 "R102" V 7650 4750 50  0000 C CNN
 F 1 "100k" V 7700 4600 50  0000 C CNN
 F 2 "" V 7630 4600 50  0001 C CNN
@@
 $EndComp
 $Comp
-L R R?
+L R R103
 U 1 1 58BD69BC
 P 7800 4600
-F 0 "R?" V 7750 4750 50  0000 C CNN
+F 0 "R103" V 7750 4750 50  0000 C CNN
 F 1 "100k" V 7800 4600 50  0000 C CNN
 F 2 "" V 7730 4600 50  0001 C CNN
@@
 $EndComp
 $Comp
-L R R?
+L R R104
 U 1 1 58BD69C2
 P 7900 4600
-F 0 "R?" V 7850 4750 50  0000 C CNN
+F 0 "R104" V 7850 4750 50  0000 C CNN
 F 1 "100k" V 7900 4600 50  0000 C CNN
 F 2 "" V 7830 4600 50  0001 C CNN
@@
 $EndComp
 $Comp
-L R R?
+L R R105
 U 1 1 58BD69D4
 P 8000 4600
-F 0 "R?" V 7950 4750 50  0000 C CNN
+F 0 "R105" V 7950 4750 50  0000 C CNN
 F 1 "100k" V 8000 4600 50  0000 C CNN
 F 2 "" V 7930 4600 50  0001 C CNN
@@
 $EndComp
 $Comp
-L R R?
+L R R106
 U 1 1 58BD69E0
 P 8100 4600
-F 0 "R?" V 8050 4750 50  0000 C CNN
+F 0 "R106" V 8050 4750 50  0000 C CNN
 F 1 "100k" V 8100 4600 50  0000 C CNN
 F 2 "" V 8030 4600 50  0001 C CNN
@@
 $EndComp
 $Comp
-L R R?
+L R R107
 U 1 1 58BD69E6
 P 8200 2200
-F 0 "R?" V 8150 2350 50  0000 C CNN
+F 0 "R107" V 8150 2350 50  0000 C CNN
 F 1 "100k" V 8200 2200 50  0000 C CNN
 F 2 "" V 8130 2200 50  0001 C CNN
@@
 $EndComp
 $Comp
-L R R?
+L R R108
 U 1 1 58BD69F2
 P 8300 4600
-F 0 "R?" V 8250 4750 50  0000 C CNN
+F 0 "R108" V 8250 4750 50  0000 C CNN
 F 1 "100k" V 8300 4600 50  0000 C CNN
 F 2 "" V 8230 4600 50  0001 C CNN
@@
 $EndComp
 Wire Wire Line
-	6800 4750 6800 4925
+	6800 4750 6800 4850
+Wire Wire Line
+	6800 4850 6800 4925
 Wire Wire Line
 	8300 4850 8300 4750
@@
 Connection ~ 6900 4850
 Wire Wire Line
-	6800 4850 8300 4850
+	6800 4850 6900 4850
+Wire Wire Line
+	6900 4850 7400 4850
+Wire Wire Line
+	7400 4850 7500 4850
+Wire Wire Line
+	7500 4850 7600 4850
+Wire Wire Line
+	7600 4850 7700 4850
+Wire Wire Line
+	7700 4850 7800 4850
+Wire Wire Line
+	7800 4850 7900 4850
+Wire Wire Line
+	7900 4850 8000 4850
+Wire Wire Line
+	8000 4850 8100 4850
+Wire Wire Line
+	8100 4850 8300 4850
 Wire Wire Line
 	8200 1950 8200 2050
@@
 Connection ~ 7100 1950
 Wire Wire Line
-	7000 1900 7000 2050
+	7000 1900 7000 1950
+Wire Wire Line
+	7000 1950 7000 2050
 Connection ~ 7000 1950
 $Comp
-L VDD_3V3B #PWR?
+L VDD_3V3B #PWR299
 U 1 1 58BD7134
 P 7000 1900
-F 0 "#PWR?" H 7000 1750 50  0001 C CNN
+F 0 "#PWR299" H 7000 1750 50  0001 C CNN
 F 1 "VDD_3V3B" H 7000 2050 50  0000 C CNN
 F 2 "" H 7000 1900 50  0000 C CNN
@@
 $EndComp
 $Comp
-L GNDD #PWR?
+L GNDD #PWR298
 U 1 1 58BD73F7
 P 6800 4925
-F 0 "#PWR?" H 6800 4675 50  0001 C CNN
+F 0 "#PWR298" H 6800 4675 50  0001 C CNN
 F 1 "GNDD" H 6800 4775 50  0000 C CNN
 F 2 "" H 6800 4925 50  0001 C CNN
@@
 	6900 2550 6150 2550
 Wire Wire Line
-	6150 2650 8425 2650
+	6150 2650 7000 2650
+Wire Wire Line
+	7000 2650 8425 2650
 Connection ~ 7000 2650
 Wire Wire Line
@@
 	8300 3950 6150 3950
 $Comp
-L PushButton S?
+L PushButton S3
 U 1 1 58BDE34C
 P 9175 2650
-F 0 "S?" H 9175 2450 60  0000 C CNN
+F 0 "S3" H 9175 2450 60  0000 C CNN
 F 1 "microSD Boot" H 9200 2550 60  0000 C CNN
 F 2 "" H 9175 2650 60  0001 C CNN
@@
 $EndComp
 $Comp
-L GNDD #PWR?
+L GNDD #PWR300
 U 1 1 58BDE353
 P 9525 2650
-F 0 "#PWR?" H 9525 2400 50  0001 C CNN
+F 0 "#PWR300" H 9525 2400 50  0001 C CNN
 F 1 "GNDD" V 9525 2450 50  0000 C CNN
 F 2 "" H 9525 2650 50  0000 C CNN
@@
 $EndComp
 $Comp
-L R R?
+L R R109
 U 1 1 58BDE507
 P 8575 2650
-F 0 "R?" V 8655 2650 50  0000 C CNN
+F 0 "R109" V 8655 2650 50  0000 C CNN
 F 1 "100" V 8575 2650 50  0000 C CNN
 F 2 "" V 8505 2650 50  0001 C CNN
@@
 	7200 2850 7200 2350
 Wire Wire Line
-	8200 1950 7000 1950
-Text HLabel 6250 4050 2    60   BiDi ~ 0
+	8200 1950 7300 1950
+Wire Wire Line
+	7300 1950 7200 1950
+Wire Wire Line
+	7200 1950 7100 1950
+Wire Wire Line
+	7100 1950 7000 1950
+Text HLabel 8400 4050 2    60   BiDi ~ 0
 GPIO2_23
 Wire Wire Line
-	6250 4050 6150 4050
-Text HLabel 6250 4150 2    60   BiDi ~ 0
+	8400 4050 6150 4050
+Text HLabel 8400 4150 2    60   BiDi ~ 0
 GPIO2_22
 Wire Wire Line
-	6250 4150 6150 4150
-Text HLabel 6250 4250 2    60   BiDi ~ 0
+	8400 4150 6150 4150
+Text HLabel 8400 4250 2    60   BiDi ~ 0
 GPIO2_24
 Wire Wire Line
-	6250 4250 6150 4250
-Text HLabel 6250 4350 2    60   BiDi ~ 0
+	8400 4250 6150 4250
+Text HLabel 8400 4350 2    60   BiDi ~ 0
 GPIO2_25
 Wire Wire Line
-	6250 4350 6150 4350
-Text Notes 8550 4425 0    60   ~ 0
+	8400 4350 6150 4350
+Text Notes 6750 5375 0    60   ~ 0
 0 1 2 3 4 5 6 7 8 9 0 1 2 3 4 5\n0 0 x 1 1 1 0 0 0 0 0 0 0 0 1 0
 $EndSCHEMATC

Commit message: erc passed, sch first version
Changed lines of the file:
@@
 $EndComp
 Wire Wire Line
-	6800 4750 6800 4850
-Wire Wire Line
-	6800 4850 6800 4925
+	6800 4750 6800 4925
 Wire Wire Line
 	8300 4850 8300 4750
@@
 Connection ~ 6900 4850
 Wire Wire Line
-	6800 4850 6900 4850
-Wire Wire Line
-	6900 4850 7400 4850
-Wire Wire Line
-	7400 4850 7500 4850
-Wire Wire Line
-	7500 4850 7600 4850
-Wire Wire Line
-	7600 4850 7700 4850
-Wire Wire Line
-	7700 4850 7800 4850
-Wire Wire Line
-	7800 4850 7900 4850
-Wire Wire Line
-	7900 4850 8000 4850
-Wire Wire Line
-	8000 4850 8100 4850
-Wire Wire Line
-	8100 4850 8300 4850
+	6800 4850 8300 4850
 Wire Wire Line
 	8200 1950 8200 2050
@@
 Connection ~ 7100 1950
 Wire Wire Line
-	7000 1900 7000 1950
-Wire Wire Line
-	7000 1950 7000 2050
+	7000 1900 7000 2050
 Connection ~ 7000 1950
 $Comp
-L VDD_3V3B #PWR299
+L VDD_3V3B #PWR0318
 U 1 1 58BD7134
 P 7000 1900
-F 0 "#PWR299" H 7000 1750 50  0001 C CNN
+F 0 "#PWR0318" H 7000 1750 50  0001 C CNN
 F 1 "VDD_3V3B" H 7000 2050 50  0000 C CNN
 F 2 "" H 7000 1900 50  0000 C CNN
@@
 $EndComp
 $Comp
-L GNDD #PWR298
+L GNDD #PWR0319
 U 1 1 58BD73F7
 P 6800 4925
-F 0 "#PWR298" H 6800 4675 50  0001 C CNN
+F 0 "#PWR0319" H 6800 4675 50  0001 C CNN
 F 1 "GNDD" H 6800 4775 50  0000 C CNN
 F 2 "" H 6800 4925 50  0001 C CNN
@@
 	6900 2550 6150 2550
 Wire Wire Line
-	6150 2650 7000 2650
-Wire Wire Line
-	7000 2650 8425 2650
+	6150 2650 8425 2650
 Connection ~ 7000 2650
 Wire Wire Line
@@
 $EndComp
 $Comp
-L GNDD #PWR300
+L GNDD #PWR0320
 U 1 1 58BDE353
 P 9525 2650
-F 0 "#PWR300" H 9525 2400 50  0001 C CNN
+F 0 "#PWR0320" H 9525 2400 50  0001 C CNN
 F 1 "GNDD" V 9525 2450 50  0000 C CNN
 F 2 "" H 9525 2650 50  0000 C CNN
@@
 	7200 2850 7200 2350
 Wire Wire Line
-	8200 1950 7300 1950
-Wire Wire Line
-	7300 1950 7200 1950
-Wire Wire Line
-	7200 1950 7100 1950
-Wire Wire Line
-	7100 1950 7000 1950
+	7000 1950 8200 1950
 Text HLabel 8400 4050 2    60   BiDi ~ 0
 GPIO2_23

Commit message: wip display connector
Changed lines of the file:
@@
 $EndComp
 Wire Wire Line
-	6800 4750 6800 4925
+	6800 4750 6800 4850
+Wire Wire Line
+	6800 4850 6800 4925
 Wire Wire Line
 	8300 4850 8300 4750
@@
 Connection ~ 6900 4850
 Wire Wire Line
-	6800 4850 8300 4850
+	6800 4850 6900 4850
+Wire Wire Line
+	6900 4850 7400 4850
+Wire Wire Line
+	7400 4850 7500 4850
+Wire Wire Line
+	7500 4850 7600 4850
+Wire Wire Line
+	7600 4850 7700 4850
+Wire Wire Line
+	7700 4850 7800 4850
+Wire Wire Line
+	7800 4850 7900 4850
+Wire Wire Line
+	7900 4850 8000 4850
+Wire Wire Line
+	8000 4850 8100 4850
+Wire Wire Line
+	8100 4850 8300 4850
 Wire Wire Line
 	8200 1950 8200 2050
@@
 Connection ~ 7100 1950
 Wire Wire Line
-	7000 1900 7000 2050
+	7000 1900 7000 1950
+Wire Wire Line
+	7000 1950 7000 2050
 Connection ~ 7000 1950
 $Comp
-L VDD_3V3B #PWR0318
+L VDD_3V3B #PWR0319
 U 1 1 58BD7134
 P 7000 1900
-F 0 "#PWR0318" H 7000 1750 50  0001 C CNN
+F 0 "#PWR0319" H 7000 1750 50  0001 C CNN
 F 1 "VDD_3V3B" H 7000 2050 50  0000 C CNN
 F 2 "" H 7000 1900 50  0000 C CNN
@@
 $EndComp
 $Comp
-L GNDD #PWR0319
+L GNDD #PWR0320
 U 1 1 58BD73F7
 P 6800 4925
-F 0 "#PWR0319" H 6800 4675 50  0001 C CNN
+F 0 "#PWR0320" H 6800 4675 50  0001 C CNN
 F 1 "GNDD" H 6800 4775 50  0000 C CNN
 F 2 "" H 6800 4925 50  0001 C CNN
@@
 	6900 2550 6150 2550
 Wire Wire Line
-	6150 2650 8425 2650
+	6150 2650 7000 2650
+Wire Wire Line
+	7000 2650 8425 2650
 Connection ~ 7000 2650
 Wire Wire Line
@@
 $EndComp
 $Comp
-L GNDD #PWR0320
+L GNDD #PWR0321
 U 1 1 58BDE353
 P 9525 2650
-F 0 "#PWR0320" H 9525 2400 50  0001 C CNN
+F 0 "#PWR0321" H 9525 2400 50  0001 C CNN
 F 1 "GNDD" V 9525 2450 50  0000 C CNN
 F 2 "" H 9525 2650 50  0000 C CNN
@@
 	7200 2850 7200 2350
 Wire Wire Line
-	7000 1950 8200 1950
+	7000 1950 7100 1950
+Wire Wire Line
+	7100 1950 7200 1950
+Wire Wire Line
+	7200 1950 7300 1950
+Wire Wire Line
+	7300 1950 8200 1950
 Text HLabel 8400 4050 2    60   BiDi ~ 0
 GPIO2_23
@@
 Text Notes 6750 5375 0    60   ~ 0
 0 1 2 3 4 5 6 7 8 9 0 1 2 3 4 5\n0 0 x 1 1 1 0 0 0 0 0 0 0 0 1 0
+Text Label 6200 4050 0    60   ~ 0
+LCD_HSYNC
+Text Label 6200 4150 0    60   ~ 0
+LCD_VSYNC
+Text Label 6200 4250 0    60   ~ 0
+LCD_CLOCK
+Text Label 6200 4350 0    60   ~ 0
+LCD_ENABLE
+Text Label 1075 4950 0    60   ~ 0
+SYS_BOOT0
+Text Label 1075 5050 0    60   ~ 0
+SYS_BOOT1
+Text Label 1075 5150 0    60   ~ 0
+SYS_BOOT2
+Text Label 1075 5250 0    60   ~ 0
+SYS_BOOT3
+Text Label 1075 5350 0    60   ~ 0
+SYS_BOOT4
+Text Label 1075 5450 0    60   ~ 0
+SYS_BOOT5
+Text Label 1075 5550 0    60   ~ 0
+SYS_BOOT6
+Text Label 1075 5650 0    60   ~ 0
+SYS_BOOT7
+Text Label 1075 5750 0    60   ~ 0
+SYS_BOOT8
+Text Label 1075 5850 0    60   ~ 0
+SYS_BOOT9
+Text Label 1075 5950 0    60   ~ 0
+SYS_BOOT10
+Text Label 1075 6050 0    60   ~ 0
+SYS_BOOT11
+Text Label 1075 6150 0    60   ~ 0
+SYS_BOOT12
+Text Label 1075 6250 0    60   ~ 0
+SYS_BOOT13
+Text Label 1075 6350 0    60   ~ 0
+SYS_BOOT14
+Text Label 1075 6450 0    60   ~ 0
+SYS_BOOT15
+Text Label 1075 6550 0    60   ~ 0
+LCD_HSYNC
+Text Label 1075 6650 0    60   ~ 0
+LCD_VSYNC
+Text Label 1075 6750 0    60   ~ 0
+LCD_CLOCK
+Text Label 1075 6850 0    60   ~ 0
+LCD_ENABLE
+Text HLabel 1075 4800 2    60   Output ~ 0
+HDMI_INT
+Text HLabel 2200 4800 0    60   BiDi ~ 0
+CSDA
+Text HLabel 2200 4975 0    60   Input ~ 0
+CSCL
+Text HLabel 2200 5150 0    60   Input ~ 0
+ACLK
+Text HLabel 2200 5300 0    60   Input ~ 0
+AP0
+Text HLabel 2225 5475 0    60   Input ~ 0
+AP1
+Text HLabel 1075 4700 2    60   Input ~ 0
+HDMICLK_DIS
 $EndSCHEMATC
