File: usb.sch (KiCad schematic (older format))
At the start: 35 parts, among them IC1 OSD335x, IC2 SN74LVC2G241DCUR, U5 TPS2065CDGN, U6 TPD4S012, U7 TPD4S012

Commit message: wip erc
Changed lines of the file:
@@
 $EndComp
 Wire Wire Line
-	4425 4400 6200 4400
-Wire Wire Line
-	6200 4400 6650 4400
-Wire Wire Line
-	4425 4500 6100 4500
-Wire Wire Line
-	6100 4500 6650 4500
+	4425 4400 6650 4400
+Wire Wire Line
+	4425 4500 6650 4500
 Wire Wire Line
 	6200 5850 6200 4400
@@
 	6000 5850 6000 4700
 Wire Wire Line
-	4425 4700 6000 4700
-Wire Wire Line
-	6000 4700 6650 4700
+	4425 4700 6650 4700
 Wire Wire Line
 	5550 6350 5550 6750
@@
 	5550 6750 6050 6750
 Wire Wire Line
-	6050 6700 6050 6750
-Wire Wire Line
-	6050 6750 6050 6775
+	6050 6700 6050 6775
 Wire Wire Line
 	5550 5850 5900 5850
@@
 	4250 6750 4750 6750
 Wire Wire Line
-	4750 6700 4750 6750
-Wire Wire Line
-	4750 6750 4750 6775
+	4750 6700 4750 6775
 Wire Wire Line
 	4250 5600 4250 6050
@@
 	4900 5850 4900 5100
 Wire Wire Line
-	1150 5100 4900 5100
-Wire Wire Line
-	4900 5100 6575 5100
+	1150 5100 6575 5100
 Wire Wire Line
 	4800 5850 4800 5200
 Wire Wire Line
-	1150 5200 4800 5200
-Wire Wire Line
-	4800 5200 6500 5200
+	1150 5200 6500 5200
 Wire Wire Line
 	5925 5600 6650 5600
@@
 	6425 5300 3500 5300
 Wire Wire Line
-	1150 5300 1200 5300
-Wire Wire Line
-	1200 5300 1500 5300
-Wire Wire Line
-	1800 5300 2100 5300
-Wire Wire Line
-	2100 5300 3200 5300
+	1150 5300 1500 5300
+Wire Wire Line
+	1800 5300 3200 5300
 Wire Wire Line
 	6650 5700 6525 5700
@@
 	6525 7125 3100 7125
 Wire Wire Line
-	3100 6325 3100 7125
-Wire Wire Line
-	3100 7125 3100 7175
+	3100 6325 3100 7175
 Connection ~ 3100 7125
 Wire Wire Line
-	3600 6075 3600 6125
-Wire Wire Line
-	3600 6125 3600 6225
-Wire Wire Line
-	3100 6125 3150 6125
-Wire Wire Line
-	3150 6125 3600 6125
+	3600 6075 3600 6225
+Wire Wire Line
+	3100 6125 3600 6125
 Wire Wire Line
 	3150 6125 3150 6225
@@
 	2100 6325 2175 6325
 Wire Wire Line
-	2100 5300 2100 5600
-Wire Wire Line
-	2100 5600 2100 6125
-Wire Wire Line
-	2100 6125 2100 6225
-Wire Wire Line
-	2100 6225 2100 6325
+	2100 5300 2100 6325
 Wire Wire Line
 	2100 6125 2175 6125
@@
 	2650 6925 2650 6875
 Wire Wire Line
-	2600 6875 2650 6875
-Wire Wire Line
-	2650 6875 2700 6875
+	2600 6875 2700 6875
 Wire Wire Line
 	2700 6875 2700 6800
@@
 	1850 6375 1850 6425
 Wire Wire Line
-	1150 6425 1850 6425
-Wire Wire Line
-	1850 6425 2175 6425
+	1150 6425 2175 6425
 Connection ~ 1850 6425
 Wire Wire Line
-	2100 5600 4250 5600
-Wire Wire Line
-	4250 5600 4600 5600
+	2100 5600 4600 5600
 Connection ~ 2100 5600
 Wire Wire Line
@@
 	3300 2850 3225 2850
 Wire Wire Line
-	3225 2800 3225 2850
-Wire Wire Line
-	3225 2850 3225 3000
+	3225 2800 3225 3000
 $Comp
 L VDD_3V3B #PWR43
@@
 	2200 3775 2200 3400
 Wire Wire Line
-	2125 3400 2200 3400
-Wire Wire Line
-	2200 3400 2775 3400
+	2125 3400 2775 3400
 $Comp
 L GNDD #PWR38
@@
 $EndComp
 Wire Wire Line
-	9700 5350 9700 5450
-Wire Wire Line
-	9700 5450 9700 5525
+	9700 5350 9700 5525
 Wire Wire Line
 	10700 5450 10700 5350
@@
 Connection ~ 9800 5450
 Wire Wire Line
-	9700 5450 9800 5450
-Wire Wire Line
-	9800 5450 9900 5450
-Wire Wire Line
-	9900 5450 10000 5450
-Wire Wire Line
-	10000 5450 10100 5450
-Wire Wire Line
-	10100 5450 10200 5450
-Wire Wire Line
-	10200 5450 10300 5450
-Wire Wire Line
-	10300 5450 10400 5450
-Wire Wire Line
-	10400 5450 10500 5450
-Wire Wire Line
-	10500 5450 10600 5450
-Wire Wire Line
-	10600 5450 10700 5450
+	9700 5450 10700 5450
 Wire Wire Line
 	10700 2400 10700 2750
 Wire Wire Line
-	10600 2350 10600 2400
-Wire Wire Line
-	10600 2400 10600 2750
+	10600 2350 10600 2750
 Connection ~ 10600 2400
 Wire Wire Line
@@
 	9800 3000 9050 3000
 Wire Wire Line
-	9050 3100 10300 3100
-Wire Wire Line
-	10300 3100 10750 3100
+	9050 3100 10750 3100
 Connection ~ 10300 3100
 Wire Wire Line
@@
 	10500 3300 10500 3050
 Wire Wire Line
-	10300 2400 10400 2400
-Wire Wire Line
-	10400 2400 10500 2400
-Wire Wire Line
-	10500 2400 10600 2400
-Wire Wire Line
-	10600 2400 10700 2400
+	10300 2400 10700 2400
 Wire Wire Line
 	10300 2400 10300 2750
@@
 	9850 5900 9850 6000
 Wire Wire Line
-	9650 6000 9850 6000
-Wire Wire Line
-	9850 6000 9950 6000
+	9650 6000 9950 6000
 Text HLabel 9950 6000 2    60   BiDi ~ 0
 GPIO0_7
@@
 $EndComp
 Wire Wire Line
-	6550 1600 6600 1600
-Wire Wire Line
-	6600 1600 6650 1600
+	6550 1600 6650 1600
 Wire Wire Line
 	6600 1800 6650 1800
 Wire Wire Line
-	6600 1600 6600 1700
-Wire Wire Line
-	6600 1700 6600 1800
+	6600 1600 6600 1800
 Connection ~ 6600 1600
 Wire Wire Line
@@
 	6550 1950 6600 1950
 Wire Wire Line
-	6600 1900 6600 1950
-Wire Wire Line
-	6600 1950 6600 2000
+	6600 1900 6600 2000
 Wire Wire Line
 	6600 1900 6650 1900
