File: mateboard.kicad_pcb (KiCad board)
At the start: 8 copper layers, 1 part

Commit message: autosave ignored
Parts:
- removed the REF** at (77.4, 57.4)
- added REF**: OSD335x, footprints:OSD3358-BAS-BGA400, F.Cu at (153.0, 116.2)
Routing:
- net (no net): track 21.0 -> 0.00 mm, vias 2 -> 0
Other:
- copper layers 8 -> 6

Commit message: start placing
Parts:
- removed REF**: OSD335x, footprints:OSD3358-BAS-BGA400
- added AE1: 2.4GHz Antenna, footprints:2450AT43B100E, F.Cu at (148.5, 105.0)
- added C1, C2, C21, C22, C23, C24, C7, C8: 2.2uF/6.3V, Capacitors_SMD:C_0603, F.Cu at (148.5, 105.0)
- added C10, C11, C3, C37, C6, C9: 10uF/6.3V, Capacitors_SMD:C_0603, F.Cu at (148.5, 105.0)
- added C12, C14, C15, C20, C26, C27, C28, C29, C30, C31, C32, C33, C39, C4, C5: 100nF/6.3V, Capacitors_SMD:C_0402, F.Cu at (148.5, 105.0)
- added C13: 220uF/6.3V, Capacitors_Tantalum_SMD:CP_Tantalum_Case-A_EIA-3216-18_Reflow, F.Cu at (148.5, 105.0)
- added C16, C17, C18, C19: 18pF/50V, Capacitors_SMD:C_0402, F.Cu at (148.5, 105.0)
- added C25: 4.7uF/6.3V, Capacitors_SMD:C_0805, F.Cu at (148.5, 105.0)
- added C34, C35, C36: 10pF, Capacitors_SMD:C_0402, F.Cu at (148.5, 105.0)
- added C38: 1uF/6.3V, Capacitors_SMD:C_0402, F.Cu at (148.5, 105.0)
- added C40: DNP 47uF, Capacitors_Tantalum_SMD:CP_Tantalum_Case-A_EIA-3216-18_Reflow, F.Cu at (148.5, 105.0)
- added D1, D2, D3: STPS140A, Diodes_SMD:D_SMA_Standard, F.Cu at (148.5, 105.0)
- added D4: BAT54C, TO_SOT_Packages_SMD:SOT-23, F.Cu at (148.5, 105.0)
- added D5, D6: LTST-C191TBKT, LEDs:LED_0603, F.Cu at (148.5, 105.0)
- added IC1: OSD335x, footprints:OSD3358-BAS-BGA400, F.Cu at (94.8, 57.0)
- added IC2: SN74LVC2G241DCUR, Housings_SSOP:VSSOP-8_2.3x2mm_Pitch0.5mm, F.Cu at (148.5, 105.0)
- added IC3: NAND_4GB, footprints:WFBGA153, F.Cu at (115.1, 140.1)
- added IC4: WL1835MODGBMOCT, bbblue:BeagleBone_Blue-GHI-IC_MOC-100(TI), F.Cu at (105.8, 104.5)
- added J1: IO1, footprints:DF40C-70DP-0.4V_51_, B.Cu at (79.9, 98.0)
- added J10, J11, J13, J14, J5, J6, J7, J8, J9: TEST_1P, Measurement_Points:Measurement_Point_Round-SMD-Pad_Small, F.Cu at (148.5, 105.0)
- added J12, J4: ANT2, footprints:BeagleBone_Blue-GHI-CONNECTORS_U.FL-R-SMT-1, F.Cu at (148.5, 105.0)
- added J15: VDDS_PLL, Measurement_Points:Measurement_Point_Round-SMD-Pad_Small, F.Cu at (148.5, 105.0)
- added J16: VDDS_DDR, Measurement_Points:Measurement_Point_Round-SMD-Pad_Small, F.Cu at (148.5, 105.0)
- added J17: VDD_MPU, Measurement_Points:Measurement_Point_Round-SMD-Pad_Small, F.Cu at (148.5, 105.0)
- added J18: VDD_CORE, Measurement_Points:Measurement_Point_Round-SMD-Pad_Small, F.Cu at (148.5, 105.0)
- added J2: IO2, footprints:DF40C-70DP-0.4V_51_, F.Cu at (148.5, 105.0)
- added J3: GS2, Connectors:GS2, F.Cu at (153.6, 113.1)
- added L1: BLM21AG221SN1D, Resistors_SMD:R_0805, F.Cu at (148.5, 105.0)
- added L2: 150ohm 1000mA, Resistors_SMD:R_0805, F.Cu at (148.5, 105.0)
- added L3: 0.1ohm 0805, Resistors_SMD:R_0805, F.Cu at (148.5, 105.0)
- added L4, L5: BLM15AG102SN1D, Resistors_SMD:R_0402, F.Cu at (148.5, 105.0)
- added Q1, Q2: BSS138, TO_SOT_Packages_SMD:SOT-23, F.Cu at (148.5, 105.0)
- added R1, R31: 1M, Resistors_SMD:R_0402, F.Cu at (148.5, 105.0)
- added R10, R34, R43, R9: 0R, Resistors_SMD:R_0402, F.Cu at (148.5, 105.0)
- added R11, R12: 0, Resistors_SMD:R_0402, F.Cu at (148.5, 105.0)
- added R13, R14, R15, R16, R17, R18, R19, R20, R21, R22, R23, R24, R25, R26, R27, R28, R7: 100k, Resistors_SMD:R_0402, F.Cu at (148.5, 105.0)
- added R2, R78, R83, R84: 1k, Resistors_SMD:R_0402, F.Cu at (148.5, 105.0)
- added R29: 100, Resistors_SMD:R_0402, F.Cu at (148.5, 105.0)
- added R3, R4, R58: 1.5k, Resistors_SMD:R_0402, F.Cu at (148.5, 105.0)
- added R30: 10k 1%, Resistors_SMD:R_0402, F.Cu at (148.5, 105.0)
- added R32: DNP 1M, Resistors_SMD:R_0402, F.Cu at (148.5, 105.0)
- added R33: 0 1%, Resistors_SMD:R_0402, F.Cu at (148.5, 105.0)
- added R35, R36, R37, R38, R39, R40, R41, R42, R44, R45, R46, R47, R48, R49, R5, R50, R52, R53, R54, R6, R8: 10k, Resistors_SMD:R_0402, F.Cu at (148.5, 105.0)
- added R51: DNP 0R, Resistors_SMD:R_0402, F.Cu at (148.5, 105.0)
- added R55, R60, R61, R62, R63, R64, R65, R67, R68, R69, R71, R72, R73, R74, R75, R76, R77, R79, R80, R81, R82: 33, Resistors_SMD:R_0402, F.Cu at (148.5, 105.0)
- added R56, R57: 150k, Resistors_SMD:R_0402, F.Cu at (148.5, 105.0)
- added R59, R66: DNP 1k, Resistors_SMD:R_0402, F.Cu at (148.5, 105.0)
- added R70: DNP 10k, Resistors_SMD:R_0402, F.Cu at (148.5, 105.0)
- added U1: AP2112K-3.3TRG1, TO_SOT_Packages_SMD:TSOT-23-5, F.Cu at (148.5, 105.0)
- added U10, U11: TXS0108, Housings_SSOP:TSSOP-20_4.4x6.5mm_Pitch0.65mm, F.Cu at (148.5, 105.0)
- added U2: AP2112K-1.8TRG1, TO_SOT_Packages_SMD:TSOT-23-5, F.Cu at (148.5, 105.0)
- added U3: TL1963A-33DCQR, footprints:SOT-223-6, F.Cu at (148.5, 105.0)
- added U4: 24LC32AT-I, TO_SOT_Packages_SMD:SOT-23-5, F.Cu at (148.5, 105.0)
- added U5: TPS2065CDGN, Housings_SSOP:VSSOP-8_2.3x2mm_Pitch0.5mm, F.Cu at (148.5, 105.0)
- added U6, U7: TPD4S012, footprints:SON-6, F.Cu at (148.5, 105.0)
- added U8: SN74LVC1G06DCK, TO_SOT_Packages_SMD:SOT-353_SC-70-5, F.Cu at (148.5, 105.0)
- added U9: 74LVC1G07DCK, TO_SOT_Packages_SMD:SOT-353_SC-70-5, F.Cu at (148.5, 105.0)
- added X1: NZ2520SB-32.768KHZ-NSA3534C, Crystals:Crystal_SMD_2520-4pin_2.5x2.0mm, F.Cu at (148.5, 105.0)
- added Y1: 24MHz, Crystals:Crystal_SMD_5032-2pin_5.0x3.2mm, F.Cu at (148.5, 105.0)
- added Y2: 32.768kHz, Crystals:Crystal_SMD_3215-2pin_3.2x1.5mm, F.Cu at (148.5, 105.0)

Commit message: wip placing
Parts:
- moved J3 79.6 mm to (92.9, 61.5), turned to 90 degrees
- moved C4 64.9 mm to (116.5, 48.5), turned to 180 degrees
- moved C7 63.8 mm to (116.2, 50.0), turned to 180 degrees
- moved C1 61.2 mm to (115.0, 53.8), turned to 90 degrees
- moved C9 61.2 mm to (111.2, 56.5)
- moved U1 60.1 mm to (118.0, 53.2), turned to 90 degrees
- moved R4 60.1 mm to (94.0, 79.8), turned to 180 degrees
- moved R3 59.6 mm to (94.0, 81.0), turned to 180 degrees
- moved U3 59.4 mm to (157.8, 46.4), turned to 90 degrees
- moved C3 59.1 mm to (114.8, 56.5), turned to 180 degrees
- moved IC1 19.7 mm to (108.6, 71.0)

Commit message: wip placing
Parts:
- IC3: footprint footprints:WFBGA153 -> bbblue:BeagleBone_Blue-GHI-IC_MICRON_EMMC_153
- J2: moved to B.Cu
- moved J2 112.0 mm to (41.9, 70.7), turned to 180 degrees
- moved AE1 109.2 mm to (52.7, 52.6), turned to 90 degrees
- moved U3 104.1 mm to (58.0, 76.0), turned to 180 degrees
- moved IC3 96.1 mm to (92.2, 46.8), turned to 90 degrees
- moved U10 85.2 mm to (74.5, 62.7)
- moved D1 81.5 mm to (70.0, 83.0)
- moved U11 80.7 mm to (74.9, 72.0)
- moved C11 72.7 mm to (80.0, 80.5), turned to 90 degrees
- moved U4 70.2 mm to (82.9, 80.2), turned to 270 degrees
- moved R5 69.6 mm to (82.4, 83.2)
- moved J1 67.3 mm to (135.4, 60.0)
- moved IC4 62.8 mm to (57.8, 63.9), turned to 180 degrees
- moved C10 55.1 mm to (97.0, 85.3)
- moved C12 55.1 mm to (97.0, 85.3)
- moved C13 55.1 mm to (97.0, 85.3)
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Connections:
- IC3 pad A1: (no net) -> /System-eMMC-GPIO/MMC1_DAT3
Other:
- board outline added: 70 x 50 mm
- net class Default: clearance 0.2 -> 0.15
- rule trace_clearance: 0.2 -> 0.15
- rule trace_min: 0.2 -> 0.15

Commit message: placing 1st iteration
Parts:
- added REF**: MountingHole_3.2mm_M3, Mounting_Holes:MountingHole_3.2mm_M3, F.Cu at (116.0, 44.0)
- added REF**: MountingHole_3.2mm_M3, Mounting_Holes:MountingHole_3.2mm_M3, F.Cu at (116.0, 86.0)
- added REF**: MountingHole_3.2mm_M3, Mounting_Holes:MountingHole_3.2mm_M3, F.Cu at (54.0, 86.0)
- added REF**: MountingHole_3.2mm_M3, Mounting_Holes:MountingHole_3.2mm_M3, F.Cu at (54.0, 44.0)
- J10, J11, J13, J14, J15, J16, J17, J18, J5, J6, J7, J8, J9: moved to B.Cu
- moved J4 56.0 mm to (53.1, 50.6), turned to 270 degrees
- moved C34 55.1 mm to (51.0, 55.0), turned to 90 degrees
- moved R70 53.4 mm to (53.7, 54.1), turned to 180 degrees
- moved R77 52.9 mm to (53.2, 55.8), turned to 90 degrees
- moved R52 52.4 mm to (55.6, 53.4), turned to 270 degrees
- moved C10 51.9 mm to (65.0, 44.5)
- moved R76 51.9 mm to (54.4, 55.8), turned to 90 degrees
- moved R53 51.4 mm to (56.8, 53.4), turned to 270 degrees
- moved R75 50.9 mm to (55.6, 55.8), turned to 90 degrees
- moved R54 50.5 mm to (58.0, 53.4), turned to 270 degrees
- moved J8 50.3 mm to (51.5, 64.0)
- moved R2 50.1 mm to (68.1, 44.4), turned to 270 degrees
- moved R74 49.9 mm to (56.8, 55.8), turned to 90 degrees
- moved C6 49.9 mm to (69.6, 43.6), turned to 270 degrees
- moved R50 49.5 mm to (59.2, 53.4), turned to 270 degrees
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Connections:
- IC4 pad G6: (no net) -> GNDD
Other:
- outline, holes or cut-outs redrawn
