File: power.sch (KiCad schematic (older format))
At the start: 27 parts, among them IC1 OSD335x, J3 GS2, U1 AP2112K-3.3TRG1, U2 AP2112K-1.8TRG1, U3 TL1963A-33DCQR, U4 24LC32AT-I

Commit message: erc passed
Parts:
- IC1: symbol OSD335x -> OSD335x-RESCUE-mateboard
Connections:
- no-connect marks 63 -> 64

Commit message: wip bom
Parts:
- C10, C11, C3, C6, C9: value 10uF/10V -> 10uF/6.3V
Changed lines of the file:
@@
 P 2200 1125
 F 0 "C3" H 2225 1225 50  0000 L CNN
-F 1 "10uF/10V" H 2225 1025 50  0000 L CNN
+F 1 "10uF/6.3V" H 2225 1025 50  0000 L CNN
 F 2 "" H 2238 975 50  0000 C CNN
 F 3 "" H 2200 1125 50  0000 C CNN
@@
 P 3250 1375
 F 0 "C9" H 3275 1475 50  0000 L CNN
-F 1 "10uF/10V" H 3275 1275 50  0000 L CNN
+F 1 "10uF/6.3V" H 3275 1275 50  0000 L CNN
 F 2 "" H 3288 1225 50  0000 C CNN
 F 3 "" H 3250 1375 50  0000 C CNN
@@
 P 4450 6875
 F 0 "C10" H 4475 6975 50  0000 L CNN
-F 1 "10uF/10V" H 4475 6775 50  0000 L CNN
+F 1 "10uF/6.3V" H 4475 6775 50  0000 L CNN
 F 2 "" H 4488 6725 50  0000 C CNN
 F 3 "" H 4450 6875 50  0000 C CNN
@@
 P 2625 7075
 F 0 "C6" H 2650 7175 50  0000 L CNN
-F 1 "10uF/10V" H 2650 6975 50  0000 L CNN
+F 1 "10uF/6.3V" H 2650 6975 50  0000 L CNN
 F 2 "" H 2663 6925 50  0000 C CNN
 F 3 "" H 2625 7075 50  0000 C CNN
@@
 P 8925 1750
 F 0 "C11" V 8975 1825 50  0000 L CNN
-F 1 "10uF/10V" V 9050 1525 50  0000 L CNN
+F 1 "10uF/6.3V" V 9050 1525 50  0000 L CNN
 F 2 "" H 8963 1600 50  0000 C CNN
 F 3 "" H 8925 1750 50  0000 C CNN

Commit message: wip footprint assoc
Parts:
- C1, C10, C11, C2, C3, C6, C7, C8, C9: footprint (none) -> Capacitors_SMD:C_0603
- C4, C5: footprint (none) -> Capacitors_SMD:C_0402
- D1, D2, D3: footprint (none) -> Diodes_SMD:D_SMA_Standard
- D4: footprint (none) -> TO_SOT_Packages_SMD:SOT-23
- IC1: footprint GHI-SoMs-Processors_OSD3358 -> footprints:OSD3358-BAS-BGA400
- L1: footprint (none) -> Resistors_SMD:R_0805
- R1, R2, R3, R4, R5: footprint (none) -> Resistors_SMD:R_0402
- U1, U2: footprint (none) -> TO_SOT_Packages_SMD:TSOT-23-5
Changed lines of the file:
@@
 F 0 "C3" H 2225 1225 50  0000 L CNN
 F 1 "10uF/6.3V" H 2225 1025 50  0000 L CNN
-F 2 "" H 2238 975 50  0000 C CNN
+F 2 "Capacitors_SMD:C_0603" H 2238 975 50  0001 C CNN
 F 3 "" H 2200 1125 50  0000 C CNN
 	1    2200 1125
@@
 F 0 "C9" H 3275 1475 50  0000 L CNN
 F 1 "10uF/6.3V" H 3275 1275 50  0000 L CNN
-F 2 "" H 3288 1225 50  0000 C CNN
+F 2 "Capacitors_SMD:C_0603" H 3288 1225 50  0001 C CNN
 F 3 "" H 3250 1375 50  0000 C CNN
 	1    3250 1375
@@
 F 0 "C1" H 800 4175 50  0000 L CNN
 F 1 "2.2uF/6.3V" H 800 3975 50  0000 L CNN
-F 2 "" H 813 3925 50  0000 C CNN
+F 2 "Capacitors_SMD:C_0603" H 813 3925 50  0001 C CNN
 F 3 "" H 775 4075 50  0000 C CNN
 	1    775  4075
@@
 F 0 "C4" H 2300 4275 50  0000 L CNN
 F 1 "100nF/6.3V" H 2300 4075 50  0000 L CNN
-F 2 "" H 2313 4025 50  0000 C CNN
+F 2 "Capacitors_SMD:C_0402" H 2313 4025 50  0001 C CNN
 F 3 "" H 2275 4175 50  0000 C CNN
 	1    2275 4175
@@
 F 0 "U1" H 1675 4300 50  0000 C CNN
 F 1 "AP2112K-3.3TRG1" H 1675 4225 50  0000 C CNN
-F 2 "" H 1725 3725 50  0000 L CNN
+F 2 "TO_SOT_Packages_SMD:TSOT-23-5" H 1725 3725 50  0001 L CNN
 F 3 "" H 1675 3975 50  0000 C CNN
 	1    1675 3975
@@
 F 0 "C7" H 2825 4275 50  0000 L CNN
 F 1 "2.2uF/6.3V" H 2825 4075 50  0000 L CNN
-F 2 "" H 2838 4025 50  0000 C CNN
+F 2 "Capacitors_SMD:C_0603" H 2838 4025 50  0001 C CNN
 F 3 "" H 2800 4175 50  0000 C CNN
 	1    2800 4175
@@
 F 0 "C2" H 800 5350 50  0000 L CNN
 F 1 "2.2uF/6.3V" H 800 5150 50  0000 L CNN
-F 2 "" H 813 5100 50  0000 C CNN
+F 2 "Capacitors_SMD:C_0603" H 813 5100 50  0001 C CNN
 F 3 "" H 775 5250 50  0000 C CNN
 	1    775  5250
@@
 F 0 "C5" H 2300 5450 50  0000 L CNN
 F 1 "100nF/6.3V" H 2300 5250 50  0000 L CNN
-F 2 "" H 2313 5200 50  0000 C CNN
+F 2 "Capacitors_SMD:C_0402" H 2313 5200 50  0001 C CNN
 F 3 "" H 2275 5350 50  0000 C CNN
 	1    2275 5350
@@
 F 0 "U2" H 1675 5475 50  0000 C CNN
 F 1 "AP2112K-1.8TRG1" H 1675 5400 50  0000 C CNN
-F 2 "" H 1725 4900 50  0000 L CNN
+F 2 "TO_SOT_Packages_SMD:TSOT-23-5" H 1725 4900 50  0001 L CNN
 F 3 "" H 1675 5150 50  0000 C CNN
 	1    1675 5150
@@
 F 0 "C8" H 2825 5450 50  0000 L CNN
 F 1 "2.2uF/6.3V" H 2825 5250 50  0000 L CNN
-F 2 "" H 2838 5200 50  0000 C CNN
+F 2 "Capacitors_SMD:C_0603" H 2838 5200 50  0001 C CNN
 F 3 "" H 2800 5350 50  0000 C CNN
 	1    2800 5350
@@
 F 0 "D4" H 2575 6625 30  0000 C CNN
 F 1 "BAT54C" H 2575 6675 30  0000 C CNN
-F 2 "" H 2425 6625 60  0001 C CNN
+F 2 "TO_SOT_Packages_SMD:SOT-23" H 2425 6625 60  0001 C CNN
 F 3 "" H 2425 6625 60  0001 C CNN
 	1    2425 6625
@@
 F 0 "D1" H 1100 6150 50  0000 C CNN
 F 1 "STPS140A" H 1100 5950 50  0000 C CNN
-F 2 "" H 1100 6050 50  0000 C CNN
+F 2 "Diodes_SMD:D_SMA_Standard" H 1100 6050 50  0001 C CNN
 F 3 "" H 1100 6050 50  0000 C CNN
 	1    1100 6050
@@
 F 0 "D2" H 1100 6475 50  0000 C CNN
 F 1 "STPS140A" H 1100 6275 50  0000 C CNN
-F 2 "" H 1100 6375 50  0000 C CNN
+F 2 "Diodes_SMD:D_SMA_Standard" H 1100 6375 50  0001 C CNN
 F 3 "" H 1100 6375 50  0000 C CNN
 	1    1100 6375
@@
 F 0 "D3" H 1100 6800 50  0000 C CNN
 F 1 "STPS140A" H 1100 6600 50  0000 C CNN
-F 2 "" H 1100 6700 50  0000 C CNN
+F 2 "Diodes_SMD:D_SMA_Standard" H 1100 6700 50  0001 C CNN
 F 3 "" H 1100 6700 50  0000 C CNN
 	1    1100 6700
@@
 F 0 "L1" V 1725 6375 50  0000 C CNN
 F 1 "BLM21AG221SN1D" V 1885 6375 50  0000 C CNN
-F 2 "" H 1775 6375 50  0000 C CNN
+F 2 "Resistors_SMD:R_0805" H 1775 6375 50  0001 C CNN
 F 3 "" H 1775 6375 50  0000 C CNN
 	1    1775 6375
@@
 F 0 "R1" V 2080 6600 50  0000 C CNN
 F 1 "1M" V 2000 6600 50  0000 C CNN
-F 2 "" V 1930 6600 50  0000 C CNN
+F 2 "Resistors_SMD:R_0402" V 1930 6600 50  0001 C CNN
 F 3 "" H 2000 6600 50  0000 C CNN
 	1    2000 6600
@@
 F 0 "R2" V 3080 6325 50  0000 C CNN
 F 1 "1k" V 3000 6325 50  0000 C CNN
-F 2 "" V 2930 6325 50  0000 C CNN
+F 2 "Resistors_SMD:R_0402" V 2930 6325 50  0001 C CNN
 F 3 "" H 3000 6325 50  0000 C CNN
 	1    3000 6325
@@
 F 0 "C10" H 4475 6975 50  0000 L CNN
 F 1 "10uF/6.3V" H 4475 6775 50  0000 L CNN
-F 2 "" H 4488 6725 50  0000 C CNN
+F 2 "Capacitors_SMD:C_0603" H 4488 6725 50  0001 C CNN
 F 3 "" H 4450 6875 50  0000 C CNN
 	1    4450 6875
@@
 F 0 "C6" H 2650 7175 50  0000 L CNN
 F 1 "10uF/6.3V" H 2650 6975 50  0000 L CNN
-F 2 "" H 2663 6925 50  0000 C CNN
+F 2 "Capacitors_SMD:C_0603" H 2663 6925 50  0001 C CNN
 F 3 "" H 2625 7075 50  0000 C CNN
 	1    2625 7075
@@
 F 0 "IC1" H 5175 3050 45  0000 L BNN
 F 1 "OSD335x" H 5100 2950 45  0000 L BNN
-F 2 "GHI-SoMs-Processors_OSD3358" H 5280 3175 20  0001 C CNN
+F 2 "footprints:OSD3358-BAS-BGA400" H 5280 3175 20  0001 C CNN
 F 3 "" H 5250 3025 60  0001 C CNN
 	3    5250 3025
@@
 F 0 "R3" V 3475 2600 50  0000 C CNN
 F 1 "1.5k" V 3500 2825 50  0000 C CNN
-F 2 "" V 3430 2825 50  0001 C CNN
+F 2 "Resistors_SMD:R_0402" V 3430 2825 50  0001 C CNN
 F 3 "" H 3500 2825 50  0001 C CNN
 	1    3500 2825
@@
 F 0 "R4" V 3475 2700 50  0000 C CNN
 F 1 "1.5k" V 3500 2925 50  0000 C CNN
-F 2 "" V 3430 2925 50  0001 C CNN
+F 2 "Resistors_SMD:R_0402" V 3430 2925 50  0001 C CNN
 F 3 "" H 3500 2925 50  0001 C CNN
 	1    3500 2925
@@
 F 0 "IC1" H 9825 4825 45  0000 L BNN
 F 1 "OSD335x" H 9750 4725 45  0000 L BNN
-F 2 "GHI-SoMs-Processors_OSD3358" H 9930 4950 20  0001 C CNN
+F 2 "footprints:OSD3358-BAS-BGA400" H 9930 4950 20  0001 C CNN
 F 3 "" H 9900 4800 60  0001 C CNN
 	4    9900 4800
@@
 F 0 "C11" V 8975 1825 50  0000 L CNN
 F 1 "10uF/6.3V" V 9050 1525 50  0000 L CNN
-F 2 "" H 8963 1600 50  0000 C CNN
+F 2 "Capacitors_SMD:C_0603" H 8963 1600 50  0001 C CNN
 F 3 "" H 8925 1750 50  0000 C CNN
 	1    8925 1750
@@
 F 0 "R5" V 9205 2150 50  0000 C CNN
 F 1 "10k" V 9125 2150 50  0000 C CNN
-F 2 "" V 9055 2150 50  0001 C CNN
+F 2 "Resistors_SMD:R_0402" V 9055 2150 50  0001 C CNN
 F 3 "" H 9125 2150 50  0001 C CNN
 	1    9125 2150

Commit message: wip footprint assoc
Parts:
- U3: footprint (none) -> footprints:SOT-223-6
Changed lines of the file:
@@
 F 0 "U3" H 3650 7050 60  0000 C CNN
 F 1 "TL1963A-33DCQR" H 3650 6950 60  0000 C CNN
-F 2 "" H 3800 6475 60  0001 C CNN
+F 2 "footprints:SOT-223-6" H 3800 6475 60  0001 C CNN
 F 3 "" H 3800 6475 60  0001 C CNN
 	1    3650 6725

Commit message: arranging signals
Parts:
- added J19: VDD_3V3AUX, Measurement_Points:Measurement_Point_Round-SMD-Pad_Small, symbol TEST_1P
Connections:
- net VDD_3V3AUX: no longer names the net of IC1.Y11 (VDD_3V3AUX)
- net VDD_3V3AUX: now also J19.1
Changed lines of the file:
@@
-	0    1    1    0
-$EndComp
-$Comp
-L VDD_3V3AUX #PWR051
-U 1 1 58DBDE72
-P 7100 2225
-F 0 "#PWR051" H 7100 2075 50  0001 C CNN
-F 1 "VDD_3V3AUX" V 7100 2575 50  0000 C CNN
-F 2 "" H 7100 2225 50  0000 C CNN
-F 3 "" H 7100 2225 50  0000 C CNN
-	1    7100 2225
 	0    1    1    0
 $EndComp
@@
 	3150 2925 3350 2925
 $Comp
-L VDD_3V3B #PWR052
+L VDD_3V3B #PWR051
 U 1 1 58DC04C7
 P 3075 2825
-F 0 "#PWR052" H 3075 2675 50  0001 C CNN
+F 0 "#PWR051" H 3075 2675 50  0001 C CNN
 F 1 "VDD_3V3B" V 3075 3150 50  0000 C CNN
 F 2 "" H 3075 2825 50  0000 C CNN
@@
 PMIC_INT
 $Comp
-L VDD_1V8 #PWR053
+L VDD_1V8 #PWR052
 U 1 1 58DC1F01
 P 6750 3425
-F 0 "#PWR053" H 6750 3275 50  0001 C CNN
+F 0 "#PWR052" H 6750 3275 50  0001 C CNN
 F 1 "VDD_1V8" V 6750 3700 50  0000 C CNN
 F 2 "" H 6750 3425 50  0000 C CNN
@@
 	4000 1925 4050 1925
 $Comp
-L VDD_3V3B #PWR054
+L VDD_3V3B #PWR053
 U 1 1 58E264BB
 P 9625 1700
-F 0 "#PWR054" H 9625 1550 50  0001 C CNN
+F 0 "#PWR053" H 9625 1550 50  0001 C CNN
 F 1 "VDD_3V3B" H 9625 1850 50  0000 C CNN
 F 2 "" H 9625 1700 50  0000 C CNN
@@
 $EndComp
 $Comp
-L GNDD #PWR055
+L GNDD #PWR054
 U 1 1 58E264C8
 P 8775 1750
-F 0 "#PWR055" H 8775 1500 50  0001 C CNN
+F 0 "#PWR054" H 8775 1500 50  0001 C CNN
 F 1 "GNDD" V 8775 1550 50  0000 C CNN
 F 2 "" H 8775 1750 50  0000 C CNN
@@
 Connection ~ 9125 1750
 $Comp
-L GNDD #PWR056
+L GNDD #PWR055
 U 1 1 58E264DC
 P 9625 2550
-F 0 "#PWR056" H 9625 2300 50  0001 C CNN
+F 0 "#PWR055" H 9625 2300 50  0001 C CNN
 F 1 "GNDD" H 9625 2400 50  0000 C CNN
 F 2 "" H 9625 2550 50  0000 C CNN
@@
 I2C0_SCL
 $Comp
-L PWR_FLAG #FLG057
+L PWR_FLAG #FLG056
 U 1 1 58DC25FF
 P 3250 1175
-F 0 "#FLG057" H 3250 1250 50  0001 C CNN
+F 0 "#FLG056" H 3250 1250 50  0001 C CNN
 F 1 "PWR_FLAG" H 3250 1325 50  0001 C CNN
 F 2 "" H 3250 1175 50  0001 C CNN
@@
 NoConn ~ 6450 4625
 $Comp
-L PWR_FLAG #FLG058
+L PWR_FLAG #FLG057
 U 1 1 58DD16BF
 P 2200 925
-F 0 "#FLG058" H 2200 1000 50  0001 C CNN
+F 0 "#FLG057" H 2200 1000 50  0001 C CNN
 F 1 "PWR_FLAG" H 2200 1075 50  0001 C CNN
 F 2 "" H 2200 925 50  0001 C CNN
@@
 	4300 6725 4175 6725
 $Comp
-L PWR_FLAG #FLG059
+L PWR_FLAG #FLG058
 U 1 1 58C61A6B
 P 2625 6375
-F 0 "#FLG059" H 2625 6450 50  0001 C CNN
+F 0 "#FLG058" H 2625 6450 50  0001 C CNN
 F 1 "PWR_FLAG" H 2625 6525 50  0000 C CNN
 F 2 "" H 2625 6375 50  0001 C CNN
@@
 $EndComp
 $Comp
-L GNDD #PWR060
+L GNDD #PWR059
 U 1 1 589F7BA8
 P 2625 7225
-F 0 "#PWR060" H 2625 6975 50  0001 C CNN
+F 0 "#PWR059" H 2625 6975 50  0001 C CNN
 F 1 "GNDD" H 2625 7075 50  0000 C CNN
 F 2 "" H 2625 7225 50  0000 C CNN
@@
 $EndComp
 $Comp
-L VDD_3V3_WIFI #PWR061
+L VDD_3V3_WIFI #PWR060
 U 1 1 589F30A3
 P 4300 6500
-F 0 "#PWR061" H 4300 6350 50  0001 C CNN
+F 0 "#PWR060" H 4300 6350 50  0001 C CNN
 F 1 "VDD_3V3_WIFI" H 4300 6650 50  0000 C CNN
 F 2 "" H 4300 6500 50  0000 C CNN
@@
 $EndComp
 $Comp
-L GNDD #PWR062
+L GNDD #PWR061
 U 1 1 589F2F41
 P 4450 7025
-F 0 "#PWR062" H 4450 6775 50  0001 C CNN
+F 0 "#PWR061" H 4450 6775 50  0001 C CNN
 F 1 "GNDD" H 4450 6875 50  0000 C CNN
 F 2 "" H 4450 7025 50  0000 C CNN
@@
 $EndComp
 $Comp
-L GNDD #PWR063
+L GNDD #PWR062
 U 1 1 589F09AB
 P 4175 6825
-F 0 "#PWR063" H 4175 6575 50  0001 C CNN
+F 0 "#PWR062" H 4175 6575 50  0001 C CNN
 F 1 "GNDD" H 4175 6675 50  0000 C CNN
 F 2 "" H 4175 6825 50  0000 C CNN
@@
 $EndComp
 $Comp
-L GNDD #PWR064
+L GNDD #PWR063
 U 1 1 589F0916
 P 3100 6825
-F 0 "#PWR064" H 3100 6575 50  0001 C CNN
+F 0 "#PWR063" H 3100 6575 50  0001 C CNN
 F 1 "GNDD" H 3100 6675 50  0000 C CNN
 F 2 "" H 3100 6825 50  0000 C CNN
@@
 $EndComp
 $Comp
-L VDD_3V3B #PWR065
+L VDD_3V3B #PWR064
 U 1 1 589F00BA
 P 3000 6175
-F 0 "#PWR065" H 3000 6025 50  0001 C CNN
+F 0 "#PWR064" H 3000 6025 50  0001 C CNN
 F 1 "VDD_3V3B" H 3000 6325 50  0000 C CNN
 F 2 "" H 3000 6175 50  0000 C CNN
@@
 NoConn ~ 2425 6425
 $Comp
-L GNDD #PWR066
+L GNDD #PWR065
 U 1 1 589EF269
 P 2425 6825
-F 0 "#PWR066" H 2425 6575 50  0001 C CNN
+F 0 "#PWR065" H 2425 6575 50  0001 C CNN
 F 1 "GNDD" H 2425 6675 50  0000 C CNN
 F 2 "" H 2425 6825 50  0000 C CNN
@@
 $EndComp
 $Comp
-L GNDD #PWR067
+L GNDD #PWR066
 U 1 1 589EF1D7
 P 2000 6750
-F 0 "#PWR067" H 2000 6500 50  0001 C CNN
+F 0 "#PWR066" H 2000 6500 50  0001 C CNN
 F 1 "GNDD" H 2000 6600 50  0000 C CNN
 F 2 "" H 2000 6750 50  0000 C CNN
@@
 $EndComp
 $Comp
-L USB_DC #PWR068
+L USB_DC #PWR067
 U 1 1 589ED7EB
 P 950 6700
-F 0 "#PWR068" H 950 6550 50  0001 C CNN
+F 0 "#PWR067" H 950 6550 50  0001 C CNN
 F 1 "USB_DC" V 950 6975 50  0000 C CNN
 F 2 "" H 950 6700 50  0000 C CNN
@@
 $EndComp
 $Comp
-L VDD_5V #PWR069
+L VDD_5V #PWR068
 U 1 1 589ED75C
 P 950 6375
-F 0 "#PWR069" H 950 6225 50  0001 C CNN
+F 0 "#PWR068" H 950 6225 50  0001 C CNN
 F 1 "VDD_5V" V 950 6625 50  0000 C CNN
 F 2 "" H 950 6375 50  0000 C CNN
@@
 $EndComp
 $Comp
-L SYS_5V #PWR070
+L SYS_5V #PWR069
 U 1 1 589ECB91
 P 950 6050
-F 0 "#PWR070" H 950 5900 50  0001 C CNN
+F 0 "#PWR069" H 950 5900 50  0001 C CNN
 F 1 "SYS_5V" V 950 6300 50  0000 C CNN
 F 2 "" H 950 6050 50  0000 C CNN
@@
 	-1   0    0    -1
 $EndComp
+$Comp
+L TEST_1P J19
+U 1 1 5906996C
+P 7100 2225
+F 0 "J19" V 7050 2275 50  0000 C CNN
+F 1 "VDD_3V3AUX" V 7100 2625 50  0000 C CNN
+F 2 "Measurement_Points:Measurement_Point_Round-SMD-Pad_Small" H 7300 2225 50  0001 C CNN
+F 3 "" H 7300 2225 50  0001 C CNN
+	1    7100 2225
+	0    1    1    0
+$EndComp
 $EndSCHEMATC
