File: wifi.sch (KiCad schematic (older format))
At the start: 69 parts, among them IC4 WL1835MODGBMOCT, J10 TEST_1P, J11 TEST_1P, J12 ANT2, J13 TEST_1P, J14 TEST_1P, J4 ANT2, J5 TEST_1P, J6 TEST_1P, J7 TEST_1P, J8 TEST_1P, J9 TEST_1P, Q1 BSS138, Q2 BSS138, U10 TXS0108, U11 TXS0108, X1 NZ2520SB-32.768KHZ-NSA3534C

Commit message: wip erc
Other:
- moved on the sheet: C33, D5, D6, Q1, Q2, R78, R83, R84, X1

Commit message: wip footprint assoc
Parts:
- C29, C30, C31, C32, C33, C34, C35, C36, C38, C39: footprint (none) -> Capacitors_SMD:C_0402
- C37: footprint (none) -> Capacitors_SMD:C_0603
- C40: footprint (none) -> Capacitors_Tantalum_SMD:CP_Tantalum_Case-A_EIA-3216-18_Reflow
- D5, D6: footprint (none) -> LEDs:LED_0603
- IC4: footprint (none) -> bbblue:BeagleBone_Blue-GHI-IC_MOC-100(TI)
- J10, J11, J13, J14, J5, J6, J7, J8, J9: footprint (none) -> Measurement_Points:Measurement_Point_Round-SMD-Pad_Small
- R48, R49, R50, R51, R52, R53, R54, R55, R56, R57, R58, R59, R60, R61, R62, R63, R64, R65, R66, R67, R68, R69, R70, R71, R72, R73, R74, R75, R76, R77, R78, R79, R80, R81, R82, R83, R84: footprint (none) -> Resistors_SMD:R_0402

Commit message: wip footprint assoc
Parts:
- J12, J4: footprint (none) -> bbblue:BeagleBone_Blue-GHI-CONNECTORS_U.FL-R-SMT-1
- U10, U11: footprint (none) -> Housings_SSOP:TSSOP-20_4.4x6.5mm_Pitch0.65mm
- X1: footprint (none) -> Crystals:Crystal_SMD_2520-4pin_2.5x2.0mm
Changed lines of the file:
@@
 F 0 "U10" H 3350 3775 60  0000 C CNN
 F 1 "TXS0108" H 3500 4975 60  0000 C CNN
-F 2 "" H 3600 4375 60  0001 C CNN
+F 2 "Housings_SSOP:TSSOP-20_4.4x6.5mm_Pitch0.65mm" H 3600 4375 60  0001 C CNN
 F 3 "" H 3600 4375 60  0001 C CNN
 	1    3600 4375
@@
 F 0 "U11" H 3350 5500 60  0000 C CNN
 F 1 "TXS0108" H 3500 6700 60  0000 C CNN
-F 2 "" H 3600 6100 60  0001 C CNN
+F 2 "Housings_SSOP:TSSOP-20_4.4x6.5mm_Pitch0.65mm" H 3600 6100 60  0001 C CNN
 F 3 "" H 3600 6100 60  0001 C CNN
 	1    3600 6100
@@
 F 0 "J4" H 7835 4820 50  0000 C CNN
 F 1 "ANT2" V 7940 4700 50  0000 C CNN
-F 2 "" H 7825 4700 50  0001 C CNN
+F 2 "bbblue:BeagleBone_Blue-GHI-CONNECTORS_U.FL-R-SMT-1" H 7825 4700 50  0001 C CNN
 F 3 "" H 7825 4700 50  0001 C CNN
 	1    7825 4700
@@
 F 0 "J12" H 9235 4995 50  0000 C CNN
 F 1 "ANT2" V 9340 4875 50  0000 C CNN
-F 2 "" H 9225 4875 50  0001 C CNN
+F 2 "bbblue:BeagleBone_Blue-GHI-CONNECTORS_U.FL-R-SMT-1" H 9225 4875 50  0001 C CNN
 F 3 "" H 9225 4875 50  0001 C CNN
 	1    9225 4875
@@
 F 0 "X1" H 4375 1400 60  0000 C CNN
 F 1 "NZ2520SB-32.768KHZ-NSA3534C" H 5100 1300 60  0000 C CNN
-F 2 "" H 4225 1650 60  0001 C CNN
+F 2 "Crystals:Crystal_SMD_2520-4pin_2.5x2.0mm" H 4225 1650 60  0001 C CNN
 F 3 "" H 4225 1650 60  0001 C CNN
 	1    4225 1650

Commit message: start placing
Parts:
- removed AE1: ACA-5036-A2-CC-S, symbol Antenna_Shield
- added AE1: 2.4GHz Antenna, footprints:2450AT43B100E, symbol Antenna
- J12, J4: footprint bbblue:BeagleBone_Blue-GHI-CONNECTORS_U.FL-R-SMT-1 -> footprints:BeagleBone_Blue-GHI-CONNECTORS_U.FL-R-SMT-1
Connections:
- net at C36.1: now also AE1.1 (A)
Changed lines of the file:
@@
 F 0 "J4" H 7835 4820 50  0000 C CNN
 F 1 "ANT2" V 7940 4700 50  0000 C CNN
-F 2 "bbblue:BeagleBone_Blue-GHI-CONNECTORS_U.FL-R-SMT-1" H 7825 4700 50  0001 C CNN
+F 2 "footprints:BeagleBone_Blue-GHI-CONNECTORS_U.FL-R-SMT-1" H 7825 4700 50  0001 C CNN
 F 3 "" H 7825 4700 50  0001 C CNN
 	1    7825 4700
@@
 F 0 "J12" H 9235 4995 50  0000 C CNN
 F 1 "ANT2" V 9340 4875 50  0000 C CNN
-F 2 "bbblue:BeagleBone_Blue-GHI-CONNECTORS_U.FL-R-SMT-1" H 9225 4875 50  0001 C CNN
+F 2 "footprints:BeagleBone_Blue-GHI-CONNECTORS_U.FL-R-SMT-1" H 9225 4875 50  0001 C CNN
 F 3 "" H 9225 4875 50  0001 C CNN
 	1    9225 4875
@@
 	9625 4400 9225 4400
 Connection ~ 9225 4400
-$Comp
-L Antenna_Shield AE1
-U 1 1 58BB7339
-P 10325 4200
-F 0 "AE1" H 10375 4525 50  0000 R CNN
-F 1 "ACA-5036-A2-CC-S" H 10775 4450 50  0000 R CNN
-F 2 "" H 10325 4300 50  0001 C CNN
-F 3 "" H 10325 4300 50  0001 C CNN
-	1    10325 4200
-	1    0    0    -1
-$EndComp
-Wire Wire Line
-	9925 4400 10325 4400
+Wire Wire Line
+	9925 4400 10300 4400
 $Comp
 L GNDD #PWR0151
-U 1 1 58BB8189
-P 10425 4400
-F 0 "#PWR0151" H 10425 4150 50  0001 C CNN
-F 1 "GNDD" H 10425 4250 50  0000 C CNN
-F 2 "" H 10425 4400 50  0000 C CNN
-F 3 "" H 10425 4400 50  0000 C CNN
-	1    10425 4400
-	1    0    0    -1
-$EndComp
-$Comp
-L GNDD #PWR0152
 U 1 1 58BB9360
 P 10125 3600
-F 0 "#PWR0152" H 10125 3350 50  0001 C CNN
+F 0 "#PWR0151" H 10125 3350 50  0001 C CNN
 F 1 "GNDD" H 10125 3450 50  0000 C CNN
 F 2 "" H 10125 3600 50  0000 C CNN
@@
 $EndComp
 $Comp
-L VDD_1V8_WIFI #PWR0153
+L VDD_1V8_WIFI #PWR0152
 U 1 1 58BBCC74
 P 4225 1200
-F 0 "#PWR0153" H 4225 1050 50  0001 C CNN
+F 0 "#PWR0152" H 4225 1050 50  0001 C CNN
 F 1 "VDD_1V8_WIFI" H 4225 1350 50  0000 C CNN
 F 2 "" H 4225 1200 50  0000 C CNN
@@
 Connection ~ 4225 1250
 $Comp
-L GNDD #PWR0154
+L GNDD #PWR0153
 U 1 1 58BBD93F
 P 4925 1250
-F 0 "#PWR0154" H 4925 1000 50  0001 C CNN
+F 0 "#PWR0153" H 4925 1000 50  0001 C CNN
 F 1 "GNDD" V 4925 1025 50  0000 C CNN
 F 2 "" H 4925 1250 50  0000 C CNN
@@
 $EndComp
 $Comp
-L GNDD #PWR0155
+L GNDD #PWR0154
 U 1 1 58BBEF7E
 P 4225 2000
-F 0 "#PWR0155" H 4225 1750 50  0001 C CNN
+F 0 "#PWR0154" H 4225 1750 50  0001 C CNN
 F 1 "GNDD" H 4225 1850 50  0000 C CNN
 F 2 "" H 4225 2000 50  0000 C CNN
@@
 	650  6050 1200 6050
 $Comp
-L VDD_1V8_WIFI #PWR0156
+L VDD_1V8_WIFI #PWR0155
 U 1 1 58BC3383
 P 10850 2950
-F 0 "#PWR0156" H 10850 2800 50  0001 C CNN
+F 0 "#PWR0155" H 10850 2800 50  0001 C CNN
 F 1 "VDD_1V8_WIFI" H 10850 3100 50  0000 C CNN
 F 2 "" H 10850 2950 50  0000 C CNN
@@
 Connection ~ 10850 3000
 $Comp
-L GNDD #PWR0157
+L GNDD #PWR0156
 U 1 1 58BC8869
 P 10750 3500
-F 0 "#PWR0157" H 10750 3250 50  0001 C CNN
+F 0 "#PWR0156" H 10750 3250 50  0001 C CNN
 F 1 "GNDD" H 10750 3350 50  0000 C CNN
 F 2 "" H 10750 3500 50  0000 C CNN
@@
 $EndComp
 $Comp
-L GNDD #PWR0158
+L GNDD #PWR0157
 U 1 1 58BC8916
 P 11000 3500
-F 0 "#PWR0158" H 11000 3250 50  0001 C CNN
+F 0 "#PWR0157" H 11000 3250 50  0001 C CNN
 F 1 "GNDD" H 11000 3350 50  0000 C CNN
 F 2 "" H 11000 3500 50  0000 C CNN
@@
 $EndComp
 $Comp
-L VDD_3V3_WIFI #PWR0159
+L VDD_3V3_WIFI #PWR0158
 U 1 1 58BCA01F
 P 10850 1950
-F 0 "#PWR0159" H 10850 1800 50  0001 C CNN
+F 0 "#PWR0158" H 10850 1800 50  0001 C CNN
 F 1 "VDD_3V3_WIFI" H 10850 2100 50  0000 C CNN
 F 2 "" H 10850 1950 50  0000 C CNN
@@
 $EndComp
 $Comp
-L GNDD #PWR0160
+L GNDD #PWR0159
 U 1 1 58BCAF5D
 P 10750 2450
-F 0 "#PWR0160" H 10750 2200 50  0001 C CNN
+F 0 "#PWR0159" H 10750 2200 50  0001 C CNN
 F 1 "GNDD" H 10750 2300 50  0000 C CNN
 F 2 "" H 10750 2450 50  0000 C CNN
@@
 $EndComp
 $Comp
-L GNDD #PWR0161
+L GNDD #PWR0160
 U 1 1 58BCB190
 P 10975 2450
-F 0 "#PWR0161" H 10975 2200 50  0001 C CNN
+F 0 "#PWR0160" H 10975 2200 50  0001 C CNN
 F 1 "GNDD" H 10975 2300 50  0000 C CNN
 F 2 "" H 10975 2450 50  0000 C CNN
@@
 	9125 550  9125 1150
 $Comp
-L GNDD #PWR0162
+L GNDD #PWR0161
 U 1 1 58BD1A26
 P 7750 1400
-F 0 "#PWR0162" H 7750 1150 50  0001 C CNN
+F 0 "#PWR0161" H 7750 1150 50  0001 C CNN
 F 1 "GNDD" V 7750 1175 50  0000 C CNN
 F 2 "" H 7750 1400 50  0000 C CNN
@@
 	975  2000 1275 2000
 $Comp
-L GNDD #PWR0163
+L GNDD #PWR0162
 U 1 1 58B8C8B1
 P 1575 2150
-F 0 "#PWR0163" H 1575 1900 50  0001 C CNN
+F 0 "#PWR0162" H 1575 1900 50  0001 C CNN
 F 1 "GNDD" H 1575 2000 50  0000 C CNN
 F 2 "" H 1575 2150 50  0000 C CNN
@@
 $EndComp
 $Comp
-L VDD_3V3_WIFI #PWR0164
+L VDD_3V3_WIFI #PWR0163
 U 1 1 58B8F17F
 P 1575 1150
-F 0 "#PWR0164" H 1575 1000 50  0001 C CNN
+F 0 "#PWR0163" H 1575 1000 50  0001 C CNN
 F 1 "VDD_3V3_WIFI" H 1575 1300 50  0000 C CNN
 F 2 "" H 1575 1150 50  0000 C CNN
@@
 	2150 2000 2450 2000
 $Comp
-L GNDD #PWR0165
+L GNDD #PWR0164
 U 1 1 58B9014E
 P 2750 2150
-F 0 "#PWR0165" H 2750 1900 50  0001 C CNN
+F 0 "#PWR0164" H 2750 1900 50  0001 C CNN
 F 1 "GNDD" H 2750 2000 50  0000 C CNN
 F 2 "" H 2750 2150 50  0000 C CNN
@@
 $EndComp
 $Comp
-L VDD_3V3_WIFI #PWR0166
+L VDD_3V3_WIFI #PWR0165
 U 1 1 58B90160
 P 2750 1150
-F 0 "#PWR0166" H 2750 1000 50  0001 C CNN
+F 0 "#PWR0165" H 2750 1000 50  0001 C CNN
 F 1 "VDD_3V3_WIFI" H 2750 1300 50  0000 C CNN
 F 2 "" H 2750 1150 50  0000 C CNN
@@
 Text HLabel 1300 4825 0    60   Input ~ 0
 LS_BUF_OE.CPU
+$Comp
+L Antenna AE1
+U 1 1 58E56AC2
+P 10300 4100
+F 0 "AE1" H 10225 4175 50  0000 R CNN
+F 1 "2.4GHz Antenna" H 10225 4100 50  0000 R CNN
+F 2 "footprints:2450AT43B100E" H 10300 4100 50  0001 C CNN
+F 3 "" H 10300 4100 50  0001 C CNN
+	1    10300 4100
+	1    0    0    -1
+$EndComp
+Wire Wire Line
+	10300 4400 10300 4300
 $EndSCHEMATC
